File: KiCad Files/DP1600i/DP1600i.sch (KiCad schematic (older format))
At the start: 31 parts, among them J10 D8, J23 D18, J24 D19, J27 5V, J28 5V, J4 Gnd, J5 D13, J55 D48, J56 D49, J57 D50, J58 D51, J59 D52, J6 D12, J60 D53, J61 Gnd, J62 Gnd, J65 RESET, J67 5V, J68 Gnd, J69 Gnd, J7 D11, J71 A0, J72 A1, J73 A2, J74 A3, J75 A4, J76 A5, J77 A6, J78 A7, J8 D10, J9 D9

Commit message: Add files via upload
Parts:
- removed J10: D8, Connector_PinHeader_2.54mm:PinHeader_1x01_P2.54mm_Vertical, symbol Connector:Conn_01x01_Male
- removed J23: D18, Connector_PinHeader_2.54mm:PinHeader_1x01_P2.54mm_Vertical, symbol Connector:Conn_01x01_Male
- removed J24: D19, Connector_PinHeader_2.54mm:PinHeader_1x01_P2.54mm_Vertical, symbol Connector:Conn_01x01_Male
- removed J27, J28, J67: 5V, Connector_PinHeader_2.54mm:PinHeader_1x01_P2.54mm_Vertical, symbol Connector:Conn_01x01_Male
- removed J4, J61, J62, J68, J69: Gnd, Connector_PinHeader_2.54mm:PinHeader_1x01_P2.54mm_Vertical, symbol Connector:Conn_01x01_Male
- removed J5: D13, Connector_PinHeader_2.54mm:PinHeader_1x01_P2.54mm_Vertical, symbol Connector:Conn_01x01_Male
- removed J55: D48, Connector_PinHeader_2.54mm:PinHeader_1x01_P2.54mm_Vertical, symbol Connector:Conn_01x01_Male
- removed J56: D49, Connector_PinHeader_2.54mm:PinHeader_1x01_P2.54mm_Vertical, symbol Connector:Conn_01x01_Male
- removed J57: D50, Connector_PinHeader_2.54mm:PinHeader_1x01_P2.54mm_Vertical, symbol Connector:Conn_01x01_Male
- removed J58: D51, Connector_PinHeader_2.54mm:PinHeader_1x01_P2.54mm_Vertical, symbol Connector:Conn_01x01_Male
- removed J59: D52, Connector_PinHeader_2.54mm:PinHeader_1x01_P2.54mm_Vertical, symbol Connector:Conn_01x01_Male
- removed J6: D12, Connector_PinHeader_2.54mm:PinHeader_1x01_P2.54mm_Vertical, symbol Connector:Conn_01x01_Male
- removed J60: D53, Connector_PinHeader_2.54mm:PinHeader_1x01_P2.54mm_Vertical, symbol Connector:Conn_01x01_Male
- removed J65: RESET, Connector_PinHeader_2.54mm:PinHeader_1x01_P2.54mm_Vertical, symbol Connector:Conn_01x01_Male
- removed J7: D11, Connector_PinHeader_2.54mm:PinHeader_1x01_P2.54mm_Vertical, symbol Connector:Conn_01x01_Male
- removed J71: A0, Connector_PinHeader_2.54mm:PinHeader_1x01_P2.54mm_Vertical, symbol Connector:Conn_01x01_Male
- removed J72: A1, Connector_PinHeader_2.54mm:PinHeader_1x01_P2.54mm_Vertical, symbol Connector:Conn_01x01_Male
- removed J73: A2, Connector_PinHeader_2.54mm:PinHeader_1x01_P2.54mm_Vertical, symbol Connector:Conn_01x01_Male
- removed J74: A3, Connector_PinHeader_2.54mm:PinHeader_1x01_P2.54mm_Vertical, symbol Connector:Conn_01x01_Male
- removed J75: A4, Connector_PinHeader_2.54mm:PinHeader_1x01_P2.54mm_Vertical, symbol Connector:Conn_01x01_Male
- removed J76: A5, Connector_PinHeader_2.54mm:PinHeader_1x01_P2.54mm_Vertical, symbol Connector:Conn_01x01_Male
- removed J77: A6, Connector_PinHeader_2.54mm:PinHeader_1x01_P2.54mm_Vertical, symbol Connector:Conn_01x01_Male
- removed J78: A7, Connector_PinHeader_2.54mm:PinHeader_1x01_P2.54mm_Vertical, symbol Connector:Conn_01x01_Male
- removed J8: D10, Connector_PinHeader_2.54mm:PinHeader_1x01_P2.54mm_Vertical, symbol Connector:Conn_01x01_Male
- removed J9: D9, Connector_PinHeader_2.54mm:PinHeader_1x01_P2.54mm_Vertical, symbol Connector:Conn_01x01_Male
- added J3: Conn_01x07, Connector_PinHeader_2.54mm:PinHeader_1x07_P2.54mm_Vertical, symbol Connector_Generic:Conn_01x07
- added J4, J9: Conn_01x08, Connector_PinHeader_2.54mm:PinHeader_1x08_P2.54mm_Vertical, symbol Connector_Generic:Conn_01x08
- added J5: Conn_01x04, Connector_PinHeader_2.54mm:PinHeader_1x04_P2.54mm_Vertical, symbol Connector_Generic:Conn_01x04
- added J6: Conn_01x02, Connector_PinHeader_2.54mm:PinHeader_1x02_P2.54mm_Vertical, symbol Connector_Generic:Conn_01x02
- added J7: Conn_02x04_Odd_Even, Connector_PinHeader_2.54mm:PinHeader_2x04_P2.54mm_Vertical, symbol Connector_Generic:Conn_02x04_Odd_Even
- added J8: Conn_01x05, Connector_PinHeader_2.54mm:PinHeader_1x05_P2.54mm_Vertical, symbol Connector_Generic:Conn_01x05
Connections:
- net labels added: MCU-D0, MCU-D1, MCU-D16, MCU-D17, MCU-D2, MCU-D3, MCU-D4, MCU-D5, MCU-D6, MCU-D7
- wire segments 0 -> 22
- no-connect marks 0 -> 1
Other:
- note added: "A4988 Dir"
- note added: "A4988 Step"
- note added: "Spare"
- note added: "Spare\n"

Commit message: Add files via upload
Other:
- note added: "Header pin connections to Arduino Mega 2560 header sockets"
- note removed: "Arduino Mega 2560 headers"
Changed lines of the file:
@@
 Text Notes 3400 1850 3    50   ~ 0
 (Inj4 control)
-Text Notes 7200 1400 0    100  ~ 0
-Arduino Mega 2560 headers
+Text Notes 2750 850  0    118  ~ 0
+Header pin connections to Arduino Mega 2560 header sockets
 Text GLabel 5250 1400 3    50   Input ~ 0
 MCU-D19

Commit message: Add files via upload
Changed lines of the file:
@@
 $Descr A4 11693 8268
 encoding utf-8
-Sheet 1 6
+Sheet 1 5
 Title "DP1600i"
 Date "2022-11-11"
@@
 F1 "file63700A4D.sch" 50
 $EndSheet
-$Sheet
-S 4950 6600 900  800
-U 637A4EA7
-F0 "temp1" 50
-F1 "file637A4EA6.sch" 50
-$EndSheet
 $Comp

Commit message: Add files via upload
Parts:
- removed J6: Conn_01x02, Connector_PinHeader_2.54mm:PinHeader_1x02_P2.54mm_Vertical, symbol Connector_Generic:Conn_01x02
- added J6: Conn_02x03_Odd_Even, Connector_PinHeader_2.54mm:PinHeader_2x03_P2.54mm_Vertical, symbol Connector_Generic:Conn_02x03_Odd_Even
Connections:
- net VDD: now also J6.1 (Pin_1), J6.2 (Pin_2)
- new net MCU-D24: J6.5 (Pin_5)
- no-connect marks 1 -> 4
Other:
- note added: "A4988 En\n"
- note removed: "Spare\n"
Changed lines of the file:
@@
 L power:VDD #PWR02
 U 1 1 63826E84
-P 7900 2350
-F 0 "#PWR02" H 7900 2200 50  0001 C CNN
-F 1 "VDD" V 7915 2477 50  0000 L CNN
-F 2 "" H 7900 2350 50  0001 C CNN
-F 3 "" H 7900 2350 50  0001 C CNN
-	1    7900 2350
+P 7600 2700
+F 0 "#PWR02" H 7600 2550 50  0001 C CNN
+F 1 "VDD" V 7615 2827 50  0000 L CNN
+F 2 "" H 7600 2700 50  0001 C CNN
+F 3 "" H 7600 2700 50  0001 C CNN
+	1    7600 2700
 	0    -1   -1   0
 $EndComp
@@
 L power:VDD #PWR038
 U 1 1 63827375
-P 8300 2350
-F 0 "#PWR038" H 8300 2200 50  0001 C CNN
-F 1 "VDD" V 8315 2477 50  0000 L CNN
-F 2 "" H 8300 2350 50  0001 C CNN
-F 3 "" H 8300 2350 50  0001 C CNN
-	1    8300 2350
+P 8450 2700
+F 0 "#PWR038" H 8450 2550 50  0001 C CNN
+F 1 "VDD" V 8465 2827 50  0000 L CNN
+F 2 "" H 8450 2700 50  0001 C CNN
+F 3 "" H 8450 2700 50  0001 C CNN
+	1    8450 2700
 	0    1    1    0
 $EndComp
@@
 Text Notes 4000 2050 1    50   ~ 0
 Spare
-Text GLabel 4650 1400 3    50   Input ~ 0
-MCU-D0
+Text GLabel 7600 2900 0    50   Input ~ 0
+MCU-D24
 Text GLabel 4550 1400 3    50   Input ~ 0
 MCU-D1
-Text Notes 4700 2050 1    50   ~ 0
-Spare\n
+Text Notes 7100 2950 2    50   ~ 0
+A4988 En\n
 Text Notes 4600 2050 1    50   ~ 0
 Spare
@@
 Text Notes 4400 2050 1    50   ~ 0
 Spare
-$Comp
-L Connector_Generic:Conn_01x02 J6
-U 1 1 6390E746
-P 8050 2150
-F 0 "J6" V 8150 2150 50  0000 R CNN
-F 1 "Conn_01x02" V 8250 2300 50  0000 R CNN
-F 2 "Connector_PinHeader_2.54mm:PinHeader_1x02_P2.54mm_Vertical" H 8050 2150 50  0001 C CNN
-F 3 "~" H 8050 2150 50  0001 C CNN
-	1    8050 2150
-	0    -1   -1   0
-$EndComp
 $Comp
 L Connector_Generic:Conn_01x04 J5
@@
 $EndComp
 Wire Wire Line
-	8150 2350 8300 2350
-Wire Wire Line
-	7900 2350 8050 2350
-Wire Wire Line
 	8650 3950 8300 3950
 Wire Wire Line
@@
 	1    0    0    -1
 $EndComp
+$Comp
+L Connector_Generic:Conn_02x03_Odd_Even J6
+U 1 1 6394E4BE
+P 7950 2800
+F 0 "J6" H 8000 3117 50  0000 C CNN
+F 1 "Conn_02x03_Odd_Even" H 8000 3026 50  0000 C CNN
+F 2 "Connector_PinHeader_2.54mm:PinHeader_2x03_P2.54mm_Vertical" H 7950 2800 50  0001 C CNN
+F 3 "~" H 7950 2800 50  0001 C CNN
+	1    7950 2800
+	1    0    0    -1
+$EndComp
+Wire Wire Line
+	7750 2700 7600 2700
+Wire Wire Line
+	7600 2900 7750 2900
+Wire Wire Line
+	8450 2700 8250 2700
+Text GLabel 4650 1400 3    50   Input ~ 0
+MCU-D0
+Text Notes 4700 2050 1    50   ~ 0
+Spare
+NoConn ~ 7750 2800
+NoConn ~ 8250 2800
+NoConn ~ 8250 2900
 $EndSCHEMATC
