File: KiCad Files/DP1600i/file637007D4.sch (KiCad schematic (older format))
At the start: 12 parts, among them U3 LM2940T-5.0

Commit message: Add files via upload
Parts:
- added J9: Conn_01x01, Connector_PinHeader_2.54mm:PinHeader_1x01_P2.54mm_Vertical, symbol Connector_Generic:Conn_01x01
Connections:
- net 12V-SW: now also J9.1 (Pin_1)
Other:
- note added: "12 volt test point header socket"
Changed lines of the file:
@@
 Connection ~ 5050 1800
 Wire Wire Line
-	5050 1800 5050 2200
+	5050 1800 5050 2000
 Wire Wire Line
 	6350 3100 6350 3350
@@
 Wire Wire Line
 	7800 1750 7800 2150
+$Comp
+L Connector_Generic:Conn_01x01 J9
+U 1 1 63756211
+P 4350 2000
+F 0 "J9" H 4268 2217 50  0000 C CNN
+F 1 "Conn_01x01" H 4268 2126 50  0000 C CNN
+F 2 "Connector_PinHeader_2.54mm:PinHeader_1x01_P2.54mm_Vertical" H 4350 2000 50  0001 C CNN
+F 3 "~" H 4350 2000 50  0001 C CNN
+	1    4350 2000
+	-1   0    0    -1
+$EndComp
+Wire Wire Line
+	4550 2000 5050 2000
+Connection ~ 5050 2000
+Wire Wire Line
+	5050 2000 5050 2200
+Text Notes 2950 2050 0    50   ~ 0
+12 volt test point header socket
 $EndSCHEMATC
