File: KiCad Files/DP1600i/file637007D4.sch (KiCad schematic (older format))
At the start: 13 parts, among them J2 Conn_01x01, U3 LM2940T-5.0

Commit message: Add files via upload
Parts:
- J2: value Conn_01x01 -> 12V Test; footprint Connector_PinHeader_2.54mm:PinHeader_1x01_P2.54mm_Vertical -> DP1600i:Jumper-Pad
Changed lines of the file:
@@
 P 4350 2000
 F 0 "J2" H 4268 2217 50  0000 C CNN
-F 1 "Conn_01x01" H 4268 2126 50  0000 C CNN
-F 2 "Connector_PinHeader_2.54mm:PinHeader_1x01_P2.54mm_Vertical" H 4350 2000 50  0001 C CNN
+F 1 "12V Test" H 4268 2126 50  0000 C CNN
+F 2 "DP1600i:Jumper-Pad" H 4350 2000 50  0001 C CNN
 F 3 "~" H 4350 2000 50  0001 C CNN
 	1    4350 2000

Commit message: Add files via upload
Parts:
- removed D13: TP6KE47A, Diode_THT:D_DO-15_P12.70mm_Horizontal, symbol Device:D_Zener
- removed D14: SB230TA, Diode_THT:D_DO-15_P12.70mm_Horizontal, symbol Device:D_Schottky
- added D13: 1N5818, Diode_THT:D_DO-41_SOD81_P10.16mm_Horizontal, symbol Device:D
- added JP2: SolderJumper_2_Open, Jumper:SolderJumper-2_P1.3mm_Open_RoundedPad1.0x1.5mm, symbol Jumper:SolderJumper_2_Open
- added RV1: ERZ-V14D220, Varistor:RV_Disc_D15.5mm_W4.7mm_P7.5mm, symbol Device:Varistor
- F1: value 0ZRP0050FF1E -> MF-R050; footprint Fuse:Fuse_BelFuse_0ZRE0055FF_L14.0mm_W4.1mm -> Fuse:Fuse_BelFuse_0ZRE0100FF_L18.7mm_W5.1mm
Connections:
- net 12V: now also C18.1, C19.1, U3.1 (VI), D13.1 (K)
- net GND: now also JP2.2 (B), RV1.2
- new net 12V-Raw: D13.2 (A), RV1.1
- new net SigRtn: JP2.1 (A)
Other:
- note added: "10V"
- note added: "35V"
- note added: "50V"
- moved on the sheet: J2
Changed lines of the file:
@@
-$EndComp
-Wire Wire Line
-	4500 2700 5050 2700
-Wire Wire Line
-	5050 2700 5500 2700
-Connection ~ 5050 2700
-$Comp
-L Device:D_Schottky D14
-U 1 1 5CD266C1
-P 5050 2350
-F 0 "D14" H 5050 2250 50  0000 C CNN
-F 1 "SB230TA" H 5050 2500 50  0000 C CNN
-F 2 "Diode_THT:D_DO-15_P12.70mm_Horizontal" H 5050 2350 50  0001 C CNN
-F 3 "https://www.mouser.com/datasheet/2/115/ds13002-60388.pdf" H 5050 2350 50  0001 C CNN
-F 4 "1655-1518-1-ND" H -650 -100 50  0001 C CNN "Digikey Part Number"
-F 5 "SMC" H -650 -100 50  0001 C CNN "Manufacturer_Name"
-F 6 "SB230TA" H -650 -100 50  0001 C CNN "Manufacturer_Part_Number"
-F 7 "https://www.digikey.com.au/product-detail/en/smc-diode-solutions/SB230TA/1655-1518-1-ND/6022963" H -650 -100 50  0001 C CNN "URL"
-	1    5050 2350
-	0    -1   -1   0
 $EndComp
 Wire Wire Line
 	5500 2700 5500 2450
-Connection ~ 5500 2700
 $Comp
 L Device:C C21
@@
 Text Notes 5900 1950 0    89   ~ 0
 Power Regulator
-Text GLabel 5050 1350 0    50   Input ~ 0
+Text GLabel 5050 1600 1    50   Input ~ 0
 12V
 Text Notes 5650 4050 0    89   ~ 0
@@
 P 7800 2300
 F 0 "F1" H 7888 2346 50  0000 L CNN
-F 1 "0ZRP0050FF1E" H 7888 2255 50  0000 L CNN
-F 2 "Fuse:Fuse_BelFuse_0ZRE0055FF_L14.0mm_W4.1mm" H 7850 2100 50  0001 L CNN
+F 1 "MF-R050" H 7888 2255 50  0000 L CNN
+F 2 "Fuse:Fuse_BelFuse_0ZRE0100FF_L18.7mm_W5.1mm" H 7850 2100 50  0001 L CNN
 F 3 "~" H 7800 2300 50  0001 C CNN
 F 4 "507-2403-ND" H 700 0   50  0001 C CNN "Digikey Part Number"
@@
 	1    0    0    -1
 $EndComp
-Wire Wire Line
-	5050 2500 5050 2700
-$Comp
-L Device:D_Zener D13
-U 1 1 60723E7D
-P 4500 2900
-F 0 "D13" H 4400 3000 50  0000 L CNN
-F 1 "TP6KE47A" H 4350 2750 50  0000 L CNN
-F 2 "Diode_THT:D_DO-15_P12.70mm_Horizontal" H 4500 2900 50  0001 C CNN
-F 3 "" H 4500 2900 50  0001 C CNN
-F 4 "F6853CT-ND" H 4500 2900 50  0001 C CNN "Digikey Part Number"
-F 5 "Littelfuse" H 4500 2900 50  0001 C CNN "Manufacturer_Name"
-F 6 "TP6KE47A" H 4500 2900 50  0001 C CNN "Manufacturer_Part_Number"
-	1    4500 2900
-	0    1    1    0
-$EndComp
-Wire Wire Line
-	4500 2700 4500 2750
 Wire Wire Line
 	4500 3100 4500 3050
@@
 	6200 5250 6350 5250
 Wire Wire Line
-	5500 2450 5750 2450
-Wire Wire Line
 	6350 3100 7600 3100
 Connection ~ 7800 2450
@@
 $EndComp
 Wire Wire Line
-	5050 1350 5050 1800
-Wire Wire Line
 	6650 2450 7200 2450
 Connection ~ 7200 2450
@@
 	0    1    1    0
 $EndComp
-Connection ~ 5050 1800
-Wire Wire Line
-	5050 1800 5050 2000
-Wire Wire Line
-	6350 3100 6350 3350
+Wire Wire Line
+	6350 3100 6350 3250
 $Comp
 L power:PWR_FLAG #FLG02
@@
 Wire Wire Line
 	6350 3350 6350 3500
-Text Notes 2800 1400 0    50   ~ 0
+Text Notes 1600 2500 0    50   ~ 0
 12 volt output from Main Relay in Aux board
-$Comp
-L power:PWR_FLAG #FLG0101
-U 1 1 6372DF73
-P 5750 2350
-F 0 "#FLG0101" H 5750 2425 50  0001 C CNN
-F 1 "PWR_FLAG" V 5750 2478 50  0000 L CNN
-F 2 "" H 5750 2350 50  0001 C CNN
-F 3 "~" H 5750 2350 50  0001 C CNN
-	1    5750 2350
-	1    0    0    -1
-$EndComp
-Wire Wire Line
-	5750 2350 5750 2450
-Connection ~ 5750 2450
-Wire Wire Line
-	5750 2450 6050 2450
 Wire Wire Line
 	7200 1500 7200 2450
@@
 Wire Wire Line
 	7800 1750 7800 2150
+Text Notes 8100 3000 0    50   ~ 0
+10V
+Text Notes 7350 3000 0    50   ~ 0
+50V
+Text Notes 5200 3000 0    50   ~ 0
+35V
+$Comp
+L Device:D D13
+U 1 1 637EC140
+P 4700 2450
+F 0 "D13" H 4700 2233 50  0000 C CNN
+F 1 "1N5818" H 4700 2324 50  0000 C CNN
+F 2 "Diode_THT:D_DO-41_SOD81_P10.16mm_Horizontal" H 4700 2450 50  0001 C CNN
+F 3 "~" H 4700 2450 50  0001 C CNN
+	1    4700 2450
+	-1   0    0    1
+$EndComp
+$Comp
+L Device:Varistor RV1
+U 1 1 637EE630
+P 4500 2900
+F 0 "RV1" V 4600 2850 50  0000 L CNN
+F 1 "ERZ-V14D220" V 4350 2650 50  0000 L CNN
+F 2 "Varistor:RV_Disc_D15.5mm_W4.7mm_P7.5mm" V 4430 2900 50  0001 C CNN
+F 3 "~" H 4500 2900 50  0001 C CNN
+	1    4500 2900
+	1    0    0    -1
+$EndComp
+Text GLabel 3800 2450 0    50   Input ~ 0
+12V-Raw
+Wire Wire Line
+	3800 2450 4500 2450
+Wire Wire Line
+	4850 2450 5050 2450
+Connection ~ 5500 2450
+Wire Wire Line
+	5050 1800 5050 2000
+Connection ~ 5050 2450
+Wire Wire Line
+	5050 2450 5500 2450
+Wire Wire Line
+	5050 2450 5050 2700
+Wire Wire Line
+	4500 2750 4500 2450
+Connection ~ 4500 2450
+Wire Wire Line
+	4500 2450 4550 2450
+Wire Wire Line
+	4800 2000 5050 2000
+Connection ~ 5050 2000
+Wire Wire Line
+	5050 2000 5050 2450
+Wire Wire Line
+	5050 1800 5050 1600
+Connection ~ 5050 1800
+Text GLabel 5050 3250 0    50   Input ~ 0
+SigRtn
+Wire Wire Line
+	6150 3250 6350 3250
+Connection ~ 6350 3250
+Wire Wire Line
+	6350 3250 6350 3350
+$Comp
+L power:VDDA #PWR0106
+U 1 1 63801F19
+P 1650 -250
+F 0 "#PWR0106" H 1650 -400 50  0001 C CNN
+F 1 "VDDA" V 1650 -100 50  0000 L CNN
+F 2 "" H 1650 -250 50  0001 C CNN
+F 3 "" H 1650 -250 50  0001 C CNN
+	1    1650 -250
+	1    0    0    -1
+$EndComp
+Wire Wire Line
+	5500 2450 6050 2450
+Text Notes 3200 2050 0    50   ~ 0
+12 volt test point header socket
 $Comp
 L Connector_Generic:Conn_01x01 J2
 U 1 1 63756211
-P 4350 2000
-F 0 "J2" H 4268 2217 50  0000 C CNN
-F 1 "12V Test" H 4268 2126 50  0000 C CNN
-F 2 "DP1600i:Jumper-Pad" H 4350 2000 50  0001 C CNN
-F 3 "~" H 4350 2000 50  0001 C CNN
-	1    4350 2000
+P 4600 2000
+F 0 "J2" H 4518 2217 50  0000 C CNN
+F 1 "12V Test" H 4518 2126 50  0000 C CNN
+F 2 "DP1600i:Jumper-Pad" H 4600 2000 50  0001 C CNN
+F 3 "~" H 4600 2000 50  0001 C CNN
+	1    4600 2000
 	-1   0    0    -1
 $EndComp
-Wire Wire Line
-	4550 2000 5050 2000
-Connection ~ 5050 2000
-Wire Wire Line
-	5050 2000 5050 2200
-Text Notes 2950 2050 0    50   ~ 0
-12 volt test point header socket
+$Comp
+L Jumper:SolderJumper_2_Open JP2
+U 1 1 637F187B
+P 6000 3250
+F 0 "JP2" H 6000 3350 50  0000 C CNN
+F 1 "SolderJumper_2_Open" H 5900 3100 50  0000 C CNN
+F 2 "Jumper:SolderJumper-2_P1.3mm_Open_RoundedPad1.0x1.5mm" H 6000 3250 50  0001 C CNN
+F 3 "~" H 6000 3250 50  0001 C CNN
+	1    6000 3250
+	1    0    0    -1
+$EndComp
+$Comp
+L power:PWR_FLAG #FLG0101
+U 1 1 6380F403
+P 5250 3350
+F 0 "#FLG0101" H 5250 3425 50  0001 C CNN
+F 1 "PWR_FLAG" V 5250 3478 50  0000 L CNN
+F 2 "" H 5250 3350 50  0001 C CNN
+F 3 "~" H 5250 3350 50  0001 C CNN
+	1    5250 3350
+	-1   0    0    1
+$EndComp
+Wire Wire Line
+	5050 3250 5250 3250
+Wire Wire Line
+	5250 3350 5250 3250
+Connection ~ 5250 3250
+Wire Wire Line
+	5250 3250 5850 3250
 $EndSCHEMATC

Commit message: Add files via upload
Other:
- note added: "5 Volt Power Regulator"
- note removed: "Power Regulator"
- moved on the sheet: C20, JP1, R12, R13
Changed lines of the file:
@@
 	7600 3000 7600 3100
 Connection ~ 7600 3100
-Text Notes 5900 1950 0    89   ~ 0
-Power Regulator
+Text Notes 5550 1100 0    89   ~ 0
+5 Volt Power Regulator
 Text GLabel 5050 1600 1    50   Input ~ 0
 12V
-Text Notes 5650 4050 0    89   ~ 0
+Text Notes 2950 4550 0    89   ~ 0
 Reset Protection
-Text Notes 5500 4200 0    58   ~ 0
+Text Notes 2800 4700 0    58   ~ 0
 Refer AVR040 Application Note
 $Comp
 L Device:C C20
 U 1 1 5CF0AAD4
-P 5700 4950
-F 0 "C20" V 5650 4700 50  0000 L CNN
-F 1 "22uF" V 5750 4700 50  0000 L CNN
-F 2 "Capacitor_THT:C_Disc_D7.5mm_W5.0mm_P5.00mm" H 5738 4800 50  0001 C CNN
-F 3 "~" H 5700 4950 50  0001 C CNN
-F 4 "445-180603-1-ND" H 0   0   50  0001 C CNN "Digikey Part Number"
-F 5 "TDK" H 0   0   50  0001 C CNN "Manufacturer_Name"
-F 6 "FA22X7R1E226MRU06" H 0   0   50  0001 C CNN "Manufacturer_Part_Number"
-F 7 "" H 0   0   50  0001 C CNN "URL"
-	1    5700 4950
+P 3000 5450
+F 0 "C20" V 2950 5200 50  0000 L CNN
+F 1 "22uF" V 3050 5200 50  0000 L CNN
+F 2 "Capacitor_THT:C_Disc_D7.5mm_W5.0mm_P5.00mm" H 3038 5300 50  0001 C CNN
+F 3 "~" H 3000 5450 50  0001 C CNN
+F 4 "445-180603-1-ND" H -2700 500 50  0001 C CNN "Digikey Part Number"
+F 5 "TDK" H -2700 500 50  0001 C CNN "Manufacturer_Name"
+F 6 "FA22X7R1E226MRU06" H -2700 500 50  0001 C CNN "Manufacturer_Part_Number"
+F 7 "" H -2700 500 50  0001 C CNN "URL"
+	1    3000 5450
 	0    1    1    0
 $EndComp
@@
 L Device:R R13
 U 1 1 5CF13C09
-P 5950 4700
-F 0 "R13" V 6050 4650 50  0000 L CNN
-F 1 "120R" V 5850 4600 50  0000 L CNN
-F 2 "Resistor_THT:R_Axial_DIN0207_L6.3mm_D2.5mm_P7.62mm_Horizontal" V 5880 4700 50  0001 C CNN
-F 3 "~" H 5950 4700 50  0001 C CNN
-F 4 "BC3453CT-ND" H 0   0   50  0001 C CNN "Digikey Part Number"
-F 5 "Vishay" H 0   0   50  0001 C CNN "Manufacturer_Name"
-F 6 "MBA02040C1200FC100" H 0   0   50  0001 C CNN "Manufacturer_Part_Number"
-F 7 "" H 0   0   50  0001 C CNN "URL"
-	1    5950 4700
+P 3250 5200
+F 0 "R13" V 3350 5150 50  0000 L CNN
+F 1 "120R" V 3150 5100 50  0000 L CNN
+F 2 "Resistor_THT:R_Axial_DIN0207_L6.3mm_D2.5mm_P7.62mm_Horizontal" V 3180 5200 50  0001 C CNN
+F 3 "~" H 3250 5200 50  0001 C CNN
+F 4 "BC3453CT-ND" H -2700 500 50  0001 C CNN "Digikey Part Number"
+F 5 "Vishay" H -2700 500 50  0001 C CNN "Manufacturer_Name"
+F 6 "MBA02040C1200FC100" H -2700 500 50  0001 C CNN "Manufacturer_Part_Number"
+F 7 "" H -2700 500 50  0001 C CNN "URL"
+	1    3250 5200
 	-1   0    0    1
 $EndComp
@@
 L power:VDD #PWR033
 U 1 1 5CF1825D
-P 6150 4550
-F 0 "#PWR033" H 6150 4400 50  0001 C CNN
-F 1 "VDD" H 6167 4723 50  0000 C CNN
-F 2 "" H 6150 4550 50  0001 C CNN
-F 3 "" H 6150 4550 50  0001 C CNN
-	1    6150 4550
+P 3450 5050
+F 0 "#PWR033" H 3450 4900 50  0001 C CNN
+F 1 "VDD" H 3467 5223 50  0000 C CNN
+F 2 "" H 3450 5050 50  0001 C CNN
+F 3 "" H 3450 5050 50  0001 C CNN
+	1    3450 5050
 	1    0    0    -1
 $EndComp
@@
 L power:GND #PWR031
 U 1 1 5CF1EB2F
-P 5450 4950
-F 0 "#PWR031" H 5450 4700 50  0001 C CNN
-F 1 "GND" V 5455 4822 50  0000 R CNN
-F 2 "" H 5450 4950 50  0001 C CNN
-F 3 "" H 5450 4950 50  0001 C CNN
-	1    5450 4950
+P 2750 5450
+F 0 "#PWR031" H 2750 5200 50  0001 C CNN
+F 1 "GND" V 2755 5322 50  0000 R CNN
+F 2 "" H 2750 5450 50  0001 C CNN
+F 3 "" H 2750 5450 50  0001 C CNN
+	1    2750 5450
 	0    1    1    0
 $EndComp
 Wire Wire Line
-	5450 4950 5550 4950
+	2750 5450 2850 5450
 Wire Wire Line
-	5950 5050 5950 4950
+	3250 5550 3250 5450
 Wire Wire Line
-	5850 4950 5950 4950
-Connection ~ 5950 4950
+	3150 5450 3250 5450
+Connection ~ 3250 5450
 Wire Wire Line
-	5950 4950 5950 4850
+	3250 5450 3250 5350
 Wire Wire Line
-	5950 4550 6150 4550
-Text GLabel 6350 5250 2    50   Input ~ 0
+	3250 5050 3450 5050
+Text GLabel 3650 5750 2    50   Input ~ 0
 RESET
 Wire Wire Line
-	5950 5050 6000 5050
+	3250 5550 3300 5550
 $Comp
 L Device:R R12
 U 1 1 5CE55978
-P 5750 5250
-F 0 "R12" V 5650 5150 50  0000 L CNN
-F 1 "10k" V 5850 5150 50  0000 L CNN
-F 2 "Resistor_THT:R_Axial_DIN0207_L6.3mm_D2.5mm_P7.62mm_Horizontal" V 5680 5250 50  0001 C CNN
-F 3 "~" H 5750 5250 50  0001 C CNN
-F 4 "BC10.0KXCT-ND" H 0   0   50  0001 C CNN "Digikey Part Number"
-F 5 "Vishay" H 0   0   50  0001 C CNN "Manufacturer_Name"
-F 6 "MBA02040C1002FRP00" H 0   0   50  0001 C CNN "Manufacturer_Part_Number"
-F 7 "https://www.digikey.com.au/product-detail/en/vishay-beyschlag-draloric-bc-components/MBA02040C1002FRP00/BC10-0KXCT-ND/336866" H 0   0   50  0001 C CNN "URL"
-	1    5750 5250
+P 3050 5750
+F 0 "R12" V 2950 5650 50  0000 L CNN
+F 1 "10k" V 3150 5650 50  0000 L CNN
+F 2 "Resistor_THT:R_Axial_DIN0207_L6.3mm_D2.5mm_P7.62mm_Horizontal" V 2980 5750 50  0001 C CNN
+F 3 "~" H 3050 5750 50  0001 C CNN
+F 4 "BC10.0KXCT-ND" H -2700 500 50  0001 C CNN "Digikey Part Number"
+F 5 "Vishay" H -2700 500 50  0001 C CNN "Manufacturer_Name"
+F 6 "MBA02040C1002FRP00" H -2700 500 50  0001 C CNN "Manufacturer_Part_Number"
+F 7 "https://www.digikey.com.au/product-detail/en/vishay-beyschlag-draloric-bc-components/MBA02040C1002FRP00/BC10-0KXCT-ND/336866" H -2700 500 50  0001 C CNN "URL"
+	1    3050 5750
 	0    1    1    0
 $EndComp
 Wire Wire Line
-	5900 5250 6200 5250
+	3200 5750 3500 5750
 $Comp
 L power:VDD #PWR032
 U 1 1 5CE5E61D
-P 5500 5250
-F 0 "#PWR032" H 5500 5100 50  0001 C CNN
-F 1 "VDD" H 5517 5423 50  0000 C CNN
-F 2 "" H 5500 5250 50  0001 C CNN
-F 3 "" H 5500 5250 50  0001 C CNN
-	1    5500 5250
+P 2800 5750
+F 0 "#PWR032" H 2800 5600 50  0001 C CNN
+F 1 "VDD" H 2817 5923 50  0000 C CNN
+F 2 "" H 2800 5750 50  0001 C CNN
+F 3 "" H 2800 5750 50  0001 C CNN
+	1    2800 5750
 	0    -1   -1   0
 $EndComp
 Wire Wire Line
-	5500 5250 5600 5250
+	2800 5750 2900 5750
 $Comp
 L Regulator_Linear:LM2937xS U3
@@
 L Device:Jumper_NO_Small JP1
 U 1 1 60E353E8
-P 6100 5050
-F 0 "JP1" H 6100 5143 50  0000 C CNN
-F 1 "Jumper_NO_Small" H 6100 5144 50  0001 C CNN
-F 2 "Connector_PinHeader_2.54mm:PinHeader_1x02_P2.54mm_Vertical" H 6100 5050 50  0001 C CNN
-F 3 "~" H 6100 5050 50  0001 C CNN
-	1    6100 5050
+P 3400 5550
+F 0 "JP1" H 3400 5643 50  0000 C CNN
+F 1 "Jumper_NO_Small" H 3400 5644 50  0001 C CNN
+F 2 "Connector_PinHeader_2.54mm:PinHeader_1x02_P2.54mm_Vertical" H 3400 5550 50  0001 C CNN
+F 3 "~" H 3400 5550 50  0001 C CNN
+	1    3400 5550
 	1    0    0    -1
 $EndComp
 Wire Wire Line
-	6200 5050 6200 5250
-Connection ~ 6200 5250
+	3500 5550 3500 5750
+Connection ~ 3500 5750
 Wire Wire Line
-	6200 5250 6350 5250
+	3500 5750 3650 5750
 Wire Wire Line
 	6350 3100 7600 3100

Commit message: Add files via upload
Other:
- note added: "Note! SigRtn connects to ground at this point only."
Changed lines of the file:
@@
 $Descr A4 11693 8268
 encoding utf-8
-Sheet 3 6
+Sheet 3 5
 Title "DP1600i"
 Date "2022-11-11"
@@
 Wire Wire Line
 	5250 3250 5850 3250
+Text Notes 3000 3450 0    50   ~ 0
+Note! SigRtn connects to ground at this point only.
 $EndSCHEMATC
