File: KiCad Files/DP1600i/DP1600i.kicad_pcb (KiCad board)
At the start: 2 copper layers, 120.4 x 100.1 mm, 116 parts, among them J1 DB25_Female, J10 D8, J2 Conn_01x01, J23 D18, J24 D19, J27 5V, J28 5V, J4 Gnd, J5 D13, J55 D48, J56 D49, J57 D50, J58 D51, J59 D52, J6 D12, J60 D53, J61 Gnd, J62 Gnd, J65 RESET, J67 5V, J68 Gnd, J69 Gnd, J7 D11, J71 A0, J72 A1, J73 A2, J74 A3, J75 A4, J76 A5, J77 A6, J78 A7, J8 D10, J9 D9, U1 MPXH6115_Adapter, U2 MPXH6115_Adapter, U3 LM2940T-5.0, U4 IXDI604PI, U5 IXDI604PI, U6 IXDI604PI, U7 IXDI604PI, U8 IXDI604PI, U9 ULN2003

Commit message: Add files via upload
Parts:
- removed C3, C4: 1uF, Capacitor_THT:C_Disc_D5.0mm_W2.5mm_P2.50mm
- C1, C2: value 0.01uF -> 0.1uF
- C10, C9: value 470pf -> 47pf
- R5, R6: value 470R -> 51K
- U1, U2: value MPXH6115_Adapter -> MPXH6115_Adapter_Vertical; footprint MPXH61115AC6U Adapter:MPXH6115_Adapter -> MPXH61115AC6U Adapter:MPXH6115_Adapter_Vertical
- U9: value ULN2003 -> ULN2004AN; footprint Package_DIP:DIP-10_W7.62mm -> Package_DIP:DIP-16_W7.62mm
- moved U8 274.3 mm to (93.5, 59.7), turned to 90 degrees
- moved R24 272.6 mm to (94.0, 49.5)
- moved C30 267.5 mm to (101.1, 43.4), turned to 180 degrees
- moved R23 264.5 mm to (101.6, 46.5), turned to 180 degrees
- moved U6 218.5 mm to (105.5, 59.6), turned to 90 degrees
- moved R21 216.8 mm to (106.0, 49.4)
- moved C28 211.9 mm to (113.2, 43.4), turned to 180 degrees
- moved R19 208.7 mm to (113.6, 46.4), turned to 180 degrees
- moved U5 169.2 mm to (134.0, 59.8), turned to 90 degrees
- moved R18 165.6 mm to (134.5, 49.6)
- moved U4 164.3 mm to (117.3, 59.8), turned to 90 degrees
- moved C27 161.0 mm to (141.7, 43.6), turned to 180 degrees
- moved R17 160.5 mm to (117.7, 49.6)
- moved R16 158.1 mm to (142.1, 46.6), turned to 180 degrees
- moved C26 155.4 mm to (124.9, 43.6), turned to 180 degrees
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
Commit message: Add files via upload
Parts:
- removed J10: D8, Connector_PinHeader_2.54mm:PinHeader_1x01_P2.54mm_Vertical
- removed J23: D18, Connector_PinHeader_2.54mm:PinHeader_1x01_P2.54mm_Vertical
- removed J24: D19, Connector_PinHeader_2.54mm:PinHeader_1x01_P2.54mm_Vertical
- removed J27, J28, J67: 5V, Connector_PinHeader_2.54mm:PinHeader_1x01_P2.54mm_Vertical
- removed J55: D48, Connector_PinHeader_2.54mm:PinHeader_1x01_P2.54mm_Vertical
- removed J56: D49, Connector_PinHeader_2.54mm:PinHeader_1x01_P2.54mm_Vertical
- removed J57: D50, Connector_PinHeader_2.54mm:PinHeader_1x01_P2.54mm_Vertical
- removed J58: D51, Connector_PinHeader_2.54mm:PinHeader_1x01_P2.54mm_Vertical
- removed J59: D52, Connector_PinHeader_2.54mm:PinHeader_1x01_P2.54mm_Vertical
- removed J60: D53, Connector_PinHeader_2.54mm:PinHeader_1x01_P2.54mm_Vertical
- removed J61, J62, J68, J69: Gnd, Connector_PinHeader_2.54mm:PinHeader_1x01_P2.54mm_Vertical
- removed J65: RESET, Connector_PinHeader_2.54mm:PinHeader_1x01_P2.54mm_Vertical
- removed J71: A0, Connector_PinHeader_2.54mm:PinHeader_1x01_P2.54mm_Vertical
- removed J72: A1, Connector_PinHeader_2.54mm:PinHeader_1x01_P2.54mm_Vertical
- removed J73: A2, Connector_PinHeader_2.54mm:PinHeader_1x01_P2.54mm_Vertical
- removed J74: A3, Connector_PinHeader_2.54mm:PinHeader_1x01_P2.54mm_Vertical
- removed J75: A4, Connector_PinHeader_2.54mm:PinHeader_1x01_P2.54mm_Vertical
- removed J76: A5, Connector_PinHeader_2.54mm:PinHeader_1x01_P2.54mm_Vertical
- removed J77: A6, Connector_PinHeader_2.54mm:PinHeader_1x01_P2.54mm_Vertical
- removed J78: A7, Connector_PinHeader_2.54mm:PinHeader_1x01_P2.54mm_Vertical
- added J3: Conn_01x07, Connector_PinHeader_2.54mm:PinHeader_1x07_P2.54mm_Vertical, F.Cu at (115.0, 63.7)
- added J87: Pin D4, DP1600i:Jumper-Pad, F.Cu at (142.0, 67.5)
- added J88: Pin D3, DP1600i:Jumper-Pad, F.Cu at (144.5, 67.5)
- added J89: Pin D2, DP1600i:Jumper-Pad, F.Cu at (147.1, 67.5)
- added J90: Pin D1, DP1600i:Jumper-Pad, F.Cu at (149.5, 67.5)
- added J91: Pin D0, DP1600i:Jumper-Pad, F.Cu at (152.1, 67.4)
- added J92: D7 out, DP1600i:Jumper-Pad, F.Cu at (133.0, 77.5)
- added J93: D6 out, DP1600i:Jumper-Pad, F.Cu at (130.5, 77.5)
- added J94: D5 out, DP1600i:Jumper-Pad, F.Cu at (128.0, 77.5)
- added J95: Step 2B, DP1600i:Jumper-Pad, F.Cu at (174.5, 83.7)
- added J96: Step 2A, DP1600i:Jumper-Pad, F.Cu at (171.9, 83.8)
- added J97: Step 1A, DP1600i:Jumper-Pad, F.Cu at (169.4, 83.8)
- added J98: Step 1B, DP1600i:Jumper-Pad, F.Cu at (166.9, 83.8)
- added U10: A4988StepStick, BPEM488CWaux:A4988StepStick, F.Cu at (179.5, 67.9)
- J1: value DB25_Female -> DB25_Male; footprint Connector_Dsub:DSUB-25_Female_Horizontal_P2.77x2.84mm_EdgePinOffset4.94mm_Housed_MountingHolesOffset7.48mm -> Connector_Dsub:DSUB-25_Male_Horizontal_P2.77x2.84mm_EdgePinOffset4.94mm_Housed_MountingHolesOffset7.48mm
- J2: value Conn_01x01 -> 12V Test; footprint Connector_PinHeader_2.54mm:PinHeader_1x01_P2.54mm_Vertical -> DP1600i:Jumper-Pad
- J4: value Gnd -> Conn_01x08; footprint Connector_PinHeader_2.54mm:PinHeader_1x01_P2.54mm_Vertical -> Connector_PinHeader_2.54mm:PinHeader_1x08_P2.54mm_Vertical
- J5: value D13 -> Conn_01x04; footprint Connector_PinHeader_2.54mm:PinHeader_1x01_P2.54mm_Vertical -> Connector_PinHeader_2.54mm:PinHeader_1x04_P2.54mm_Vertical
- J6: value D12 -> Conn_01x02; footprint Connector_PinHeader_2.54mm:PinHeader_1x01_P2.54mm_Vertical -> Connector_PinHeader_2.54mm:PinHeader_1x02_P2.54mm_Vertical
- J7: value D11 -> Conn_02x04; footprint Connector_PinHeader_2.54mm:PinHeader_1x01_P2.54mm_Vertical -> Connector_PinHeader_2.54mm:PinHeader_2x04_P2.54mm_Vertical
- J8: value D10 -> Conn_01x05; footprint Connector_PinHeader_2.54mm:PinHeader_1x01_P2.54mm_Vertical -> Connector_PinHeader_2.54mm:PinHeader_1x05_P2.54mm_Vertical
- J9: value D9 -> Conn_01x08; footprint Connector_PinHeader_2.54mm:PinHeader_1x01_P2.54mm_Vertical -> Connector_PinHeader_2.54mm:PinHeader_1x08_P2.54mm_Vertical
- JP1: value Jumper_NO_Small -> Reset Prot
- U1, U2: value MPXH6115_Adapter_Vertical -> MPXH6115
- moved C29 161.9 mm to (145.4, 97.2), turned to 270 degrees
- moved R20 155.8 mm to (148.4, 96.7), turned to 270 degrees
- moved R22 153.1 mm to (151.4, 104.3), turned to 90 degrees
- moved C17 143.1 mm to (188.2, 69.0), turned to 180 degrees
- moved D17 141.6 mm to (188.1, 71.9), turned to 270 degrees
- moved C25 136.7 mm to (195.6, 68.6), turned to 180 degrees
- moved D11 134.9 mm to (195.5, 71.5), turned to 270 degrees
- moved U7 133.7 mm to (161.6, 104.8), turned to 180 degrees
- moved D18 133.6 mm to (184.8, 82.1), turned to 90 degrees
- moved D12 125.4 mm to (192.2, 81.7), turned to 90 degrees
- moved U2 81.0 mm to (95.9, 97.6), turned to 180 degrees
- moved C27 73.7 mm to (166.7, 112.9), turned to 0 degrees
- moved J7 69.7 mm to (182.6, 99.3)
- moved R18 69.5 mm to (173.9, 106.9), turned to 180 degrees
- moved R16 67.8 mm to (166.2, 109.9), turned to 0 degrees
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Connections:
- C10 pad 1: MCU-A5 -> MCU-A0
- C14 pad 1: ADC-Clamp-2 -> ADC-Clamp-5
- C15 pad 1: ADC-Clamp-0 -> ADC-Clamp-3
- C16 pad 1: ADC-Clamp-1 -> ADC-Clamp-4
- C8 pad 1: ADC-Clamp-4 -> ADC-Clamp-2
- C9 pad 1: MCU-A3 -> MCU-A1
- D1 pad 1: ADC-Clamp-0 -> ADC-Clamp-3
- D2 pad 2: ADC-Clamp-0 -> ADC-Clamp-3
- D3 pad 1: ADC-Clamp-1 -> ADC-Clamp-5
- D4 pad 2: ADC-Clamp-1 -> ADC-Clamp-5
- J1 pad 1: IAT_Sensor -> Spare-ADC
- J1 pad 14: CLT_Sensor -> O2_Sensor
- J1 pad 15: TPS_Sensor -> CLT_Sensor
- J1 pad 2: O2_Sensor -> TPS_Sensor
- J1 pad 3: Spare-ADC -> IAT_Sensor
- J4 pad 1: SigRtn -> MCU-D7
- J5 pad 1: MCU-D13 -> MCU-D16
- J6 pad 1: MCU-D12 -> VDD
- J7 pad 1: MCU-D11 -> MCU-D48
- J8 pad 1: MCU-D10 -> RESET
- J9 pad 1: MCU-D9 -> MCU-A0
- R10 pad 1: ADC-Clamp-0 -> ADC-Clamp-3
- R11 pad 1: ADC-Clamp-1 -> ADC-Clamp-4
- R4 pad 1: ADC-Clamp-4 -> ADC-Clamp-2
- R5 pad 1: MCU-A3 -> MCU-A1
- R6 pad 1: MCU-A5 -> MCU-A0
- R9 pad 1: ADC-Clamp-2 -> ADC-Clamp-5
- U9 pad 3: Net-(U9-Pad3) -> MCU-D7
- U9 pad 4: Net-(U9-Pad4) -> MCU-D6
- U9 pad 5: Net-(U9-Pad5) -> MCU-D5
Other:
- board text added: "48"
- board text added: "49"
- board text added: "50"
- board text added: "51"
- board text added: "52"
- board text added: "53"
- board text added: "54"
- board text added: "55"
- board text added: "A0"
- board text added: "A1"
- board text added: "A2"
- board text added: "A3"
- board text added: "A4"
- board text added: "A5"
- board text added: "A6"
- board text added: "A7"
- board text added: "Baro"
- board text added: "Bat"
- board text added: "CLT"
- board text added: "Gnd"
- board text added: "IAT"
- board text added: "MAP"
- board text added: "N/C"
- board text added: "O2"
- board text added: "Reset"
- board text added: "Spare"
- board text added: "TPS"
- board text added: "VDDA"

Commit message: Add files via upload
Parts:
- removed D14: SB230TA, Diode_THT:D_DO-15_P12.70mm_Horizontal
- added ?: , , F.Cu at (108.8, 53.8)
- added ?: , , F.Cu at (106.6, 52.1)
- added ?: , , F.Cu at (142.0, 70.1)
- added J10: Conn_01x01, DP1600i:Jumper-Pad, F.Cu at (195.4, 99.3)
- added J11: Conn_01x05, Connector_PinHeader_2.54mm:PinHeader_1x05_P2.54mm_Vertical, F.Cu at (99.4, 48.3)
- added J12: Conn_01x05, Connector_PinHeader_2.54mm:PinHeader_1x05_P2.54mm_Vertical, F.Cu at (99.4, 63.5)
- added J13: Conn_01x05, Connector_PinHeader_2.54mm:PinHeader_1x05_P2.54mm_Vertical, F.Cu at (99.4, 66.0)
- added J14: Conn_01x05, Connector_PinHeader_2.54mm:PinHeader_1x05_P2.54mm_Vertical, F.Cu at (99.4, 68.6)
- added J15: Conn_01x05, Connector_PinHeader_2.54mm:PinHeader_1x05_P2.54mm_Vertical, F.Cu at (99.4, 71.1)
- added J16: Conn_01x05, Connector_PinHeader_2.54mm:PinHeader_1x05_P2.54mm_Vertical, F.Cu at (99.4, 73.7)
- added J17: Conn_01x05, Connector_PinHeader_2.54mm:PinHeader_1x05_P2.54mm_Vertical, F.Cu at (99.4, 76.2)
- added J18: Conn_01x05, Connector_PinHeader_2.54mm:PinHeader_1x05_P2.54mm_Vertical, F.Cu at (99.4, 78.7)
- added J19: Conn_01x23, Connector_PinHeader_2.54mm:PinHeader_1x23_P2.54mm_Vertical, F.Cu at (99.4, 81.3)
- added J20: Conn_01x23, Connector_PinHeader_2.54mm:PinHeader_1x23_P2.54mm_Vertical, F.Cu at (99.4, 83.8)
- added J21: Conn_01x17, Connector_PinHeader_2.54mm:PinHeader_1x17_P2.54mm_Vertical, F.Cu at (114.6, 86.4)
- added J22: Conn_01x17, Connector_PinHeader_2.54mm:PinHeader_1x17_P2.54mm_Vertical, F.Cu at (114.6, 88.9)
- added J23: Conn_01x17, Connector_PinHeader_2.54mm:PinHeader_1x17_P2.54mm_Vertical, F.Cu at (114.6, 91.4)
- added J24: Conn_01x10, Connector_PinHeader_2.54mm:PinHeader_1x10_P2.54mm_Vertical, F.Cu at (114.6, 94.0)
- added J25: Conn_01x10, Connector_PinHeader_2.54mm:PinHeader_1x10_P2.54mm_Vertical, F.Cu at (114.6, 96.5)
- added J26: Conn_01x09, Connector_PinHeader_2.54mm:PinHeader_1x09_P2.54mm_Vertical, F.Cu at (117.2, 99.1)
- added J27: Conn_01x09, Connector_PinHeader_2.54mm:PinHeader_1x09_P2.54mm_Vertical, F.Cu at (117.2, 101.6)
- added J28: Conn_01x01, Connector_PinHeader_2.54mm:PinHeader_1x01_P2.54mm_Vertical, F.Cu at (110.1, 53.3)
- added J29: Conn_01x02, Connector_PinHeader_2.54mm:PinHeader_1x02_P2.54mm_Vertical, F.Cu at (107.3, 55.9)
- added J30: Conn_01x03, Connector_PinHeader_2.54mm:PinHeader_1x03_P2.54mm_Vertical, F.Cu at (104.5, 58.4)
- added J31: Conn_01x04, Connector_PinHeader_2.54mm:PinHeader_1x04_P2.54mm_Vertical, F.Cu at (101.9, 61.0)
- added JP2: SolderJumper_2_Open, Jumper:SolderJumper-2_P1.3mm_Open_RoundedPad1.0x1.5mm, F.Cu at (164.6, 54.8)
- added RV1: ERZ-V14D220, Varistor:RV_Disc_D15.5mm_W4.7mm_P7.5mm, F.Cu at (204.5, 55.5)
- D13: value TP6KE47A -> 1N5818; footprint Diode_THT:D_DO-15_P12.70mm_Horizontal -> Diode_THT:D_DO-41_SOD81_P10.16mm_Horizontal
- F1: value 0ZRP0050FF1E -> MF-R050; footprint Fuse:Fuse_BelFuse_0ZRE0055FF_L14.0mm_W4.1mm -> Fuse:Fuse_BelFuse_0ZRE0100FF_L18.7mm_W5.1mm
- J7: value Conn_02x04 -> Conn_02x04_Odd_Even
- J92: value D7 out -> D7out
- J93: value D6 out -> D6out
- J94: value D5 out -> D5out
- JP1: value Reset Prot -> Jumper_NO_Small
- U1, U2: value MPXH6115 -> MPXH6115_Adapter_Vertical
- moved F1 32.3 mm to (188.5, 58.0), turned to 180 degrees
- moved C26 31.0 mm to (155.8, 41.8)
- moved R15 31.0 mm to (156.3, 44.8)
- moved R17 31.0 mm to (148.6, 47.8)
- moved U4 31.0 mm to (148.2, 58.0)
- moved C25 30.8 mm to (164.8, 67.8), turned to 270 degrees
- moved D11 28.0 mm to (167.7, 67.9), turned to 0 degrees
- moved C28 28.0 mm to (141.1, 41.7)
- moved R21 28.0 mm to (133.9, 47.7)
- moved U6 28.0 mm to (133.5, 57.9)
- moved R19 28.0 mm to (141.6, 44.7)
- moved C30 25.5 mm to (126.5, 41.6)
- moved R23 25.5 mm to (127.0, 44.6)
- moved R24 25.5 mm to (119.4, 47.6)
- moved U8 25.5 mm to (118.9, 57.9)
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Connections:
- C1 pad 2: VDD -> VDDA
- C17 pad 1: SigRtn -> GND
- C18 pad 1: Net-(C18-Pad1) -> 12V
- C18 pad 2: SigRtn -> GND
- C19 pad 1: Net-(C18-Pad1) -> 12V
- C19 pad 2: SigRtn -> GND
- C2 pad 2: VDD -> VDDA
- C20 pad 2: SigRtn -> GND
- C21 pad 2: SigRtn -> GND
- C22 pad 2: SigRtn -> GND
- C25 pad 1: SigRtn -> GND
- C26 pad 1: SigRtn -> GND
- C27 pad 1: SigRtn -> GND
- C28 pad 1: SigRtn -> GND
- C29 pad 1: SigRtn -> GND
- C30 pad 1: SigRtn -> GND
- D11 pad 2: SigRtn -> GND
- D13 pad 1: Net-(C18-Pad1) -> 12V
- D13 pad 2: SigRtn -> 12V-Raw
- D17 pad 2: SigRtn -> GND
- J1 pad 13: 12V -> 12V-Raw
- J1 pad 18: SigRtn -> GND
- J1 pad 5: SigRtn -> GND
- J3 pad 1: SigRtn -> GND
- J7 pad 7: SigRtn -> GND
- J7 pad 8: SigRtn -> GND
- J8 pad 4: SigRtn -> GND
- J8 pad 5: SigRtn -> GND
- U1 pad 2: VDD -> VDDA
- U10 pad 15: SigRtn -> GND
- U10 pad 9: SigRtn -> GND
- U2 pad 2: VDD -> VDDA
- U3 pad 1: Net-(C18-Pad1) -> 12V
- U3 pad 2: SigRtn -> GND
- U4 pad 3: SigRtn -> GND
- U5 pad 3: SigRtn -> GND
- U6 pad 3: SigRtn -> GND
- U7 pad 3: SigRtn -> GND
- U8 pad 3: SigRtn -> GND
- U9 pad 8: SigRtn -> GND
Routing:
- net SigRtn: track 0.00 -> 503.3 mm, vias 0 -> 5
- net 12V: track 0.00 -> 363.9 mm, vias 0 -> 5
- net VDDA: track 0.00 -> 363.6 mm, vias 0 -> 2
- net VDD: track 0.00 -> 341.9 mm, vias 0 -> 3
- net D13-control: track 0.00 -> 111.1 mm
- net D12-control: track 0.00 -> 104.9 mm
- net IAT_Sensor: track 0.00 -> 96.8 mm, vias 0 -> 1
- net D11-control: track 0.00 -> 96.5 mm
- net D10-control: track 0.00 -> 89.8 mm
- net MCU-D49: track 0.00 -> 84.9 mm, vias 0 -> 4
- net D49-control: track 0.00 -> 83.7 mm
- net D48-control: track 0.00 -> 83.4 mm
- net CLT_Sensor: track 0.00 -> 82.0 mm, vias 0 -> 1
- net D9-control: track 0.00 -> 81.1 mm
- net MCU-D48: track 0.00 -> 76.5 mm, vias 0 -> 2
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- added copper zone on B.Cu, net GND
- added copper zone on F.Cu, net GND
Other:
- board text added: "0"
- board text added: "1"
- board text added: "10"
- board text added: "11"
- board text added: "12"
- board text added: "12V"
- board text added: "13"
- board text added: "16"
- board text added: "17"
- board text added: "18"
- board text added: "19"
- board text added: "2"
- board text added: "3"
- board text added: "4"
- board text added: "5"
- board text added: "5V"
- board text added: "6"
- board text added: "7"
- board text added: "8"
- board text added: "9"
- board text added: "Bat Volt"
- board text added: "Idle&Spare"
- board text added: "Inj1&Inj2"
- board text added: "Inj3&Inj4"
- board text added: "MPXH6115"
- board text added: "Reset Prot"
- board text added: "SigRtn"
- board text added: "VDD"
- board text removed: "54"
- board text removed: "55"

Commit message: Add files via upload
Parts:
- removed J10: Conn_01x01, DP1600i:Jumper-Pad
- J92: value D7out -> D7 out
- J93: value D6out -> D6 out
- J94: value D5out -> D5 out
Connections:
- J1 pad 17: Net-(J1-Pad17) -> VDD
Routing:
- net VDD: track 341.9 -> 406.4 mm, vias 3 -> 5
- net Net-(J1-Pad17): track 13.8 -> 0.00 mm
- net GND: vias 27 -> 40

Commit message: Add files via upload
Parts:
- J2: value 12V Test -> 12V
- J87: value Pin D4 -> Pin4
- J88: value Pin D3 -> Pin3
- J89: value Pin D2 -> Pin2
- J90: value Pin D1 -> Pin1
- J91: value Pin D0 -> Pin0
- J92: value D7 out -> D7out
- J93: value D6 out -> D6out
- J94: value D5 out -> D5out
- J95: value Step 2B -> Step2B
- J96: value Step 2A -> Step2A
- J97: value Step 1A -> Step1A
- J98: value Step 1B -> Step1B
Connections:
- net ADC-Clamp-18 renamed Clamp-18
- net ADC-Clamp-19 renamed Clamp-19
- D12 pad 1: VDDA -> VDD
- D18 pad 1: VDDA -> VDD
Routing:
- net VDD: track 406.4 -> 438.0 mm
- net VDDA: track 363.6 -> 335.1 mm
- net GND: vias 40 -> 39
Other:
- board text added: "Ign1&Ign2"
- board text added: "Ign3&Ign4"
- board text added: "Reset Prot."
- board text removed: "Reset Prot"

Commit message: Add files via upload
Other:
- board text added: "DP1600i"
- board text added: "MADE FOR SPEEDUINO"
- board text added: "PCB design by Robert Hiebert December 2022"

Commit message: Add files via upload
Parts:
- D10, D12, D16, D18, D2, D4, D6, D8: value 1N5818 -> 1N5231B
- J2: value 12V -> 12V Test
- J87: value Pin4 -> Pin D4
- J88: value Pin3 -> Pin D3
- J89: value Pin2 -> Pin D2
- J90: value Pin1 -> Pin D1
- J91: value Pin0 -> Pin D0
- J92: value D7out -> D7 out
- J93: value D6out -> D6 out
- J94: value D5out -> D5 out
- J95: value Step2B -> Step 2B
- J96: value Step2A -> Step 2A
- J97: value Step1A -> Step 1A
- J98: value Step1B -> Step 1B
- U4, U5, U6, U7, U8: value IXDI604PI -> IXDNI604PI
- moved D4 0.15 mm to (169.2, 124.2)
- moved D18 0.13 mm to (195.5, 71.1)
- moved D6 0.13 mm to (102.2, 118.0)
- moved D10 0.09 mm to (142.5, 130.4)
- moved D2 0.08 mm to (125.7, 133.8)
Connections:
- D10 pad 1: VDDA -> SigRtn
- D12 pad 1: VDD -> GND
- D16 pad 1: VDDA -> SigRtn
- D18 pad 1: VDD -> GND
- D2 pad 1: VDDA -> SigRtn
- D4 pad 1: VDDA -> SigRtn
- D6 pad 1: VDDA -> SigRtn
- D8 pad 1: VDDA -> SigRtn
Routing:
- net VDDA: track 335.1 -> 267.8 mm, vias 2 -> 4
- net VDD: track 438.0 -> 406.4 mm
- net SigRtn: track 503.3 -> 502.0 mm
- net GND: track 47.2 -> 48.1 mm, vias 39 -> 69

Commit message: Add files via upload
Parts:
- U3: value LM2940T-5.0 -> LM2937ET-5.0
