File: KiCad Files/DP1600i/DP1600i.kicad_pcb (KiCad board)
At the start: 2 copper layers, 120.4 x 100.1 mm, 128 parts, among them J1 DB25_Male, J11 Conn_01x05, J12 Conn_01x05, J13 Conn_01x05, J14 Conn_01x05, J15 Conn_01x05, J16 Conn_01x05, J17 Conn_01x05, J18 Conn_01x05, J19 Conn_01x23, J2 12V Test, J20 Conn_01x23, J21 Conn_01x17, J22 Conn_01x17, J23 Conn_01x17, J24 Conn_01x10, J25 Conn_01x10, J26 Conn_01x09, J27 Conn_01x09, J28 Conn_01x01, J29 Conn_01x02, J3 Conn_01x07, J30 Conn_01x03, J31 Conn_01x04, J4 Conn_01x08, J5 Conn_01x04, J6 Conn_01x02, J7 Conn_02x04_Odd_Even, J8 Conn_01x05, J87 Pin D4, J88 Pin D3, J89 Pin D2, J9 Conn_01x08, J90 Pin D1, J91 Pin D0, J92 D7 out, J93 D6 out, J94 D5 out, J95 Step 2B, J96 Step 2A, J97 Step 1A, J98 Step 1B, U1 MPXH6115_Adapter_Vertical, U10 A4988StepStick, U2 MPXH6115_Adapter_Vertical, U3 LM2937ET-5.0, U4 IXDNI604PI, U5 IXDNI604PI, U6 IXDNI604PI, U7 IXDNI604PI, U8 IXDNI604PI, U9 ULN2004AN

Commit message: Add files via upload
Parts:
- removed C28, C29, C30: 0.1uF, Capacitor_THT:C_Disc_D5.0mm_W2.5mm_P2.50mm
- removed J11, J12, J13, J14, J15, J16, J17, J18: Conn_01x05, Connector_PinHeader_2.54mm:PinHeader_1x05_P2.54mm_Vertical
- removed J19, J20: Conn_01x23, Connector_PinHeader_2.54mm:PinHeader_1x23_P2.54mm_Vertical
- removed J21, J22, J23: Conn_01x17, Connector_PinHeader_2.54mm:PinHeader_1x17_P2.54mm_Vertical
- removed J24, J25: Conn_01x10, Connector_PinHeader_2.54mm:PinHeader_1x10_P2.54mm_Vertical
- removed J26, J27: Conn_01x09, Connector_PinHeader_2.54mm:PinHeader_1x09_P2.54mm_Vertical
- removed J28: Conn_01x01, Connector_PinHeader_2.54mm:PinHeader_1x01_P2.54mm_Vertical
- removed J29: Conn_01x02, Connector_PinHeader_2.54mm:PinHeader_1x02_P2.54mm_Vertical
- removed J30: Conn_01x03, Connector_PinHeader_2.54mm:PinHeader_1x03_P2.54mm_Vertical
- removed J31: Conn_01x04, Connector_PinHeader_2.54mm:PinHeader_1x04_P2.54mm_Vertical
- added C3: .01uF, Capacitor_THT:C_Disc_D5.0mm_W2.5mm_P2.50mm, F.Cu at (154.5, 53.5)
- added C4: 1uF, Capacitor_THT:C_Disc_D5.0mm_W2.5mm_P2.50mm, F.Cu at (157.6, 53.5)
- added R25: 100K, Resistor_THT:R_Axial_DIN0207_L6.3mm_D2.5mm_P7.62mm_Horizontal, F.Cu at (132.8, 43.1)
- added R26: 100K, Resistor_THT:R_Axial_DIN0207_L6.3mm_D2.5mm_P7.62mm_Horizontal, F.Cu at (132.7, 49.4)
- added R27: 100K, Resistor_THT:R_Axial_DIN0207_L6.3mm_D2.5mm_P7.62mm_Horizontal, F.Cu at (102.2, 42.9)
- added R28: 100K, Resistor_THT:R_Axial_DIN0207_L6.3mm_D2.5mm_P7.62mm_Horizontal, F.Cu at (102.3, 49.1)
- added R29: 100K, Resistor_THT:R_Axial_DIN0207_L6.3mm_D2.5mm_P7.62mm_Horizontal, F.Cu at (105.1, 68.4)
- added R30: 100K, Resistor_THT:R_Axial_DIN0207_L6.3mm_D2.5mm_P7.62mm_Horizontal, F.Cu at (98.8, 68.4)
- added R31: 1K, Resistor_THT:R_Axial_DIN0207_L6.3mm_D2.5mm_P7.62mm_Horizontal, F.Cu at (132.7, 46.3)
- added R32: 1K, Resistor_THT:R_Axial_DIN0207_L6.3mm_D2.5mm_P7.62mm_Horizontal, F.Cu at (132.7, 52.5)
- added R33: 1K, Resistor_THT:R_Axial_DIN0207_L6.3mm_D2.5mm_P7.62mm_Horizontal, F.Cu at (102.2, 46.0)
- added R34: 1K, Resistor_THT:R_Axial_DIN0207_L6.3mm_D2.5mm_P7.62mm_Horizontal, F.Cu at (102.2, 52.2)
- added R35: 1K, Resistor_THT:R_Axial_DIN0207_L6.3mm_D2.5mm_P7.62mm_Horizontal, F.Cu at (102.0, 68.4)
- added R36: 1K, Resistor_THT:R_Axial_DIN0207_L6.3mm_D2.5mm_P7.62mm_Horizontal, F.Cu at (95.7, 68.4)
- added R37: 100K, Resistor_THT:R_Axial_DIN0207_L6.3mm_D2.5mm_P7.62mm_Horizontal, F.Cu at (159.2, 104.4)
- added R38: 100K, Resistor_THT:R_Axial_DIN0207_L6.3mm_D2.5mm_P7.62mm_Horizontal, F.Cu at (159.2, 98.2)
- added R39: 100K, Resistor_THT:R_Axial_DIN0207_L6.3mm_D2.5mm_P7.62mm_Horizontal, F.Cu at (130.3, 104.3)
- added R40: 100K, Resistor_THT:R_Axial_DIN0207_L6.3mm_D2.5mm_P7.62mm_Horizontal, F.Cu at (130.2, 98.1)
- added R41: 1K, Resistor_THT:R_Axial_DIN0207_L6.3mm_D2.5mm_P7.62mm_Horizontal, F.Cu at (159.2, 101.3)
- added R42: 1K, Resistor_THT:R_Axial_DIN0207_L6.3mm_D2.5mm_P7.62mm_Horizontal, F.Cu at (159.2, 95.1)
- added R43: 1K, Resistor_THT:R_Axial_DIN0207_L6.3mm_D2.5mm_P7.62mm_Horizontal, F.Cu at (130.3, 101.2)
- added R44: 1K, Resistor_THT:R_Axial_DIN0207_L6.3mm_D2.5mm_P7.62mm_Horizontal, F.Cu at (130.2, 95.1)
- C26: value 0.1uF -> .01uF
- C27: value 0.1uF -> 1uF
- J6: value Conn_01x02 -> Conn_02x03_Odd_Even; footprint Connector_PinHeader_2.54mm:PinHeader_1x02_P2.54mm_Vertical -> Connector_PinHeader_2.54mm:PinHeader_2x03_P2.54mm_Vertical
- U3: value LM2937ET-5.0 -> LM2940T-5.0
- moved C27 59.4 mm to (157.6, 45.4), turned to 90 degrees
- moved R23 49.6 mm to (96.6, 83.9), turned to 0 degrees
- moved D12 44.3 mm to (135.5, 84.2)
- moved D18 42.7 mm to (154.3, 82.6)
- moved D11 37.6 mm to (135.6, 87.4), turned to 180 degrees
- moved R24 36.6 mm to (104.2, 80.9), turned to 180 degrees
- moved D17 36.0 mm to (154.3, 85.9), turned to 180 degrees
- moved C25 32.9 mm to (138.5, 87.6), turned to 90 degrees
- moved U6 32.2 mm to (104.5, 43.8), turned to 0 degrees
- moved C17 31.2 mm to (157.3, 86.1), turned to 90 degrees
- moved R20 29.2 mm to (114.7, 95.8)
- moved R22 29.2 mm to (117.7, 103.5)
- moved U7 29.2 mm to (128.0, 103.4)
- moved R19 24.7 mm to (117.8, 51.4), turned to 90 degrees
- moved U5 21.5 mm to (156.9, 103.6)
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Connections:
- C21 pad 1: VDD -> 5V-Drivers
- C22 pad 1: VDD -> 5V-Drivers
- C26 pad 2: VDD -> 12V
- C27 pad 2: VDD -> 12V
- D10 pad 1: SigRtn -> ADC-Clamp-4
- D10 pad 2: ADC-Clamp-4 -> SigRtn
- D12 pad 1: GND -> Clamp-18
- D12 pad 2: Clamp-18 -> GND
- D16 pad 1: SigRtn -> ADC-Clamp-6
- D16 pad 2: ADC-Clamp-6 -> SigRtn
- D18 pad 1: GND -> Clamp-19
- D18 pad 2: Clamp-19 -> GND
- D2 pad 1: SigRtn -> ADC-Clamp-3
- D2 pad 2: ADC-Clamp-3 -> SigRtn
- D4 pad 1: SigRtn -> ADC-Clamp-5
- D4 pad 2: ADC-Clamp-5 -> SigRtn
- D6 pad 1: SigRtn -> ADC-Clamp-2
- D6 pad 2: ADC-Clamp-2 -> SigRtn
- D8 pad 1: SigRtn -> ADC-Clamp-7
- D8 pad 2: ADC-Clamp-7 -> SigRtn
- F1 pad 2: VDD -> 5V-Drivers
- J1 pad 17: VDD -> 5V-Drivers
- J6 pad 1: VDD -> 5V-Drivers
- J6 pad 2: VDD -> 5V-Drivers
- J8 pad 3: VDD -> 5V-Drivers
- R12 pad 2: VDD -> 5V-Drivers
- R13 pad 2: VDD -> 5V-Drivers
- U10 pad 1: Net-(U10-Pad1) -> MCU-D24
- U10 pad 10: VDD -> 5V-Drivers
- U3 pad 3: VDD -> 5V-Drivers
- U4 pad 2: MCU-D8 -> Net-(R31-Pad1)
- U4 pad 4: MCU-D9 -> Net-(R32-Pad1)
- U4 pad 6: VDD -> 12V
- U5 pad 2: MCU-D50 -> Net-(R41-Pad1)
- U5 pad 4: MCU-D51 -> Net-(R42-Pad1)
- U5 pad 6: VDD -> 5V-Drivers
- U6 pad 2: MCU-D10 -> Net-(R33-Pad1)
- U6 pad 4: MCU-D11 -> Net-(R34-Pad1)
- U6 pad 6: VDD -> 12V
- U7 pad 2: MCU-D52 -> Net-(R43-Pad1)
- U7 pad 4: MCU-D53 -> Net-(R44-Pad1)
- U7 pad 6: VDD -> 5V-Drivers
- U8 pad 2: MCU-D12 -> Net-(R35-Pad1)
- U8 pad 4: MCU-D13 -> Net-(R36-Pad1)
- U8 pad 6: VDD -> 12V
Routing:
- net VDD: track 406.4 -> 0.00 mm, vias 5 -> 0
- net 5V-Drivers: track 0.00 -> 254.7 mm, vias 0 -> 5
- net 12V: track 363.9 -> 430.8 mm, vias 5 -> 4
- net VDDA: track 267.8 -> 211.3 mm, vias 4 -> 3
- net MCU-D51: track 23.6 -> 69.4 mm, vias 0 -> 2
- net Clamp-18: track 60.2 -> 106.0 mm, vias 1 -> 2
- net D12-control: track 104.9 -> 148.4 mm, vias 0 -> 2
- net Clamp-19: track 56.4 -> 92.7 mm, vias 1 -> 2
- net MCU-D52: track 29.3 -> 60.3 mm
- net SigRtn: track 502.0 -> 473.2 mm, vias 5 -> 6
- net D53-control: track 75.5 -> 100.1 mm, vias 2 -> 0
- net MCU-D53: track 59.2 -> 83.2 mm, vias 1 -> 0
- net D52-control: track 72.8 -> 96.8 mm, vias 2 -> 0
- net MCU-D50: track 17.0 -> 36.4 mm
- net D13-control: track 111.1 -> 130.0 mm, vias 0 -> 1
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Other:
- board text added: "22"
- board text added: "23"
- board text added: "24"
- board text added: "25"
- board text removed: "12V"
- board text removed: "SigRtn"
- board text removed: "VDDA"
