File: KiCad Files/DP1600i/file63700699.sch (KiCad schematic (older format))
At the start: 50 parts, among them U1 MPXH6115_Adapter, U2 MPXH6115_Adapter

Commit message: Add files via upload
Parts:
- removed C3, C4: 1uF, Capacitor_THT:C_Disc_D5.0mm_W2.5mm_P2.50mm, symbol Device:C
- removed U1, U2: MPXH6115_Adapter, MPXH61115AC6U Adapter:MPXH6115_Adapter, symbol DP1600i:MPXH6115_Adapter
- added U1, U2: MPXH6115_Adapter_Vertical, MPXH61115AC6U Adapter:MPXH6115_Adapter_Vertical, symbol DP1600i:MPXH6115_Adapter_Vertical
- C1, C2: value 0.01uF -> 0.1uF
- C10, C9: value 470pf -> 47pf
- R5, R6: value 470R -> 51K
Connections:
- wire segments 187 -> 179
- no-connect marks 10 -> 2
Other:
- moved on the sheet: C1, C2
Changed lines of the file:
@@
 	0    1    1    0
 $EndComp
-Wire Wire Line
-	1050 1850 1150 1850
 $Comp
 L Device:C C1
 U 1 1 5CD20B6A
-P 1150 1500
-F 0 "C1" H 950 1550 50  0000 L CNN
-F 1 "0.01uF" H 850 1450 50  0000 L CNN
-F 2 "Capacitor_THT:C_Disc_D5.0mm_W2.5mm_P2.50mm" H 1188 1350 50  0001 C CNN
-F 3 "~" H 1150 1500 50  0001 C CNN
-F 4 "445-174244-1-ND" H 0   0   50  0001 C CNN "Digikey Part Number"
-F 5 "TDK" H 0   0   50  0001 C CNN "Manufacturer_Name"
-F 6 "FA18X7R1H103KNU06" H 0   0   50  0001 C CNN "Manufacturer_Part_Number"
-F 7 "https://www.digikey.com.au/product-detail/en/tdk-corporation/FA18X7R1H103KNU06/445-174244-1-ND/5865002" H 0   0   50  0001 C CNN "URL"
-	1    1150 1500
-	1    0    0    -1
-$EndComp
-$Comp
-L Device:C C3
-U 1 1 5CD2115B
-P 1450 1500
-F 0 "C3" H 1565 1546 50  0000 L CNN
-F 1 "1uF" H 1565 1455 50  0000 L CNN
-F 2 "Capacitor_THT:C_Disc_D5.0mm_W2.5mm_P2.50mm" H 1488 1350 50  0001 C CNN
-F 3 "~" H 1450 1500 50  0001 C CNN
-F 4 "445-180543-1-ND" H 0   0   50  0001 C CNN "Digikey Part Number"
-F 5 "TDK" H 0   0   50  0001 C CNN "Manufacturer_Name"
-F 6 "FA18X7R1E105KRU06" H 0   0   50  0001 C CNN "Manufacturer_Part_Number"
-F 7 "https://www.digikey.com.au/product-detail/en/tdk-corporation/FA18X7R1E105KRU06/445-180543-1-ND/9560669" H 0   0   50  0001 C CNN "URL"
-	1    1450 1500
+P 1450 1550
+F 0 "C1" H 1250 1600 50  0000 L CNN
+F 1 "0.1uF" H 1150 1500 50  0000 L CNN
+F 2 "Capacitor_THT:C_Disc_D5.0mm_W2.5mm_P2.50mm" H 1488 1400 50  0001 C CNN
+F 3 "~" H 1450 1550 50  0001 C CNN
+F 4 "445-174244-1-ND" H 300 50  50  0001 C CNN "Digikey Part Number"
+F 5 "TDK" H 300 50  50  0001 C CNN "Manufacturer_Name"
+F 6 "FA18X7R1H103KNU06" H 300 50  50  0001 C CNN "Manufacturer_Part_Number"
+F 7 "https://www.digikey.com.au/product-detail/en/tdk-corporation/FA18X7R1H103KNU06/445-174244-1-ND/5865002" H 300 50  50  0001 C CNN "URL"
+	1    1450 1550
 	1    0    0    -1
 $EndComp
@@
 L power:GND #PWR07
 U 1 1 5CD21884
-P 1300 1100
-F 0 "#PWR07" H 1300 850 50  0001 C CNN
-F 1 "GND" H 1305 927 50  0000 C CNN
-F 2 "" H 1300 1100 50  0001 C CNN
-F 3 "" H 1300 1100 50  0001 C CNN
-	1    1300 1100
+P 1450 1250
+F 0 "#PWR07" H 1450 1000 50  0001 C CNN
+F 1 "GND" H 1455 1077 50  0000 C CNN
+F 2 "" H 1450 1250 50  0001 C CNN
+F 3 "" H 1450 1250 50  0001 C CNN
+	1    1450 1250
 	-1   0    0    1
 $EndComp
-Wire Wire Line
-	1150 1350 1300 1350
-Wire Wire Line
-	1300 1350 1300 1100
-Connection ~ 1300 1350
-Wire Wire Line
-	1300 1350 1450 1350
-Wire Wire Line
-	1150 1850 1150 1650
-Connection ~ 1150 1850
-Wire Wire Line
-	1150 1850 1450 1850
-Wire Wire Line
-	1450 1850 1450 1650
 Text Notes 1800 1200 0    74   ~ 0
 MAP Sensor
@@
 P 2650 1900
 F 0 "R5" V 2750 1900 50  0000 C CNN
-F 1 "470R" V 2850 1900 50  0000 C CNN
+F 1 "51K" V 2850 1900 50  0000 C CNN
 F 2 "Resistor_THT:R_Axial_DIN0207_L6.3mm_D2.5mm_P7.62mm_Horizontal" V 2580 1900 50  0001 C CNN
 F 3 "~" H 2650 1900 50  0001 C CNN
@@
 P 2950 2050
 F 0 "C9" H 3065 2096 50  0000 L CNN
-F 1 "470pf" H 3065 2005 50  0000 L CNN
+F 1 "47pf" H 3065 2005 50  0000 L CNN
 F 2 "Capacitor_THT:C_Disc_D5.0mm_W2.5mm_P2.50mm" H 2988 1900 50  0001 C CNN
 F 3 "~" H 2950 2050 50  0001 C CNN
@@
 	0    1    1    0
 $EndComp
-Wire Wire Line
-	1100 3550 1200 3550
 $Comp
 L Device:C C2
 U 1 1 63876419
-P 1200 3200
-F 0 "C2" H 1000 3250 50  0000 L CNN
-F 1 "0.01uF" H 900 3150 50  0000 L CNN
-F 2 "Capacitor_THT:C_Disc_D5.0mm_W2.5mm_P2.50mm" H 1238 3050 50  0001 C CNN
-F 3 "~" H 1200 3200 50  0001 C CNN
-F 4 "445-174244-1-ND" H 50  1700 50  0001 C CNN "Digikey Part Number"
-F 5 "TDK" H 50  1700 50  0001 C CNN "Manufacturer_Name"
-F 6 "FA18X7R1H103KNU06" H 50  1700 50  0001 C CNN "Manufacturer_Part_Number"
-F 7 "https://www.digikey.com.au/product-detail/en/tdk-corporation/FA18X7R1H103KNU06/445-174244-1-ND/5865002" H 50  1700 50  0001 C CNN "URL"
-	1    1200 3200
-	1    0    0    -1
-$EndComp
-$Comp
-L Device:C C4
-U 1 1 63876423
-P 1500 3200
-F 0 "C4" H 1615 3246 50  0000 L CNN
-F 1 "1uF" H 1615 3155 50  0000 L CNN
-F 2 "Capacitor_THT:C_Disc_D5.0mm_W2.5mm_P2.50mm" H 1538 3050 50  0001 C CNN
-F 3 "~" H 1500 3200 50  0001 C CNN
-F 4 "445-180543-1-ND" H 50  1700 50  0001 C CNN "Digikey Part Number"
-F 5 "TDK" H 50  1700 50  0001 C CNN "Manufacturer_Name"
-F 6 "FA18X7R1E105KRU06" H 50  1700 50  0001 C CNN "Manufacturer_Part_Number"
-F 7 "https://www.digikey.com.au/product-detail/en/tdk-corporation/FA18X7R1E105KRU06/445-180543-1-ND/9560669" H 50  1700 50  0001 C CNN "URL"
-	1    1500 3200
+P 1500 3250
+F 0 "C2" H 1300 3300 50  0000 L CNN
+F 1 "0.1uF" H 1200 3200 50  0000 L CNN
+F 2 "Capacitor_THT:C_Disc_D5.0mm_W2.5mm_P2.50mm" H 1538 3100 50  0001 C CNN
+F 3 "~" H 1500 3250 50  0001 C CNN
+F 4 "445-174244-1-ND" H 350 1750 50  0001 C CNN "Digikey Part Number"
+F 5 "TDK" H 350 1750 50  0001 C CNN "Manufacturer_Name"
+F 6 "FA18X7R1H103KNU06" H 350 1750 50  0001 C CNN "Manufacturer_Part_Number"
+F 7 "https://www.digikey.com.au/product-detail/en/tdk-corporation/FA18X7R1H103KNU06/445-174244-1-ND/5865002" H 350 1750 50  0001 C CNN "URL"
+	1    1500 3250
 	1    0    0    -1
 $EndComp
@@
 L power:GND #PWR08
 U 1 1 63876429
-P 1350 2800
-F 0 "#PWR08" H 1350 2550 50  0001 C CNN
-F 1 "GND" H 1355 2627 50  0000 C CNN
-F 2 "" H 1350 2800 50  0001 C CNN
-F 3 "" H 1350 2800 50  0001 C CNN
-	1    1350 2800
+P 1500 2950
+F 0 "#PWR08" H 1500 2700 50  0001 C CNN
+F 1 "GND" H 1505 2777 50  0000 C CNN
+F 2 "" H 1500 2950 50  0001 C CNN
+F 3 "" H 1500 2950 50  0001 C CNN
+	1    1500 2950
 	-1   0    0    1
 $EndComp
-Wire Wire Line
-	1200 3050 1350 3050
-Wire Wire Line
-	1350 3050 1350 2800
-Connection ~ 1350 3050
-Wire Wire Line
-	1350 3050 1500 3050
-Wire Wire Line
-	1200 3550 1200 3350
-Connection ~ 1200 3550
-Wire Wire Line
-	1200 3550 1500 3550
-Wire Wire Line
-	1500 3550 1500 3350
 Text Notes 1850 2900 0    74   ~ 0
 Baro Sensor
@@
 P 2700 3600
 F 0 "R6" V 2800 3600 50  0000 C CNN
-F 1 "470R" V 2900 3600 50  0000 C CNN
+F 1 "51K" V 2900 3600 50  0000 C CNN
 F 2 "Resistor_THT:R_Axial_DIN0207_L6.3mm_D2.5mm_P7.62mm_Horizontal" V 2630 3600 50  0001 C CNN
 F 3 "~" H 2700 3600 50  0001 C CNN
@@
 P 3000 3750
 F 0 "C10" H 3115 3796 50  0000 L CNN
-F 1 "470pf" H 3115 3705 50  0000 L CNN
+F 1 "47pf" H 3115 3705 50  0000 L CNN
 F 2 "Capacitor_THT:C_Disc_D5.0mm_W2.5mm_P2.50mm" H 3038 3600 50  0001 C CNN
 F 3 "~" H 3000 3750 50  0001 C CNN
@@
 Text Notes 8300 5450 0    50   ~ 0
 VR conditoner module is in Aux board
-$Comp
-L DP1600i:MPXH6115_Adapter U1
-U 1 1 6379BA31
-P 2000 2000
-F 0 "U1" H 2000 2365 50  0000 C CNN
-F 1 "MPXH6115_Adapter" H 2000 2274 50  0000 C CNN
-F 2 "MPXH61115AC6U Adapter:MPXH6115_Adapter" H 2000 2000 50  0001 C CNN
-F 3 "" H 2000 2000 50  0001 C CNN
-	1    2000 2000
-	1    0    0    -1
-$EndComp
-$Comp
-L DP1600i:MPXH6115_Adapter U2
-U 1 1 6379C307
-P 2000 3700
-F 0 "U2" H 2000 4065 50  0000 C CNN
-F 1 "MPXH6115_Adapter" H 2000 3974 50  0000 C CNN
-F 2 "MPXH61115AC6U Adapter:MPXH6115_Adapter" H 2000 3700 50  0001 C CNN
-F 3 "" H 2000 3700 50  0001 C CNN
-	1    2000 3700
-	1    0    0    -1
-$EndComp
 Wire Wire Line
 	1650 2000 1450 2000
 Wire Wire Line
 	1450 2000 1450 1850
-Connection ~ 1450 1850
 Wire Wire Line
 	1000 2100 1650 2100
@@
 Wire Wire Line
 	1500 3700 1500 3550
-Connection ~ 1500 3550
 Wire Wire Line
 	1050 3800 1650 3800
@@
 	2550 4100 2550 3600
 NoConn ~ 1650 1900
-NoConn ~ 2350 1900
-NoConn ~ 2350 2000
-NoConn ~ 2350 2100
-NoConn ~ 2350 2200
-NoConn ~ 2350 3600
-NoConn ~ 2350 3700
-NoConn ~ 2350 3800
-NoConn ~ 2350 3900
 NoConn ~ 1650 3600
 $Comp
@@
 	4900 1250 5050 1250
 Connection ~ 5050 1250
+Wire Wire Line
+	1050 1850 1450 1850
+Wire Wire Line
+	1100 3550 1500 3550
+Wire Wire Line
+	1500 2950 1500 3100
+Wire Wire Line
+	1500 3400 1500 3550
+Connection ~ 1500 3550
+Wire Wire Line
+	1450 1250 1450 1400
+Wire Wire Line
+	1450 1700 1450 1850
+Connection ~ 1450 1850
+$Comp
+L DP1600i:MPXH6115_Adapter_Vertical U1
+U 1 1 6381C9E7
+P 2000 2000
+F 0 "U1" H 1850 2350 50  0000 L CNN
+F 1 "MPXH6115_Adapter_Vertical" H 1650 2250 50  0000 L CNN
+F 2 "MPXH61115AC6U Adapter:MPXH6115_Adapter_Vertical" H 2000 2000 50  0001 C CNN
+F 3 "" H 2000 2000 50  0001 C CNN
+	1    2000 2000
+	1    0    0    -1
+$EndComp
+$Comp
+L DP1600i:MPXH6115_Adapter_Vertical U2
+U 1 1 6381CCD6
+P 2000 3700
+F 0 "U2" H 1850 4050 50  0000 L CNN
+F 1 "MPXH6115_Adapter_Vertical" H 1650 3950 50  0000 L CNN
+F 2 "MPXH61115AC6U Adapter:MPXH6115_Adapter_Vertical" H 2000 3700 50  0001 C CNN
+F 3 "" H 2000 3700 50  0001 C CNN
+	1    2000 3700
+	1    0    0    -1
+$EndComp
 $EndSCHEMATC

Commit message: Add files via upload
Connections:
- net ADC-Clamp-2: now also C8.1, R4.1; no longer C14.1, R9.1
- net ADC-Clamp-4: now also C16.1, R11.1; no longer C8.1, R4.1
- net ADC-Clamp-0 renamed ADC-Clamp-3
- net ADC-Clamp-1 renamed ADC-Clamp-5
- net ADC-Clamp-5: now also C14.1, R9.1; no longer C16.1, R11.1
- net MCU-A3 renamed MCU-A1
- net MCU-A5 renamed MCU-A0
Changed lines of the file:
@@
 Wire Wire Line
 	6200 6650 6200 6850
-Text GLabel 6000 6350 2    50   Input ~ 0
+Text GLabel 2450 6350 2    50   Input ~ 0
 ADC-Clamp-2
 Wire Wire Line
@@
 	5000 6650 5150 6650
 Connection ~ 5150 6650
-Text GLabel 6400 6650 2    50   Input ~ 0
+Text GLabel 2850 6650 2    50   Input ~ 0
 MCU-A2
 Wire Wire Line
@@
 	4950 3100 5100 3100
 Connection ~ 5100 3100
-Text GLabel 6350 3100 2    50   Input ~ 0
+Text GLabel 3400 3600 2    50   Input ~ 0
 MCU-A0
 Wire Wire Line
@@
 	5000 4950 5150 4950
 Connection ~ 5150 4950
-Text GLabel 6400 4950 2    50   Input ~ 0
+Text GLabel 3350 1900 2    50   Input ~ 0
 MCU-A1
 Wire Wire Line
@@
 	2650 6650 2650 6850
 Text GLabel 5950 2800 2    50   Input ~ 0
-ADC-Clamp-0
+ADC-Clamp-3
 Wire Wire Line
 	2450 6350 2450 6650
@@
 	2450 6650 2650 6650
 Connection ~ 1600 6650
-Text GLabel 2850 6650 2    50   Input ~ 0
+Text GLabel 6400 4950 2    50   Input ~ 0
 MCU-A4
 Wire Wire Line
@@
 	1    0    0    -1
 $EndComp
-Text GLabel 3350 1900 2    50   Input ~ 0
+Text GLabel 6350 3100 2    50   Input ~ 0
 MCU-A3
 Wire Wire Line
@@
 Text GLabel 2400 4650 2    50   Input ~ 0
 ADC-Clamp-7
-Text GLabel 2450 6350 2    50   Input ~ 0
+Text GLabel 6000 4650 2    50   Input ~ 0
 ADC-Clamp-4
-Text GLabel 6000 4650 2    50   Input ~ 0
-ADC-Clamp-1
+Text GLabel 6000 6350 2    50   Input ~ 0
+ADC-Clamp-5
 $Comp
 L Diode:1N5818 D9
@@
 	1    0    0    -1
 $EndComp
-Text GLabel 3400 3600 2    50   Input ~ 0
+Text GLabel 6400 6650 2    50   Input ~ 0
 MCU-A5
 Wire Wire Line
@@
 	8100 2200 8200 2200
 Text GLabel 7950 2100 0    50   Input ~ 0
-ADC-Clamp-1
+ADC-Clamp-5
 Wire Wire Line
 	7950 2100 8100 2100
@@
 	8100 1400 8200 1400
 Text GLabel 7950 1300 0    50   Input ~ 0
-ADC-Clamp-0
+ADC-Clamp-3
 Wire Wire Line
 	7950 1300 8100 1300

Commit message: Add files via upload
Connections:
- net VDD is gone; now on net VDDA: C1.2, C2.2, U1.2 (VCC), U2.2 (VCC)
- net GND: no longer C1.1, C10.2, C11.2, C12.2, C13.2, C14.2, C15.2, C16.2, C2.1, C23.2, C24.2, C5.2, C6.2, C7.2, C8.2, C9.2, D1.2 (A), D15.2 (A), D3.2 (A), D5.2 (A), D7.2 (A), D9.2 (A), R1.1, U1.3 (Gnd), U2.3 (Gnd)
- new net SigRtn: C1.1, C10.2, C11.2, C12.2, C13.2, C14.2, C15.2, C16.2, C2.1, C23.2, C24.2, C5.2, C6.2, C7.2, C8.2, C9.2, D1.2 (A), D15.2 (A), D3.2 (A), D5.2 (A), D7.2 (A), D9.2 (A), R1.1, U1.3 (Gnd), U2.3 (Gnd)

Commit message: Add files via upload
Connections:
- net VDDA: no longer D12.1 (K), D18.1 (K)
- net ADC-Clamp-18 renamed Clamp-18
- net ADC-Clamp-19 renamed Clamp-19
- new net VDD: D12.1 (K), D18.1 (K)
Changed lines of the file:
@@
 	0    -1   -1   0
-$EndComp
-$Comp
-L power:VDDA #PWR030
-U 1 1 6381A0BB
-P 10450 3000
-F 0 "#PWR030" H 10450 2850 50  0001 C CNN
-F 1 "VDDA" V 10467 3128 50  0000 L CNN
-F 2 "" H 10450 3000 50  0001 C CNN
-F 3 "" H 10450 3000 50  0001 C CNN
-	1    10450 3000
-	0    1    1    0
 $EndComp
 Wire Wire Line
@@
 	9950 3000 10050 3000
 Text GLabel 9800 2900 0    50   Input ~ 0
-ADC-Clamp-18
+Clamp-18
 Wire Wire Line
 	9800 2900 9950 2900
@@
 Connection ~ 9250 6350
 Text GLabel 9050 6050 0    50   Input ~ 0
-ADC-Clamp-19
+Clamp-19
 Text GLabel 8850 6350 0    50   Input ~ 0
 MCU-D19
@@
 	0    -1   -1   0
 $EndComp
-$Comp
-L power:VDDA #PWR050
-U 1 1 6386F39D
-P 10450 3850
-F 0 "#PWR050" H 10450 3700 50  0001 C CNN
-F 1 "VDDA" V 10467 3978 50  0000 L CNN
-F 2 "" H 10450 3850 50  0001 C CNN
-F 3 "" H 10450 3850 50  0001 C CNN
-	1    10450 3850
-	0    1    1    0
-$EndComp
 Wire Wire Line
 	10350 3650 10450 3650
@@
 	9950 3850 10050 3850
 Text GLabel 9800 3750 0    50   Input ~ 0
-ADC-Clamp-19
+Clamp-19
 Wire Wire Line
 	9800 3750 9950 3750
@@
 Connection ~ 9250 5150
 Text GLabel 9050 4850 0    50   Input ~ 0
-ADC-Clamp-18
+Clamp-18
 Text GLabel 8850 5150 0    50   Input ~ 0
 MCU-D18
@@
 Text GLabel 10450 2000 2    50   Input ~ 0
 SigRtn
+$Comp
+L power:VDD #PWR?
+U 1 1 63819CE9
+P 10450 3850
+F 0 "#PWR?" H 10450 3700 50  0001 C CNN
+F 1 "VDD" V 10465 3978 50  0000 L CNN
+F 2 "" H 10450 3850 50  0001 C CNN
+F 3 "" H 10450 3850 50  0001 C CNN
+	1    10450 3850
+	0    1    1    0
+$EndComp
+$Comp
+L power:VDD #PWR?
+U 1 1 63823921
+P 10450 3000
+F 0 "#PWR?" H 10450 2850 50  0001 C CNN
+F 1 "VDD" V 10465 3128 50  0000 L CNN
+F 2 "" H 10450 3000 50  0001 C CNN
+F 3 "" H 10450 3000 50  0001 C CNN
+	1    10450 3000
+	0    1    1    0
+$EndComp
 $EndSCHEMATC

Commit message: Add files via upload
Parts:
- removed D10, D12, D16, D18, D2, D4, D6, D8: 1N5818, Diode_THT:D_DO-41_SOD81_P10.16mm_Horizontal, symbol Diode:1N5818
- added D10, D12, D16, D18, D2, D4, D6, D8: 1N5231B, Diode_THT:D_DO-41_SOD81_P10.16mm_Horizontal, symbol V10-Ign-Inj-Drivers-V2-rescue:ZENERsmall
Connections:
- net ADC-Clamp-2: now also D6.2 (A)
- net ADC-Clamp-3: now also D2.2 (A)
- net ADC-Clamp-4: now also D10.2 (A)
- net ADC-Clamp-5: now also D4.2 (A)
- net ADC-Clamp-6: now also D16.2 (A)
- net ADC-Clamp-7: now also D8.2 (A)
- net Clamp-18: now also D12.2 (A)
- net Clamp-19: now also D18.2 (A)
- net GND: now also D12.1 (K), D18.1 (K)
- net SigRtn: now also D10.1 (K), D16.1 (K), D2.1 (K), D4.1 (K), D6.1 (K), D8.1 (K)

Commit message: Add files via upload
Connections:
- net ADC-Clamp-2: now also D6.1 (K); no longer D6.2 (A)
- net ADC-Clamp-3: now also D2.1 (K); no longer D2.2 (A)
- net ADC-Clamp-4: now also D10.1 (K); no longer D10.2 (A)
- net ADC-Clamp-5: now also D4.1 (K); no longer D4.2 (A)
- net ADC-Clamp-6: now also D16.1 (K); no longer D16.2 (A)
- net ADC-Clamp-7: now also D8.1 (K); no longer D8.2 (A)
- net Clamp-18: now also D12.1 (K); no longer D12.2 (A)
- net Clamp-19: now also D18.1 (K); no longer D18.2 (A)
- net GND: now also D12.2 (A), D18.2 (A); no longer D12.1 (K), D18.1 (K)
- net SigRtn: now also D10.2 (A), D16.2 (A), D2.2 (A), D4.2 (A), D6.2 (A), D8.2 (A); no longer D10.1 (K), D16.1 (K), D2.1 (K), D4.1 (K), D6.1 (K), D8.1 (K)
Other:
- note added: "5.1V 500mA"
- note added: "NOTE! SigRtn is the dedicated ADC return grounded at one point only."
Changed lines of the file:
@@
 U 1 1 638CFCC2
 P 8300 1400
-F 0 "D2" H 8300 1200 50  0000 C CNN
-F 1 "1N5231B" H 8300 1300 50  0000 C CNN
+F 0 "D2" H 8300 1600 50  0000 C CNN
+F 1 "1N5231B" H 8300 1500 50  0000 C CNN
 F 2 "Diode_THT:D_DO-41_SOD81_P10.16mm_Horizontal" H 8300 1400 50  0001 C CNN
 F 3 "" H 8300 1400 50  0000 C CNN
 	1    8300 1400
-	-1   0    0    -1
+	1    0    0    1
 $EndComp
 $Comp
@@
 U 1 1 638DABDC
 P 8300 2200
-F 0 "D4" H 8300 2000 50  0000 C CNN
-F 1 "1N5231B" H 8300 2100 50  0000 C CNN
+F 0 "D4" H 8300 2400 50  0000 C CNN
+F 1 "1N5231B" H 8300 2300 50  0000 C CNN
 F 2 "Diode_THT:D_DO-41_SOD81_P10.16mm_Horizontal" H 8300 2200 50  0001 C CNN
 F 3 "" H 8300 2200 50  0000 C CNN
 	1    8300 2200
-	-1   0    0    -1
+	1    0    0    1
 $EndComp
 $Comp
@@
 U 1 1 638DB002
 P 8300 3000
-F 0 "D6" H 8300 2800 50  0000 C CNN
-F 1 "1N5231B" H 8300 2900 50  0000 C CNN
+F 0 "D6" H 8300 3200 50  0000 C CNN
+F 1 "1N5231B" H 8300 3100 50  0000 C CNN
 F 2 "Diode_THT:D_DO-41_SOD81_P10.16mm_Horizontal" H 8300 3000 50  0001 C CNN
 F 3 "" H 8300 3000 50  0000 C CNN
 	1    8300 3000
-	-1   0    0    -1
+	1    0    0    1
 $EndComp
 $Comp
@@
 U 1 1 638DB36D
 P 8300 3850
-F 0 "D10" H 8300 3650 50  0000 C CNN
-F 1 "1N5231B" H 8300 3750 50  0000 C CNN
+F 0 "D10" H 8300 4050 50  0000 C CNN
+F 1 "1N5231B" H 8300 3950 50  0000 C CNN
 F 2 "Diode_THT:D_DO-41_SOD81_P10.16mm_Horizontal" H 8300 3850 50  0001 C CNN
 F 3 "" H 8300 3850 50  0000 C CNN
 	1    8300 3850
-	-1   0    0    -1
+	1    0    0    1
 $EndComp
 $Comp
@@
 U 1 1 638DB85A
 P 10150 1400
-F 0 "D16" H 10150 1200 50  0000 C CNN
-F 1 "1N5231B" H 10150 1300 50  0000 C CNN
+F 0 "D16" H 10150 1600 50  0000 C CNN
+F 1 "1N5231B" H 10150 1500 50  0000 C CNN
 F 2 "Diode_THT:D_DO-41_SOD81_P10.16mm_Horizontal" H 10150 1400 50  0001 C CNN
 F 3 "" H 10150 1400 50  0000 C CNN
 	1    10150 1400
-	-1   0    0    -1
+	1    0    0    1
 $EndComp
 $Comp
@@
 U 1 1 638DBC04
 P 10150 2200
-F 0 "D8" H 10150 2000 50  0000 C CNN
-F 1 "1N5231B" H 10150 2100 50  0000 C CNN
+F 0 "D8" H 10150 2400 50  0000 C CNN
+F 1 "1N5231B" H 10150 2300 50  0000 C CNN
 F 2 "Diode_THT:D_DO-41_SOD81_P10.16mm_Horizontal" H 10150 2200 50  0001 C CNN
 F 3 "" H 10150 2200 50  0000 C CNN
 	1    10150 2200
-	-1   0    0    -1
+	1    0    0    1
 $EndComp
 $Comp
@@
 U 1 1 638DBE45
 P 10150 3000
-F 0 "D12" H 10150 2800 50  0000 C CNN
-F 1 "1N5231B" H 10150 2900 50  0000 C CNN
+F 0 "D12" H 10150 3200 50  0000 C CNN
+F 1 "1N5231B" H 10150 3100 50  0000 C CNN
 F 2 "Diode_THT:D_DO-41_SOD81_P10.16mm_Horizontal" H 10150 3000 50  0001 C CNN
 F 3 "" H 10150 3000 50  0000 C CNN
 	1    10150 3000
-	-1   0    0    -1
+	1    0    0    1
 $EndComp
 $Comp
@@
 U 1 1 638DC05A
 P 10150 3850
-F 0 "D18" H 10150 3650 50  0000 C CNN
-F 1 "1N5231B" H 10150 3750 50  0000 C CNN
+F 0 "D18" H 10150 4050 50  0000 C CNN
+F 1 "1N5231B" H 10150 3950 50  0000 C CNN
 F 2 "Diode_THT:D_DO-41_SOD81_P10.16mm_Horizontal" H 10150 3850 50  0001 C CNN
 F 3 "" H 10150 3850 50  0000 C CNN
 	1    10150 3850
-	-1   0    0    -1
+	1    0    0    1
 $EndComp
 Text GLabel 8600 1400 2    50   Input ~ 0
@@
 	0    -1   -1   0
 $EndComp
+Text Notes 8400 1600 0    50   ~ 0
+5.1V 500mA
+Text Notes 10250 1600 0    50   ~ 0
+5.1V 500mA
+Text Notes 8400 2400 0    50   ~ 0
+5.1V 500mA
+Text Notes 10250 2400 0    50   ~ 0
+5.1V 500mA
+Text Notes 10250 3200 0    50   ~ 0
+5.1V 500mA
+Text Notes 8400 3200 0    50   ~ 0
+5.1V 500mA
+Text Notes 8400 4050 0    50   ~ 0
+5.1V 500mA
+Text Notes 10250 4050 0    50   ~ 0
+5.1V 500mA
+Text Notes 7450 700  0    50   ~ 0
+NOTE! SigRtn is the dedicated ADC return grounded at one point only.
 $EndSCHEMATC
