File: KiCad Files/DP1600i/file63700915.sch (KiCad schematic (older format))
At the start: 1 part, among them J1 DB25_Female

Commit message: Add files via upload
Parts:
- J1: value DB25_Female -> DB25_Male; footprint Connector_Dsub:DSUB-25_Female_Horizontal_P2.77x2.84mm_EdgePinOffset4.94mm_Housed_MountingHolesOffset7.48mm -> Connector_Dsub:DSUB-25_Male_Horizontal_P2.77x2.84mm_EdgePinOffset4.94mm_Housed_MountingHolesOffset7.48mm
Connections:
- net CLT_Sensor: now also J1.15 (P15); no longer J1.14 (P14)
- net IAT_Sensor: now also J1.3; no longer J1.1
- net O2_Sensor: now also J1.14 (P14); no longer J1.2
- net Spare-ADC: now also J1.1; no longer J1.3
- net TPS_Sensor: now also J1.2; no longer J1.15 (P15)
Changed lines of the file:
@@
 P 5800 3400
 F 0 "J1" H 5980 3446 50  0000 L CNN
-F 1 "DB25_Female" H 5980 3355 50  0000 L CNN
-F 2 "Connector_Dsub:DSUB-25_Female_Horizontal_P2.77x2.84mm_EdgePinOffset4.94mm_Housed_MountingHolesOffset7.48mm" H 5800 3400 50  0001 C CNN
+F 1 "DB25_Male" H 5980 3355 50  0000 L CNN
+F 2 "Connector_Dsub:DSUB-25_Male_Horizontal_P2.77x2.84mm_EdgePinOffset4.94mm_Housed_MountingHolesOffset7.48mm" H 5800 3400 50  0001 C CNN
 F 3 " ~" H 5800 3400 50  0001 C CNN
 	1    5800 3400
 	-1   0    0    1
 $EndComp
-Text GLabel 6350 4600 2    50   Input ~ 0
-IAT_Sensor
 Text GLabel 7000 4500 2    50   Input ~ 0
-CLT_Sensor
+O2_Sensor
 Text GLabel 6350 4400 2    50   Input ~ 0
-O2_Sensor
-Text GLabel 7000 4300 2    50   Input ~ 0
 TPS_Sensor
 Text GLabel 7000 4100 2    50   Input ~ 0
@@
 Wire Wire Line
 	6100 4600 6350 4600
-Wire Wire Line
-	6100 4500 7000 4500
 Wire Wire Line
 	6100 4400 6350 4400
@@
 Text GLabel 7000 3600 2    50   Input ~ 0
 MCU-D18
-Text GLabel 6350 4200 2    50   Input ~ 0
+Text GLabel 6350 4600 2    50   Input ~ 0
 Spare-ADC
 Wire Wire Line
@@
 Text Notes 7350 4150 0    50   ~ 0
 Sensor ground
-Text Notes 6850 4250 0    50   ~ 0
+Text Notes 6850 4650 0    50   ~ 0
 Spare ADC
+Text Notes 6850 4450 0    50   ~ 0
+Throttle Position Sensor
+Text Notes 7450 4550 0    50   ~ 0
+Wide Band O2 sensor
 Text Notes 7500 4350 0    50   ~ 0
-Throttle Position Sensor
-Text Notes 6800 4450 0    50   ~ 0
-Wide Band O2 sensor
-Text Notes 7500 4550 0    50   ~ 0
 Cylinder head temperaure
-Text Notes 6850 4650 0    50   ~ 0
-Inlet Air Temperature
 NoConn ~ 6100 3900
 Wire Wire Line
@@
 Text Notes 5400 5150 0    50   ~ 0
 Common ground
+Text Notes 6850 4250 0    50   ~ 0
+Inlet Air Temperature
+Wire Wire Line
+	6100 4500 7000 4500
+Text GLabel 7000 4300 2    50   Input ~ 0
+CLT_Sensor
+Text GLabel 6350 4200 2    50   Input ~ 0
+IAT_Sensor
 $EndSCHEMATC

Commit message: Add files via upload
Parts:
- added J10: Conn_01x01, DP1600i:Jumper-Pad, symbol Connector_Generic:Conn_01x01
- added J11, J12, J13, J14, J15, J16, J17, J18: Conn_01x05, Connector_PinHeader_2.54mm:PinHeader_1x05_P2.54mm_Vertical, symbol Connector_Generic:Conn_01x05
- added J19, J20: Conn_01x23, Connector_PinHeader_2.54mm:PinHeader_1x23_P2.54mm_Vertical, symbol Connector_Generic:Conn_01x23
- added J21, J22, J23: Conn_01x17, Connector_PinHeader_2.54mm:PinHeader_1x17_P2.54mm_Vertical, symbol Connector_Generic:Conn_01x17
- added J24, J25: Conn_01x10, Connector_PinHeader_2.54mm:PinHeader_1x10_P2.54mm_Vertical, symbol Connector_Generic:Conn_01x10
- added J26, J27: Conn_01x09, Connector_PinHeader_2.54mm:PinHeader_1x09_P2.54mm_Vertical, symbol Connector_Generic:Conn_01x09
- added J28: Conn_01x01, Connector_PinHeader_2.54mm:PinHeader_1x01_P2.54mm_Vertical, symbol Connector_Generic:Conn_01x01
- added J29: Conn_01x02, Connector_PinHeader_2.54mm:PinHeader_1x02_P2.54mm_Vertical, symbol Connector_Generic:Conn_01x02
- added J30: Conn_01x03, Connector_PinHeader_2.54mm:PinHeader_1x03_P2.54mm_Vertical, symbol Connector_Generic:Conn_01x03
- added J31: Conn_01x04, Connector_PinHeader_2.54mm:PinHeader_1x04_P2.54mm_Vertical, symbol Connector_Generic:Conn_01x04
Connections:
- net 12V: now also J11.2 (Pin_2); no longer J1.13
- net GND: now also J11.5 (Pin_5); no longer J1.16 (P16)
- net VDDA: now also J11.4 (Pin_4)
- net at J1.17 (P17): now also J10.1 (Pin_1)
- new net 12V-Raw: J1.13
- new net SigRtn: J1.16 (P16), J11.1 (Pin_1)
- new net VDD: J11.3 (Pin_3)
- no-connect marks 1 -> 180
Other:
- note added: "Jumper pad"
- note added: "Proto header 1"
- note added: "Proto header 10\n\n"
- note added: "Proto header 11\n\n"
- note added: "Proto header 12\n\n"
- note added: "Proto header 13\n\n\n"
- note added: "Proto header 14\n\n\n"
- note added: "Proto header 15\n\n\n"
- note added: "Proto header 16\n\n\n"
- note added: "Proto header 17\n\n\n"
- note added: "Proto header 2"
- note added: "Proto header 3"
- note added: "Proto header 4"
- note added: "Proto header 5"
- note added: "Proto header 6"
- note added: "Proto header 7"
- note added: "Proto header 8"
- note added: "Proto header 9\n"

Commit message: Add files via upload
Parts:
- removed J10: Conn_01x01, DP1600i:Jumper-Pad, symbol Connector_Generic:Conn_01x01
Connections:
- net VDD: now also J1.17 (P17)
Other:
- note added: "5 volt"
- note added: "5V ADC"
- note removed: "5 volt ADC"
- note removed: "Jumper pad"
Changed lines of the file:
@@
 SigRtn
-$Comp
-L power:VDDA #PWR042
-U 1 1 638C6550
-P 6350 4000
-F 0 "#PWR042" H 6350 3850 50  0001 C CNN
-F 1 "VDDA" V 6368 4128 50  0000 L CNN
-F 2 "" H 6350 4000 50  0001 C CNN
-F 3 "" H 6350 4000 50  0001 C CNN
-	1    6350 4000
-	0    1    1    0
-$EndComp
 $Comp
 L power:GND #PWR041
@@
 Text Notes 6650 3850 0    50   ~ 0
 Common ground
-Text Notes 6700 4050 0    50   ~ 0
-5 volt ADC
 Text Notes 7350 4150 0    50   ~ 0
 Sensor ground
@@
 Wire Wire Line
 	6100 4200 6350 4200
-Wire Wire Line
-	6100 4100 7000 4100
 Text Notes 6850 4250 0    50   ~ 0
 Inlet Air Temperature
@@
 Text GLabel 6350 4200 2    50   Input ~ 0
 IAT_Sensor
-$Comp
-L Connector_Generic:Conn_01x01 J10
-U 1 1 63818FB5
-P 7200 3900
-F 0 "J10" H 7300 3900 50  0000 L CNN
-F 1 "Conn_01x01" H 7450 3900 50  0000 L CNN
-F 2 "DP1600i:Jumper-Pad" H 7200 3900 50  0001 C CNN
-F 3 "~" H 7200 3900 50  0001 C CNN
-	1    7200 3900
-	1    0    0    -1
-$EndComp
 Wire Wire Line
 	6100 3900 7000 3900
-Text Notes 7950 3950 0    50   ~ 0
-Jumper pad
+Text Notes 6700 4050 0    50   ~ 0
+5V ADC
 $Comp
 L Connector_Generic:Conn_01x05 J11
@@
 NoConn ~ 1850 2600
 NoConn ~ 1750 2600
+$Comp
+L power:VDD #PWR?
+U 1 1 63860120
+P 7000 3900
+F 0 "#PWR?" H 7000 3750 50  0001 C CNN
+F 1 "VDD" V 7015 4028 50  0000 L CNN
+F 2 "" H 7000 3900 50  0001 C CNN
+F 3 "" H 7000 3900 50  0001 C CNN
+	1    7000 3900
+	0    1    1    0
+$EndComp
+Wire Wire Line
+	6100 4100 7000 4100
+Text Notes 7300 3950 0    50   ~ 0
+5 volt
+$Comp
+L power:VDDA #PWR?
+U 1 1 63898C7D
+P 6350 4000
+F 0 "#PWR?" H 6350 3850 50  0001 C CNN
+F 1 "VDDA" V 6365 4128 50  0000 L CNN
+F 2 "" H 6350 4000 50  0001 C CNN
+F 3 "" H 6350 4000 50  0001 C CNN
+	1    6350 4000
+	0    1    1    0
+$EndComp
 $EndSCHEMATC

Commit message: Add files via upload
Other:
- note added: "DB25 connections to DP1600iAuxBot board"
- note added: "Proto board connections\n"
- note removed: "Connections to Aux board"
Changed lines of the file:
@@
 	0    -1   -1   0
 $EndComp
-Text Notes 5550 1750 0    100  ~ 0
-Connections to Aux board
+Text Notes 5150 1900 0    100  ~ 0
+DB25 connections to DP1600iAuxBot board
 Wire Wire Line
 	6350 4000 6100 4000
@@
 	0    1    1    0
 $EndComp
+Text Notes 1200 750  0    100  ~ 0
+Proto board connections\n
 $EndSCHEMATC

Commit message: Add files via upload
Parts:
- removed J11, J12, J13, J14, J15, J16, J17, J18: Conn_01x05, Connector_PinHeader_2.54mm:PinHeader_1x05_P2.54mm_Vertical, symbol Connector_Generic:Conn_01x05
- removed J19, J20: Conn_01x23, Connector_PinHeader_2.54mm:PinHeader_1x23_P2.54mm_Vertical, symbol Connector_Generic:Conn_01x23
- removed J21, J22, J23: Conn_01x17, Connector_PinHeader_2.54mm:PinHeader_1x17_P2.54mm_Vertical, symbol Connector_Generic:Conn_01x17
- removed J24, J25: Conn_01x10, Connector_PinHeader_2.54mm:PinHeader_1x10_P2.54mm_Vertical, symbol Connector_Generic:Conn_01x10
- removed J26, J27: Conn_01x09, Connector_PinHeader_2.54mm:PinHeader_1x09_P2.54mm_Vertical, symbol Connector_Generic:Conn_01x09
- removed J28: Conn_01x01, Connector_PinHeader_2.54mm:PinHeader_1x01_P2.54mm_Vertical, symbol Connector_Generic:Conn_01x01
- removed J29: Conn_01x02, Connector_PinHeader_2.54mm:PinHeader_1x02_P2.54mm_Vertical, symbol Connector_Generic:Conn_01x02
- removed J30: Conn_01x03, Connector_PinHeader_2.54mm:PinHeader_1x03_P2.54mm_Vertical, symbol Connector_Generic:Conn_01x03
- removed J31: Conn_01x04, Connector_PinHeader_2.54mm:PinHeader_1x04_P2.54mm_Vertical, symbol Connector_Generic:Conn_01x04
Connections:
- no-connect marks 180 -> 0
Other:
- note removed: "Proto board connections\n"
- note removed: "Proto header 1"
- note removed: "Proto header 10\n\n"
- note removed: "Proto header 11\n\n"
- note removed: "Proto header 12\n\n"
- note removed: "Proto header 13\n\n\n"
- note removed: "Proto header 14\n\n\n"
- note removed: "Proto header 15\n\n\n"
- note removed: "Proto header 16\n\n\n"
- note removed: "Proto header 17\n\n\n"
- note removed: "Proto header 2"
- note removed: "Proto header 3"
- note removed: "Proto header 4"
- note removed: "Proto header 5"
- note removed: "Proto header 6"
- note removed: "Proto header 7"
- note removed: "Proto header 8"
- note removed: "Proto header 9\n"
