File: KiCad Files/DP1600i/file63700A4D.sch (KiCad schematic (older format))
At the start: 21 parts, among them U4 IXDI604PI, U5 IXDI604PI, U6 IXDI604PI, U7 IXDI604PI, U8 IXDI604PI, U9 ULN2003

Commit message: Add files via upload
Parts:
- U9: value ULN2003 -> ULN2004AN; footprint Package_DIP:DIP-10_W7.62mm -> Package_DIP:DIP-16_W7.62mm
Changed lines of the file:
@@
 AR Path="/637A4EA7/6495AC6B" Ref="U?"  Part="1"
 F 0 "U9" H 2900 7217 50  0000 C CNN
-F 1 "ULN2003" H 2900 7126 50  0000 C CNN
-F 2 "Package_DIP:DIP-10_W7.62mm" H 2950 6000 50  0001 L CNN
+F 1 "ULN2004AN" H 2900 7126 50  0000 C CNN
+F 2 "Package_DIP:DIP-16_W7.62mm" H 2950 6000 50  0001 L CNN
 F 3 "http://www.ti.com/lit/ds/symlink/uln2003a.pdf" H 3000 6350 50  0001 C CNN
 F 4 "296-16971-5-ND" H 2900 6550 50  0001 C CNN "Digikey Part Number"

Commit message: Add files via upload
Parts:
- added J87: Pin D4, DP1600i:Jumper-Pad, symbol Connector_Generic:Conn_01x01
- added J88: Pin D3, DP1600i:Jumper-Pad, symbol Connector_Generic:Conn_01x01
- added J89: Pin D2, DP1600i:Jumper-Pad, symbol Connector_Generic:Conn_01x01
- added J90: Pin D1, DP1600i:Jumper-Pad, symbol Connector_Generic:Conn_01x01
- added J91: Pin D0, DP1600i:Jumper-Pad, symbol Connector_Generic:Conn_01x01
- added J92: D7 out, DP1600i:Jumper-Pad, symbol Connector_Generic:Conn_01x01
- added J93: D6 out, DP1600i:Jumper-Pad, symbol Connector_Generic:Conn_01x01
- added J94: D5 out, DP1600i:Jumper-Pad, symbol Connector_Generic:Conn_01x01
- added J95: Step 2B, DP1600i:Jumper-Pad, symbol Connector_Generic:Conn_01x01
- added J96: Step 2A, DP1600i:Jumper-Pad, symbol Connector_Generic:Conn_01x01
- added J97: Step 1A, DP1600i:Jumper-Pad, symbol Connector_Generic:Conn_01x01
- added J98: Step 1B, DP1600i:Jumper-Pad, symbol Connector_Generic:Conn_01x01
- added U10: A4988StepStick, BPEM488CWaux:A4988StepStick, symbol a4988stepstick:A4988StepStick
Connections:
- net 12V: now also U10.16 (V_Mot)
- net GND: now also U10.15 (Mot_Gnd), U10.9 (Gnd)
- net VDD: now also U10.10 (VDD)
- net at U9.12 (O5): now also J94.1 (Pin_1)
- net at U9.13 (O4): now also J93.1 (Pin_1)
- net at U9.14 (O3): now also J92.1 (Pin_1)
- net MCU-D7: now reaches U9.3 (I3)
- net MCU-D6: now reaches U9.4 (I4)
- net MCU-D5: now reaches U9.5 (I5)
- new net: J98.1 (Pin_1), U10.11 (1B)
- new net: J97.1 (Pin_1), U10.12 (1A)
- new net: J96.1 (Pin_1), U10.13 (2A)
- new net: J95.1 (Pin_1), U10.14 (2B)
- new net: U10.5 (Reset), U10.6 (Sleep)
- new net MCU-D0: J91.1 (Pin_1)
- new net MCU-D1: J90.1 (Pin_1)
- new net MCU-D16: U10.8 (Dir)
- new net MCU-D17: U10.7 (Step)
- new net MCU-D2: J89.1 (Pin_1)
- new net MCU-D3: J88.1 (Pin_1)
- new net MCU-D4: J87.1 (Pin_1)
- no-connect marks 20 -> 18

Commit message: Add files via upload
Other:
- note added: "High current output drivers control"
- note added: "Low current outputs and control"
- note added: "Stepper motor idle control"
- moved on the sheet: C30, J95, J96, J97, J98, R23, R24, U10, U8

Commit message: Add files via upload
Parts:
- U4, U5, U6, U7, U8: value IXDI604PI -> IXDNI604PI
Other:
- note added: "MCU-D48 (ASD Relay)) Pin default Low, Hi to energise relay, Lo to de-energise relay."
- note added: "MCU-D51 (Ign1) Pin default Low, Hi to energise coil, Lo to de-energise coil."
- note added: "MCU-D52 (Ign2) Pin default Low, Hi to energise coil, Lo to de-energise coil."
- note added: "MCU-D8 (Inj1) Pin default Low, Hi to energise injector, Lo to de-energise injector."
- note added: "MCU-D9 (Inj2) Pin default Low, Hi to energise injector, Lo to de-energise injector."
- note added: "eMCU-D49 (Tachometer) Pin default Low, Goes Hi after boot sequence.\nGoes Lo at start of dwell, goes Hi at end of dwell."
- moved on the sheet: C30, J87, J88, J89, J90, J91, J92, J93, J94, J95, J96, J97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

Commit message: Add files via upload
Parts:
- removed C28, C29, C30: 0.1uF, Capacitor_THT:C_Disc_D5.0mm_W2.5mm_P2.50mm, symbol Device:C
- removed U4, U5, U6, U7, U8: IXDNI604PI, Package_DIP:DIP-8_W7.62mm, symbol V10-Ign-Inj-Drivers-V2-rescue:IXDI604PI
- added C3: .01uF, Capacitor_THT:C_Disc_D5.0mm_W2.5mm_P2.50mm, symbol Device:C
- added C4: 1uF, Capacitor_THT:C_Disc_D5.0mm_W2.5mm_P2.50mm, symbol Device:C
- added R25, R26, R27, R28, R29, R30, R37, R38, R39, R40: 100K, Resistor_THT:R_Axial_DIN0207_L6.3mm_D2.5mm_P7.62mm_Horizontal, symbol Device:R
- added R31, R32, R33, R34, R35, R36, R41, R42, R43, R44: 1K, Resistor_THT:R_Axial_DIN0207_L6.3mm_D2.5mm_P7.62mm_Horizontal, symbol Device:R
- added U4, U5, U6, U7, U8: IXDNI604PI, Package_DIP:DIP-8_W7.62mm, symbol DP1600i:IXDNI604PI
- C26: value 0.1uF -> .01uF
- C27: value 0.1uF -> 1uF
Connections:
- net 12V: now also C26.2, C27.2, U4.6 (VCC), U6.6 (VCC), U8.6 (VCC)
- net GND: now also C3.1, C4.1, R25.1, R26.1, R27.1, R28.1, R29.1, R30.1, R37.1, R38.1, R39.1, R40.1, U4.3 (Gnd~), U5.3 (Gnd~), U6.3 (Gnd~), U7.3 (Gnd~), U8.3 (Gnd~)
- net MCU-D10: now also R27.2, R33.2
- net MCU-D11: now also R28.2, R34.2
- net MCU-D12: now also R29.2, R35.2
- net MCU-D13: now also R30.2, R36.2
- net MCU-D50: now also R37.2, R41.2
- net MCU-D51: now also R38.2, R42.2
- net MCU-D52: now also R39.2, R43.2
- net MCU-D53: now also R40.2, R44.2
- net MCU-D8: now also R25.2, R31.2
- net MCU-D9: now also R26.2, R32.2
- net VDD: now also C3.2, C4.2, U5.6 (VCC), U7.6 (VCC); no longer C26.2, C27.2
- net MCU-D24: now reaches U10.1 (Enable)
- net at R17.2: now also U4.5 (OUTB)
- net at R15.2: now also U4.7 (OUTA)
- net at R21.2: now also U6.5 (OUTB)
- net at R19.2: now also U6.7 (OUTA)
- net at R24.2: now also U8.5 (OUTB)
- net at R23.2: now also U8.7 (OUTA)
- net at R18.2: now also U5.5 (OUTB)
- net at R16.2: now also U5.7 (OUTA)
- net at R22.2: now also U7.5 (OUTB)
- net at R20.2: now also U7.7 (OUTA)
- new net: R32.1, U4.4 (INB)
- new net: R31.1, U4.2 (INA)
- new net: R41.1, U5.2 (INA)
- new net: R35.1, U8.2 (INA)
- new net: R33.1, U6.2 (INA)
- new net: R34.1, U6.4 (INB)
- new net: R43.1, U7.2 (INA)
- new net: R44.1, U7.4 (INB)
- new net: R42.1, U5.4 (INB)
- new net: R36.1, U8.4 (INB)
- no-connect marks 18 -> 17
Other:
- note added: "(AUIRF3205)"
- note added: "(ISL9V3040P3)"
- note added: "(Optional)"
- moved on the sheet: J87, J88, J89, J90, J95, J96, J97, J98, R15, R16, R17, R18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
