File: KiCad Files/DP1600iAuxTop/file63777FAF.sch (KiCad schematic (older format))
At the start: 51 parts

Commit message: Add files via upload
Parts:
- removed D?: Yellow LED, LED_THT:LED_D3.0mm, symbol Device:LED
- removed J?: DB25_Female, Connector_Dsub:DSUB-25_Female_Horizontal_P2.77x2.84mm_EdgePinOffset4.94mm_Housed_MountingHolesOffset7.48mm, symbol Connector:DB25_Female
- removed J?: Conn_01x01, symbol Connector_Generic:Conn_01x01
- removed R?: 1K, Resistor_THT:R_Axial_DIN0207_L6.3mm_D2.5mm_P7.62mm_Horizontal, symbol Device:R
- J33, J34, J35, J36, J37, J38, J39, J40, J41, J42, J43, J44, J45, J46, J47, J48, J49, J50, J51, J52, J53, J54, J55, J56, J57, J58, J59, J60, J61, J62: renamed from J?; footprint (none) -> Connector_PinHeader_2.54mm:PinHeader_1x01_P2.54mm_Vertical
- R23, R24, R25: renamed from R?; footprint Resistor_THT:R_Axial_DIN0207_L6.3mm_D2.5mm_P7.62mm_Horizontal -> Resistor_THT:R_Axial_DIN0207_L6.3mm_D2.5mm_P10.16mm_Horizontal
- R26, R27: renamed from R?; footprint Resistor_THT:R_Axial_DIN0204_L3.6mm_D1.6mm_P5.08mm_Horizontal -> Resistor_THT:R_Axial_DIN0207_L6.3mm_D2.5mm_P10.16mm_Horizontal
- gave numbers to parts that had none: 12
Connections:
- net VDD: now also D36.1 (K), D38.1 (K), R26.2, R27.2
- net VDDA: no longer D36.1 (K), D38.1 (K), R26.2, R27.2
- net 12V renamed 12V-Raw
- net CKP-VR+ renamed CKP+
- net CKP-VR- renamed CKP-
- net CLT_Sensor renamed CLT-Sensor
- net CMP-VR+ renamed CMP+
- net CMP-VR- renamed CMP-
- net IAT_Sensor renamed IAT-Sensor
- net O2_Sensor renamed O2-Sensor
- net TPS_Sensor renamed TPS-Sensor
Other:
- note removed: "5 volt ADC"
- note removed: "5 volt general"
- note removed: "Common ground"
- note removed: "Connections to DP1600i board"
- moved on the sheet: J33
