File: KiCad Files/DP1600iAuxTop/DP1600iAuxTop.kicad_pcb (KiCad board)
At the start: 2 copper layers, 120.4 x 99.9 mm, 109 parts, among them J1 Conn_01x01, J10 Conn_01x01, J11 Conn_01x01, J12 Conn_01x01, J13 Conn_01x01, J14 Conn_01x01, J15 Conn_01x01, J16 Conn_01x01, J17 Conn_01x01, J18 Conn_01x01, J19 Conn_01x01, J2 Conn_01x01, J20 Conn_01x01, J21 Conn_01x01, J22 Conn_01x01, J23 Conn_01x01, J24 Conn_01x01, J25 Conn_01x01, J26 Screw_Terminal_01x02, J27 Screw_Terminal_01x08, J28 Screw_Terminal_01x06, J29 Screw_Terminal_01x02, J3 Conn_01x01, J30 Screw_Terminal_01x06, J31 Screw_Terminal_01x02, J32 Screw_Terminal_01x07, J4 Conn_01x01, J5 Conn_01x01, J6 Conn_01x01, J7 Conn_01x01, J8 Conn_01x01, J9 Conn_01x01, K1 Main, K2 Automatic Shut Down, Q1 AUIRF3205, Q10 ISL9V3040P3, Q2 AUIRF3205, Q3 AUIRF3205, Q4 AUIRF3205, Q5 AUIRF3205, Q6 AUIRF3205, Q7 ISL9V3040P3, Q8 ISL9V3040P3, Q9 ISL9V3040P3

Commit message: Add files via upload
Parts:
- removed the J19 at (351.8, 108.2)
- removed the J20 at (381.4, 95.2)
- removed the J21 at (377.2, 111.3)
- removed the J22 at (337.6, 118.2)
- removed J24, J25: Conn_01x01, Connector_PinHeader_2.54mm:PinHeader_1x01_P2.54mm_Vertical
- removed J27: Screw_Terminal_01x08, DP1600iAuxTop:Phoenix_1729076
- removed J28: Screw_Terminal_01x06, DP1600iAuxTop:Phoenix_1715190
- added J3: Conn_01x01, Connector_PinHeader_2.54mm:PinHeader_1x01_P2.54mm_Vertical, F.Cu at (229.8, 113.0)
- added J31: Screw_Terminal_01x08, DP1600iAuxTop:Phoenix_1729076_Rt, F.Cu at (220.6, 16.6)
- added J32: Screw_Terminal_01x07, DP1600iAuxTop:Phoenix_1729063_Rt, F.Cu at (217.9, 117.2)
- added J4: Conn_01x01, Connector_PinHeader_2.54mm:PinHeader_1x01_P2.54mm_Vertical, F.Cu at (229.0, 119.3)
- added J5: Conn_01x01, Connector_PinHeader_2.54mm:PinHeader_1x01_P2.54mm_Vertical, F.Cu at (97.3, 77.8)
- added J6: Conn_01x01, Connector_PinHeader_2.54mm:PinHeader_1x01_P2.54mm_Vertical, F.Cu at (99.0, 83.6)
- D10, D11, D12, D13, D2, D22, D23, D24, D25, D26, D27, D28, D29, D4, D5, D6, D7, D8, D9: value DIODE -> 1N4001
- J23: value Conn_01x01 -> Conn_01x07; footprint Connector_PinHeader_2.54mm:PinHeader_1x01_P2.54mm_Vertical -> Connector_PinHeader_2.54mm:PinHeader_1x07_P2.54mm_Vertical
- moved J12 362.0 mm to (30.9, 54.6)
- moved J17 349.3 mm to (33.5, 109.8)
- moved J11 347.2 mm to (31.2, 79.4)
- moved J8 340.7 mm to (32.4, 30.5)
- moved J9 325.8 mm to (32.1, -0.15)
- moved J13 325.5 mm to (69.9, 59.5)
- moved J10 323.8 mm to (78.8, 4.29)
- moved J19 299.3 mm to (70.3, 85.2)
- moved J16 272.3 mm to (78.7, 32.8)
- moved J2 268.1 mm to (111.1, -22.5)
- moved J18 267.3 mm to (77.4, 119.7)
- moved J7 249.2 mm to (125.9, -5.41)
- moved R18 236.0 mm to (125.9, -8.61), turned to 180 degrees
- moved R7 228.7 mm to (121.0, -25.7), turned to 180 degrees
- moved J14 224.6 mm to (148.4, 17.3)
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- renumbered J6 to J10, J7 to J11, J8 to J12, J9 to J13, J10 to J14, J11 to J15, J12 to J16, J13 to J17, J14 to J18, J15 to J19, J16 to J20, J17 to J21, J18 to J22, J26 to J30, J29 to J33, J30 to J34, J31 to J35, J32 to J36, J3 to J7, J4 to J8, J5 to J9
Connections:
- D10 pad 2: F3-out -> F6-out
- D11 pad 2: F3-out -> F6-out
- D12 pad 2: F4-out -> F5-out
- D13 pad 2: F4-out -> F5-out
- D15 pad 1: F7-out -> F3-out
- D16 pad 1: F3-out -> F6-out
- D17 pad 1: F3-out -> F6-out
- D18 pad 1: F4-out -> F5-out
- D19 pad 1: F4-out -> F5-out
- D26 pad 2: F5-out -> F7-out
- D27 pad 2: F6-out -> F4-out
- D28 pad 2: F5-out -> F7-out
- D29 pad 2: F6-out -> F4-out
- D30 pad 1: F5-out -> F7-out
- D31 pad 1: F5-out -> F7-out
- D32 pad 1: F6-out -> F4-out
- D33 pad 1: F6-out -> F4-out
- D9 pad 2: F7-out -> F3-out
- J23 pad 1: O2-Sensor -> VDDA
- J33 pad 1: F9-out -> F3-out
- J33 pad 2: D13-out -> F4-out
- J34 pad 1: F3-out -> F5-out
- J34 pad 2: D10-out -> D13-out
- J34 pad 3: D11-out -> D52-out
- J34 pad 4: F5-out -> D53-out
- J34 pad 5: D52-out -> D10-out
- J34 pad 6: D53-out -> D11-out
- J36 pad 1: IAT-Sensor -> VDDA
- J36 pad 2: CLT-Sensor -> SigRtn
- J36 pad 3: TPS-Sensor -> IAT-Sensor
- J36 pad 4: VDDA -> CLT-Sensor
- J36 pad 5: SigRtn -> TPS-Sensor
Routing:
- net F5-out: track 0.00 -> 103.9 mm
- net F4-out: track 0.00 -> 96.3 mm
- net F3-out: track 0.00 -> 85.1 mm
- net Net-(F3-Pad1): track 0.00 -> 66.8 mm
- net F6-out: track 0.00 -> 52.1 mm
- net F7-out: track 0.00 -> 44.2 mm
- net F9-out: track 0.00 -> 41.8 mm
- net Bat+s: track 0.00 -> 40.6 mm
- net F8-out: track 0.00 -> 38.3 mm
- net Net-(D34-Pad1): track 0.00 -> 21.8 mm
- net Bat+: track 0.00 -> 8.79 mm
- net Net-(F1-Pad1): track 0.00 -> 7.52 mm

Commit message: Add files via upload
Parts:
- removed D2, D22, D23, D24, D25, D4, D5, D6, D7: 1N4001, Diode_THT:D_DO-41_SOD81_P10.16mm_Horizontal
- removed D3: DIODE, Diode_THT:D_DO-41_SOD81_P10.16mm_Horizontal
- removed J10, J11, J12, J14, J15, J16, J17, J18, J19, J2, J21, J22, J3, J4, J6, J7, J8, J9: Conn_01x01, Connector_PinHeader_2.54mm:PinHeader_1x01_P2.54mm_Vertical
- removed R1, R14, R15, R16, R17, R2, R3, R4, R5, R6: 10M, Resistor_THT:R_Axial_DIN0207_L6.3mm_D2.5mm_P10.16mm_Horizontal
- J1: value Conn_01x01 -> Conn_01x10; footprint Connector_PinHeader_2.54mm:PinHeader_1x01_P2.54mm_Vertical -> Connector_PinHeader_2.54mm:PinHeader_1x10_P2.54mm_Vertical
- J13: value Conn_01x01 -> Conn_01x06; footprint Connector_PinHeader_2.54mm:PinHeader_1x01_P2.54mm_Vertical -> Connector_PinHeader_2.54mm:PinHeader_1x06_P2.54mm_Vertical
- J20: value Conn_01x01 -> Conn_01x03; footprint Connector_PinHeader_2.54mm:PinHeader_1x01_P2.54mm_Vertical -> Connector_PinHeader_2.54mm:PinHeader_1x03_P2.54mm_Vertical
- J23: value Conn_01x07 -> Conn_01x09; footprint Connector_PinHeader_2.54mm:PinHeader_1x07_P2.54mm_Vertical -> Connector_PinHeader_2.54mm:PinHeader_1x09_P2.54mm_Vertical
- J5: value Conn_01x01 -> Conn_01x02; footprint Connector_PinHeader_2.54mm:PinHeader_1x01_P2.54mm_Vertical -> Connector_PinHeader_2.54mm:PinHeader_1x02_P2.54mm_Vertical
- Q1, Q10, Q2, Q3, Q4, Q5, Q6, Q7, Q8, Q9: footprint Package_TO_SOT_THT:TO-220-3_Vertical -> Buggly Gruesome AuxTop:TO-220-3_Vertical_Wide
- moved D32 169.4 mm to (165.0, 121.3), turned to 90 degrees
- moved D1 168.5 mm to (210.7, 118.7), turned to 270 degrees
- moved R7 167.5 mm to (210.8, 115.6), turned to 90 degrees
- moved D33 156.9 mm to (171.6, 121.3), turned to 90 degrees
- moved R21 156.5 mm to (164.9, 105.5), turned to 270 degrees
- moved D19 153.5 mm to (158.5, 121.3), turned to 90 degrees
- moved D17 150.3 mm to (197.6, 121.3), turned to 90 degrees
- moved D18 148.2 mm to (152.1, 121.3), turned to 90 degrees
- moved D31 148.0 mm to (184.6, 121.3), turned to 90 degrees
- moved D30 141.4 mm to (178.1, 121.3), turned to 90 degrees
- moved R22 141.2 mm to (171.6, 105.5), turned to 270 degrees
- moved D15 141.0 mm to (145.6, 121.3), turned to 90 degrees
- moved R13 137.2 mm to (158.6, 105.4), turned to 270 degrees
- moved D16 135.3 mm to (191.1, 121.3), turned to 90 degrees
- moved D14 134.2 mm to (204.1, 121.3), turned to 90 degrees
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Connections:
- D30 pad 2: Net-(D22-Pad1) -> Net-(D30-Pad2)
- D31 pad 2: Net-(D23-Pad1) -> Net-(D31-Pad2)
- D32 pad 2: Net-(D24-Pad1) -> Net-(D32-Pad2)
- D33 pad 2: Net-(D25-Pad1) -> Net-(D33-Pad2)
- J1 pad 1: F7-out -> GND
- J13 pad 1: D13-control -> D48-control
- J23 pad 1: VDDA -> Tachometer
- J23 pad 2: SigRtn -> 12V-Raw
- J23 pad 3: IAT-Sensor -> VDDA
- J23 pad 4: CLT-Sensor -> SigRtn
- J23 pad 5: TPS-Sensor -> IAT-Sensor
- J23 pad 6: O2-Sensor -> CLT-Sensor
- J23 pad 7: Spare-ADC -> TPS-Sensor
- J32 pad 2: D9-out -> D12-out
- J32 pad 3: D12-out -> D9-out
- J34 pad 3: D52-out -> D10-out
- J34 pad 4: D53-out -> D11-out
- J34 pad 5: D10-out -> D52-out
- J34 pad 6: D11-out -> D53-out
- R10 pad 2: Net-(D4-Pad2) -> Net-(D16-Pad2)
- R11 pad 2: Net-(D5-Pad2) -> Net-(D17-Pad2)
- R12 pad 2: Net-(D6-Pad2) -> Net-(D18-Pad2)
- R13 pad 2: Net-(D7-Pad2) -> Net-(D19-Pad2)
- R19 pad 2: Net-(D22-Pad2) -> Net-(D30-Pad2)
- R20 pad 2: Net-(D23-Pad2) -> Net-(D31-Pad2)
- R21 pad 2: Net-(D24-Pad2) -> Net-(D32-Pad2)
- R22 pad 2: Net-(D25-Pad2) -> Net-(D33-Pad2)
- R8 pad 2: Net-(D2-Pad2) -> Net-(D14-Pad2)
- R9 pad 2: Net-(D3-Pad2) -> Net-(D15-Pad2)
Routing:
- net Net-(D34-Pad1): track 21.8 -> 202.1 mm, vias 0 -> 1
- net F7-out: track 44.2 -> 224.5 mm, vias 0 -> 5
- net Net-(F3-Pad1): track 66.8 -> 223.1 mm
- net D50-out: track 0.00 -> 151.5 mm, vias 0 -> 1
- net F4-out: track 96.3 -> 246.2 mm, vias 0 -> 5
- net D52-out: track 0.00 -> 140.2 mm, vias 0 -> 1
- net D11-out: track 0.00 -> 137.3 mm, vias 0 -> 1
- net D10-out: track 0.00 -> 133.3 mm, vias 0 -> 1
- net D13-out: track 0.00 -> 128.6 mm, vias 0 -> 1
- net D51-out: track 0.00 -> 127.7 mm, vias 0 -> 1
- net D8-out: track 0.00 -> 101.3 mm
- net Tachometer: track 0.00 -> 99.0 mm
- net F5-out: track 103.9 -> 198.3 mm, vias 0 -> 6
- net D53-out: track 0.00 -> 87.6 mm
- net F3-out: track 85.1 -> 163.0 mm, vias 0 -> 5
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- added copper zone on B.Cu, net GND
- added copper zone on F.Cu, net GND

Commit message: Add files via upload
Connections:
- D14 pad 1: F7-out -> F9-out
- D8 pad 2: F7-out -> F9-out
- J1 pad 5: F7-out -> F9-out
Routing:
- net F9-out: track 46.1 -> 185.7 mm, vias 0 -> 3
- net F7-out: track 224.5 -> 175.7 mm, vias 5 -> 3
- net GND: vias 53 -> 54

Commit message: Add files via upload
Parts:
- added D2: LED, LED_THT:LED_D5.0mm, F.Cu at (208.4, 53.3)
- added R1: 1K, Resistor_THT:R_Axial_DIN0207_L6.3mm_D2.5mm_P2.54mm_Vertical, F.Cu at (204.9, 55.0)
- D20: value ECU -> LED
- moved D20 2.58 mm to (139.0, 118.7), turned to 270 degrees
Connections:
- D20 pad 1: GND -> Net-(D20-Pad1)
- D20 pad 2: Net-(D20-Pad2) -> GND
- R18 pad 2: Net-(D20-Pad2) -> Net-(D20-Pad1)
Routing:
- net Net-(F3-Pad1): track 223.1 -> 236.1 mm
- net Bat+s: track 83.0 -> 90.9 mm
- net F9-out: track 185.7 -> 192.5 mm
- net Net-(D2-Pad1): track 0.00 -> 3.84 mm
- net Net-(D20-Pad2): track 3.08 -> 0.00 mm
- net Net-(D20-Pad1): track 0.00 -> 3.04 mm
Other:
- board text added: "12V-Raw"
- board text added: "Bat+"
- board text added: "Bat+s"
- board text added: "Bat-"
- board text added: "CKP+"
- board text added: "CKP-"
- board text added: "CLT"
- board text added: "CMP+"
- board text added: "CMP-"
- board text added: "D10cntrl"
- board text added: "D10out"
- board text added: "D11cntrl"
- board text added: "D11out"
- board text added: "D12cnt"
- board text added: "D12out"
- board text added: "D13cntrl"
- board text added: "D13out"
- board text added: "D48cntrl"
- board text added: "D50out"
- board text added: "D51out"
- board text added: "D52cnt"
- board text added: "D52cntrl"
- board text added: "D52out"
- board text added: "D53cnt"
- board text added: "D53cntrl"
- board text added: "D53out"
- board text added: "D8cnt"
- board text added: "D8out"
- board text added: "D9cnt"
- board text added: "D9out"
- board text added: "DP1600iAuxTop"
- board text added: "F3out"
- board text added: "F4out"
- board text added: "F5out"
- board text added: "F6out"
- board text added: "F7out"
- board text added: "F8out"
- board text added: "F9out"
- board text added: "Gnd"
- board text added: "IAT"
- board text added: "MADE FOR SPEEDUINO"
- board text added: "O2"
- board text added: "PCB design by Robert Hiebert December 2022"
- board text added: "SigRtn"
- board text added: "Spare"
- board text added: "TPS"
- board text added: "Tachometer"
- board text added: "VDDA"

Commit message: Add files via upload
Parts:
- added RN1: R_Network03_US, Resistor_THT:R_Array_SIP4, F.Cu at (116.8, 49.0)
- added RN2: R_Pack02_SIP, Resistor_THT:R_Array_SIP4, F.Cu at (149.8, 100.1)
- R1, R18: value 1K -> 2.4K
Routing:
- net D10-control: track 14.3 -> 19.4 mm
- net D11-control: track 25.2 -> 30.1 mm
- net D13-control: track 14.9 -> 19.8 mm
- net D9-control: track 34.7 -> 39.3 mm
- net D8-control: track 24.8 -> 29.4 mm
- net F4-out: track 246.2 -> 243.3 mm
