File: KiCad Files/DP1600iAuxTop/DP1600iAuxTop.sch (KiCad schematic (older format))
At the start: 122 parts, among them K1 Main, K2 Automatic Shut Down

Commit message: Add files via upload
Parts:
- removed J? (x3): Conn_01x07, symbol Connector_Generic:Conn_01x07
- removed J?: DB25_Female, Connector_Dsub:DSUB-25_Female_Horizontal_P2.77x2.84mm_EdgePinOffset4.94mm_Housed_MountingHolesOffset7.48mm, symbol Connector:DB25_Female
- removed J? (x4): Conn_01x01, symbol Connector_Generic:Conn_01x01
- removed J? (x2): Conn_01x08, symbol Connector_Generic:Conn_01x08
- removed J?: Conn_01x04, symbol Connector_Generic:Conn_01x04
- removed J?: Conn_01x06, symbol Connector_Generic:Conn_01x06
- removed J?: Conn_01x05, symbol Connector_Generic:Conn_01x05
- D1, D14, D15, D16, D17, D18, D19, D30, D31, D32, D33: renamed from D?; footprint LEDs:LED-3MM -> LED_THT:LED_D5.0mm
- D10, D11, D12, D13, D2, D22, D23, D24, D25, D26, D27, D28, D29, D3, D4, D5, D6, D7, D8, D9: renamed from D?; footprint (none) -> Diode_THT:D_DO-41_SOD81_P10.16mm_Horizontal
- F1, F3, F4, F5, F6, F7, F8, F9: footprint Buggly Gruesome Aux:01530008Z_Fuse_Holder -> DP1600iAuxTop:01530008Z_Fuse_Holder
- J1, J10, J11, J12, J13, J14, J15, J16, J17, J18, J19, J2, J20, J21, J22, J23, J24, J25, J3, J4, J5, J6, J7, J8, J9: renamed from J?; footprint (none) -> Connector_PinHeader_2.54mm:PinHeader_1x01_P2.54mm_Vertical
- J26: renamed from J?; footprint (none) -> DP1600iAuxTop:Phoenix_1714955
- J27: renamed from J?; footprint (none) -> DP1600iAuxTop:Phoenix_1729076
- J28, J30: renamed from J?; footprint (none) -> DP1600iAuxTop:Phoenix_1715190
- J29, J31: renamed from J?; footprint (none) -> DP1600iAuxTop:Phoenix_1730010
- J32: renamed from J?; footprint (none) -> DP1600iAuxTop:Phoenix_1729063
- K1, K2: footprint Buggly Gruesome Aux:Panasonic_CM1-R-12V -> DP1600iAuxTop:VCF4-1000
- Q1, Q10, Q2, Q3, Q4, Q5, Q6, Q7, Q8, Q9: renamed from Q?; footprint TO_SOT_Packages_THT:TO-220_Neutral123_Vertical -> Package_TO_SOT_THT:TO-220-3_Vertical
- R1, R10, R11, R12, R13, R14, R15, R16, R17, R19, R2, R20, R21, R22, R3, R4, R5, R6, R7, R8, R9: renamed from R?; footprint Resistors_ThroughHole:Resistor_Horizontal_RM7mm -> Resistor_THT:R_Axial_DIN0207_L6.3mm_D2.5mm_P10.16mm_Horizontal
- gave numbers to parts that had none: 2
- renumbered D1 to D20, R1 to R18
Connections:
- net labels added: 12V-Raw, CLT-Sensor, O2-Sensor, TPS-Sensor
- net labels removed: 12V, 5V, ASD, Bat-, CKP-VR+, CKP-VR-, CLT-sensor, CLT_Sensor, CMP-VR+, CMP-VR-, HC1-control, HC2-control, HC3-control, HC4-control, HC5-control, HC6-control, IAT_Sensor, LC5-control, LC6-control, LC7-control, LC8-control, MCU-D18, MCU-D19, O2-sensor, O2_Sensor, Sig-Rtn, TPS-sensor, TPS_Sensor
- wire segments 253 -> 217
Other:
- note removed: "5 Volt"
- note removed: "5 volt ADC"
- note removed: "5 volt general"
- note removed: "Automatic Shutdown Relay"
- note removed: "CKP input"
- note removed: "CMP input"
- note removed: "Common ground"
- note removed: "Connections to DP1600i board"
- note removed: "Signal Return"
- note removed: "Spare HC out"
- moved on the sheet: D1, D15, D3, D9, J26, J27, J28, Q2, R2, R7, R9

Commit message: Add files via upload
Parts:
- removed J11, J19, J20, J21, J22, J23, J24, J25: Conn_01x01, Connector_PinHeader_2.54mm:PinHeader_1x01_P2.54mm_Vertical, symbol Connector_Generic:Conn_01x01
- removed J28: Screw_Terminal_01x06, DP1600iAuxTop:Phoenix_1715190, symbol Connector:Screw_Terminal_01x06
- added J23: Conn_01x07, Connector_PinHeader_2.54mm:PinHeader_1x07_P2.54mm_Vertical, symbol Connector_Generic:Conn_01x07
- added J3, J4, J5, J6: Conn_01x01, Connector_PinHeader_2.54mm:PinHeader_1x01_P2.54mm_Vertical, symbol Connector_Generic:Conn_01x01
- added J32: Screw_Terminal_01x07, DP1600iAuxTop:Phoenix_1729063_Rt, symbol Connector:Screw_Terminal_01x07
- D10, D11, D12, D13, D2, D22, D23, D24, D25, D26, D27, D28, D29, D4, D5, D6, D7, D8, D9: value DIODE -> 1N4001
- J31: renamed from J27; footprint DP1600iAuxTop:Phoenix_1729076 -> DP1600iAuxTop:Phoenix_1729076_Rt
- renumbered J6 to J10, J7 to J11, J8 to J12, J9 to J13, J10 to J14, J12 to J16, J13 to J17, J14 to J18, J15 to J19, J16 to J20, J17 to J21, J18 to J22, J26 to J30, J29 to J33, J30 to J34, J31 to J35, J32 to J36, J3 to J7, J4 to J8, J5 to J9
Connections:
- net labels removed: D49-control
- wire segments 217 -> 218

Commit message: Add files via upload
Parts:
- removed D2, D22, D23, D24, D25, D4, D5, D6, D7: 1N4001, Diode_THT:D_DO-41_SOD81_P10.16mm_Horizontal, symbol Simulation_SPICE:DIODE
- removed D3: DIODE, Diode_THT:D_DO-41_SOD81_P10.16mm_Horizontal, symbol Simulation_SPICE:DIODE
- removed J1, J10, J11, J12, J13, J14, J16, J17, J18, J19, J2, J20, J21, J22, J3, J4, J5, J6, J7, J8, J9: Conn_01x01, Connector_PinHeader_2.54mm:PinHeader_1x01_P2.54mm_Vertical, symbol Connector_Generic:Conn_01x01
- removed J23: Conn_01x07, Connector_PinHeader_2.54mm:PinHeader_1x07_P2.54mm_Vertical, symbol Connector_Generic:Conn_01x07
- removed R1, R14, R15, R16, R17, R2, R3, R4, R5, R6: 10M, Resistor_THT:R_Axial_DIN0207_L6.3mm_D2.5mm_P10.16mm_Horizontal, symbol Device:R
- added J1: Conn_01x10, Connector_PinHeader_2.54mm:PinHeader_1x10_P2.54mm_Vertical, symbol Connector_Generic:Conn_01x10
- added J13: Conn_01x06, Connector_PinHeader_2.54mm:PinHeader_1x06_P2.54mm_Vertical, symbol Connector_Generic:Conn_01x06
- added J20: Conn_01x03, Connector_PinHeader_2.54mm:PinHeader_1x03_P2.54mm_Vertical, symbol Connector_Generic:Conn_01x03
- added J23: Conn_01x09, Connector_PinHeader_2.54mm:PinHeader_1x09_P2.54mm_Vertical, symbol Connector_Generic:Conn_01x09
- added J5: Conn_01x02, Connector_PinHeader_2.54mm:PinHeader_1x02_P2.54mm_Vertical, symbol Connector_Generic:Conn_01x02
- Q1, Q10, Q2, Q3, Q4, Q5, Q6, Q7, Q8, Q9: footprint Package_TO_SOT_THT:TO-220-3_Vertical -> Buggly Gruesome AuxTop:TO-220-3_Vertical_Wide
Connections:
- net labels removed: VDD
- wire segments 218 -> 197

Commit message: Add files via upload
Other:
- moved on the sheet: J1, J13, J20, J5
Changed lines of the file:
@@
 Text GLabel 7800 5800 0    50   Input ~ 0
 SigRtn
+Text GLabel 7800 3750 0    50   Input ~ 0
+D51-control
+Text GLabel 7800 3850 0    50   Input ~ 0
+D50-control
+Text GLabel 7800 4600 0    50   Input ~ 0
+D48-control
+Text GLabel 7800 3450 0    50   Input ~ 0
+D12-control
+Text GLabel 7800 4900 0    50   Input ~ 0
+D11-control
+Text GLabel 7800 4800 0    50   Input ~ 0
+D10-control
 Text GLabel 7800 3550 0    50   Input ~ 0
-D51-control
-Text GLabel 7800 3650 0    50   Input ~ 0
-D50-control
-Text GLabel 7800 4400 0    50   Input ~ 0
-D48-control
-Text GLabel 7800 3250 0    50   Input ~ 0
-D12-control
-Text GLabel 7800 4700 0    50   Input ~ 0
-D11-control
-Text GLabel 7800 4600 0    50   Input ~ 0
-D10-control
-Text GLabel 7800 3350 0    50   Input ~ 0
 D9-control
 Text GLabel 7800 5600 0    50   Input ~ 0
 12V-Raw
-Text GLabel 7800 3450 0    50   Input ~ 0
+Text GLabel 7800 3650 0    50   Input ~ 0
 D8-control
 Text Notes 7350 5650 2    50   ~ 0
 12 volt from main relay
-Text Notes 7150 3500 0    50   ~ 0
+Text Notes 7150 3700 0    50   ~ 0
 Inj1
-Text Notes 7150 3400 0    50   ~ 0
+Text Notes 7150 3600 0    50   ~ 0
 Inj2
-Text Notes 7100 4650 0    50   ~ 0
+Text Notes 7100 4850 0    50   ~ 0
 Inj3
-Text Notes 7100 4750 0    50   ~ 0
+Text Notes 7100 4950 0    50   ~ 0
 Inj4
-Text Notes 6900 3300 0    50   ~ 0
+Text Notes 6900 3500 0    50   ~ 0
 PWM Idle
-Text Notes 6600 4450 0    50   ~ 0
+Text Notes 6600 4650 0    50   ~ 0
 ASD relay control
-Text Notes 7100 3700 0    50   ~ 0
+Text Notes 7100 3900 0    50   ~ 0
 Ign1
-Text Notes 7100 3600 0    50   ~ 0
+Text Notes 7100 3800 0    50   ~ 0
 Ign2
 Text Notes 6950 5850 0    50   ~ 0
@@
 L power:GND #PWR?
 U 1 1 63ACA746
-P 7800 2750
+P 7800 2950
 AR Path="/63777FB0/63ACA746" Ref="#PWR?"  Part="1"
 AR Path="/63ACA746" Ref="#PWR017"  Part="1"
-F 0 "#PWR017" H 7800 2500 50  0001 C CNN
-F 1 "GND" V 7805 2622 50  0000 R CNN
-F 2 "" H 7800 2750 50  0001 C CNN
-F 3 "" H 7800 2750 50  0001 C CNN
-	1    7800 2750
+F 0 "#PWR017" H 7800 2700 50  0001 C CNN
+F 1 "GND" V 7805 2822 50  0000 R CNN
+F 2 "" H 7800 2950 50  0001 C CNN
+F 3 "" H 7800 2950 50  0001 C CNN
+	1    7800 2950
 	0    1    1    0
 $EndComp
@@
 L power:GND #PWR?
 U 1 1 63ACA74C
-P 7800 3900
+P 7800 4150
 AR Path="/63777FB0/63ACA74C" Ref="#PWR?"  Part="1"
 AR Path="/63ACA74C" Ref="#PWR016"  Part="1"
-F 0 "#PWR016" H 7800 3650 50  0001 C CNN
-F 1 "GND" V 7805 3772 50  0000 R CNN
-F 2 "" H 7800 3900 50  0001 C CNN
-F 3 "" H 7800 3900 50  0001 C CNN
-	1    7800 3900
+F 0 "#PWR016" H 7800 3900 50  0001 C CNN
+F 1 "GND" V 7805 4022 50  0000 R CNN
+F 2 "" H 7800 4150 50  0001 C CNN
+F 3 "" H 7800 4150 50  0001 C CNN
+	1    7800 4150
 	0    1    1    0
 $EndComp
@@
 	1    0    0    -1
 $EndComp
-Text GLabel 7800 3150 0    50   Input ~ 0
-F7-out
-Text Notes 6600 3200 0    50   ~ 0
+Text GLabel 7800 3350 0    50   Input ~ 0
+F9-out
+Text Notes 6600 3400 0    50   ~ 0
 Tach & WB & Idle +
 Text Notes 5600 5550 0    50   ~ 0
@@
 Connection ~ 5100 1900
 Text GLabel 3000 4200 2    50   Input ~ 0
-F7-out
+F9-out
 Text GLabel 2650 4650 2    50   Input ~ 0
-F7-out
+F9-out
 Text GLabel 3000 5250 2    50   Input ~ 0
 F3-out
@@
 Wire Wire Line
 	6700 5700 7800 5700
-Text GLabel 7800 3050 0    50   Input ~ 0
+Text GLabel 7800 3250 0    50   Input ~ 0
 CKP-
-Text GLabel 7800 2950 0    50   Input ~ 0
+Text GLabel 7800 3150 0    50   Input ~ 0
 CKP+
-Text GLabel 5000 3150 0    50   Input ~ 0
+Text GLabel 7800 2700 0    50   Input ~ 0
 CMP-
-Text GLabel 5000 3050 0    50   Input ~ 0
+Text GLabel 7800 2600 0    50   Input ~ 0
 CMP+
-Text Notes 4300 3200 0    50   ~ 0
+Text Notes 7100 2750 0    50   ~ 0
 CMP VR-
-Text Notes 4300 3100 0    50   ~ 0
+Text Notes 7100 2650 0    50   ~ 0
 CMP VR+
-Text Notes 7450 3100 2    50   ~ 0
+Text Notes 7450 3300 2    50   ~ 0
 CKP VR-
-Text Notes 7450 3000 2    50   ~ 0
+Text Notes 7450 3200 2    50   ~ 0
 CKP VR+
 $Comp
@@
 Wire Wire Line
 	6700 5350 6700 5700
-Text Notes 6250 4550 0    50   ~ 0
+Text Notes 6250 4750 0    50   ~ 0
 Spare high current output
-Text GLabel 7800 4500 0    50   Input ~ 0
+Text GLabel 7800 4700 0    50   Input ~ 0
 D13-control
-Text Notes 7050 4950 0    50   ~ 0
+Text Notes 7050 5150 0    50   ~ 0
 Ign4
-Text Notes 7050 4850 0    50   ~ 0
+Text Notes 7050 5050 0    50   ~ 0
 Ign3
-Text GLabel 7800 4800 0    50   Input ~ 0
+Text GLabel 7800 5000 0    50   Input ~ 0
 D52-control
-Text GLabel 7800 4900 0    50   Input ~ 0
+Text GLabel 7800 5100 0    50   Input ~ 0
 D53-control
 $Comp
 L Connector_Generic:Conn_01x06 J13
 U 1 1 63A44278
-P 8000 4600
-F 0 "J13" V 8100 4500 50  0000 L CNN
-F 1 "Conn_01x06" V 8200 4400 50  0000 L CNN
-F 2 "Connector_PinHeader_2.54mm:PinHeader_1x06_P2.54mm_Vertical" H 8000 4600 50  0001 C CNN
-F 3 "~" H 8000 4600 50  0001 C CNN
-	1    8000 4600
+P 8000 4800
+F 0 "J13" V 8100 4700 50  0000 L CNN
+F 1 "Conn_01x06" V 8200 4600 50  0000 L CNN
+F 2 "Connector_PinHeader_2.54mm:PinHeader_1x06_P2.54mm_Vertical" H 8000 4800 50  0001 C CNN
+F 3 "~" H 8000 4800 50  0001 C CNN
+	1    8000 4800
 	1    0    0    -1
 $EndComp
@@
 L Connector_Generic:Conn_01x02 J5
 U 1 1 63A65D5A
-P 5200 3050
-F 0 "J5" V 5300 2950 50  0000 L CNN
-F 1 "Conn_01x02" V 5400 2800 50  0000 L CNN
-F 2 "Connector_PinHeader_2.54mm:PinHeader_1x02_P2.54mm_Vertical" H 5200 3050 50  0001 C CNN
-F 3 "~" H 5200 3050 50  0001 C CNN
-	1    5200 3050
+P 8000 2600
+F 0 "J5" V 8100 2500 50  0000 L CNN
+F 1 "Conn_01x02" V 8200 2350 50  0000 L CNN
+F 2 "Connector_PinHeader_2.54mm:PinHeader_1x02_P2.54mm_Vertical" H 8000 2600 50  0001 C CNN
+F 3 "~" H 8000 2600 50  0001 C CNN
+	1    8000 2600
 	1    0    0    -1
 $EndComp
@@
 L Connector_Generic:Conn_01x10 J1
 U 1 1 63A66B13
-P 8000 3150
-F 0 "J1" V 8100 3050 50  0000 L CNN
-F 1 "Conn_01x10" V 8200 2950 50  0000 L CNN
-F 2 "Connector_PinHeader_2.54mm:PinHeader_1x10_P2.54mm_Vertical" H 8000 3150 50  0001 C CNN
-F 3 "~" H 8000 3150 50  0001 C CNN
-	1    8000 3150
+P 8000 3350
+F 0 "J1" V 8100 3250 50  0000 L CNN
+F 1 "Conn_01x10" V 8200 3150 50  0000 L CNN
+F 2 "Connector_PinHeader_2.54mm:PinHeader_1x10_P2.54mm_Vertical" H 8000 3350 50  0001 C CNN
+F 3 "~" H 8000 3350 50  0001 C CNN
+	1    8000 3350
 	1    0    0    -1
 $EndComp
@@
 L Connector_Generic:Conn_01x03 J20
 U 1 1 638BBCF8
-P 8000 4000
-F 0 "J20" V 8100 3950 50  0000 L CNN
-F 1 "Conn_01x03" V 8200 3800 50  0000 L CNN
-F 2 "Connector_PinHeader_2.54mm:PinHeader_1x03_P2.54mm_Vertical" H 8000 4000 50  0001 C CNN
-F 3 "~" H 8000 4000 50  0001 C CNN
-	1    8000 4000
+P 8000 4250
+F 0 "J20" V 8100 4200 50  0000 L CNN
+F 1 "Conn_01x03" V 8200 4050 50  0000 L CNN
+F 2 "Connector_PinHeader_2.54mm:PinHeader_1x03_P2.54mm_Vertical" H 8000 4250 50  0001 C CNN
+F 3 "~" H 8000 4250 50  0001 C CNN
+	1    8000 4250
 	1    0    0    -1
 $EndComp
@@
 L power:GND #PWR?
 U 1 1 638BE07F
-P 7800 4000
+P 7800 4250
 AR Path="/63777FB0/638BE07F" Ref="#PWR?"  Part="1"
 AR Path="/638BE07F" Ref="#PWR0101"  Part="1"
-F 0 "#PWR0101" H 7800 3750 50  0001 C CNN
-F 1 "GND" V 7805 3872 50  0000 R CNN
-F 2 "" H 7800 4000 50  0001 C CNN
-F 3 "" H 7800 4000 50  0001 C CNN
-	1    7800 4000
+F 0 "#PWR0101" H 7800 4000 50  0001 C CNN
+F 1 "GND" V 7805 4122 50  0000 R CNN
+F 2 "" H 7800 4250 50  0001 C CNN
+F 3 "" H 7800 4250 50  0001 C CNN
+	1    7800 4250
 	0    1    1    0
 $EndComp
@@
 L power:GND #PWR?
 U 1 1 638BE1F1
-P 7800 4100
+P 7800 4350
 AR Path="/63777FB0/638BE1F1" Ref="#PWR?"  Part="1"
 AR Path="/638BE1F1" Ref="#PWR0102"  Part="1"
-F 0 "#PWR0102" H 7800 3850 50  0001 C CNN
-F 1 "GND" V 7805 3972 50  0000 R CNN
-F 2 "" H 7800 4100 50  0001 C CNN
-F 3 "" H 7800 4100 50  0001 C CNN
-	1    7800 4100
+F 0 "#PWR0102" H 7800 4100 50  0001 C CNN
+F 1 "GND" V 7805 4222 50  0000 R CNN
+F 2 "" H 7800 4350 50  0001 C CNN
+F 3 "" H 7800 4350 50  0001 C CNN
+	1    7800 4350
 	0    1    1    0
 $EndComp
@@
 L power:GND #PWR?
 U 1 1 638D1F7A
-P 7800 2850
+P 7800 3050
 AR Path="/63777FB0/638D1F7A" Ref="#PWR?"  Part="1"
 AR Path="/638D1F7A" Ref="#PWR?"  Part="1"
-F 0 "#PWR?" H 7800 2600 50  0001 C CNN
-F 1 "GND" V 7805 2722 50  0000 R CNN
-F 2 "" H 7800 2850 50  0001 C CNN
-F 3 "" H 7800 2850 50  0001 C CNN
-	1    7800 2850
-	0    1    1    0
-$EndComp
+F 0 "#PWR?" H 7800 2800 50  0001 C CNN
+F 1 "GND" V 7805 2922 50  0000 R CNN
+F 2 "" H 7800 3050 50  0001 C CNN
+F 3 "" H 7800 3050 50  0001 C CNN
+	1    7800 3050
+	0    1    1    0
+$EndComp

Commit message: Add files via upload
Parts:
- removed D20: ECU, LED_THT:LED_D5.0mm, symbol Device:LED
- added D2, D20: LED, LED_THT:LED_D5.0mm, symbol V10-Ign-Inj-Drivers-V2-rescue:LED
- added R1: 2.4K, Resistor_THT:R_Axial_DIN0207_L6.3mm_D2.5mm_P2.54mm_Vertical, symbol Device:R
- R18: value 1K -> 2.4K
Connections:
- wire segments 197 -> 201
Other:
- note added: "Header terminal connections to DB1600iAuxBot board"
- note added: "Left side vehicle wiring terminals"
- note added: "Right side vehicle wiring terminals"
- moved on the sheet: J1, J13, J20, J23, J5

Commit message: Add files via upload
Parts:
- added RN1: R_Network03_US, Resistor_THT:R_Array_SIP4, symbol Device:R_Network03_US
- added RN2: R_Pack02_SIP, Resistor_THT:R_Array_SIP4, symbol Device:R_Pack02_SIP
Connections:
- wire segments 201 -> 209
Other:
- note added: "100K"
Changed lines of the file:
@@
 	6900 1850 6900 1500
 Connection ~ 6900 1500
+$Comp
+L Device:R_Network03_US RN1
+U 1 1 639FC361
+P 1800 6800
+F 0 "RN1" V 1483 6800 50  0000 C CNN
+F 1 "R_Network03_US" V 1574 6800 50  0000 C CNN
+F 2 "Resistor_THT:R_Array_SIP4" V 2075 6800 50  0001 C CNN
+F 3 "http://www.vishay.com/docs/31509/csc.pdf" H 1800 6800 50  0001 C CNN
+	1    1800 6800
+	0    1    1    0
+$EndComp
+$Comp
+L power:GND #PWR?
+U 1 1 63A3DFE7
+P 2150 6700
+AR Path="/63777FB0/63A3DFE7" Ref="#PWR?"  Part="1"
+AR Path="/63A3DFE7" Ref="#PWR0104"  Part="1"
+F 0 "#PWR0104" H 2150 6450 50  0001 C CNN
+F 1 "GND" H 2150 6550 50  0000 C CNN
+F 2 "" H 2150 6700 50  0000 C CNN
+F 3 "" H 2150 6700 50  0000 C CNN
+	1    2150 6700
+	0    -1   -1   0
+$EndComp
+Text GLabel 1500 6700 0    60   Input ~ 0
+D13-control
+Text GLabel 1500 6800 0    60   Input ~ 0
+D10-control
+Text GLabel 1500 6900 0    60   Input ~ 0
+D11-control
+Text GLabel 4100 2950 3    60   Input ~ 0
+D8-control
+Text GLabel 4300 2950 3    60   Input ~ 0
+D9-control
+$Comp
+L power:GND #PWR0105
+U 1 1 63A3EC69
+P 4400 2950
+F 0 "#PWR0105" H 4400 2700 50  0001 C CNN
+F 1 "GND" V 4400 2750 50  0000 C CNN
+F 2 "" H 4400 2950 50  0001 C CNN
+F 3 "" H 4400 2950 50  0001 C CNN
+	1    4400 2950
+	1    0    0    -1
+$EndComp
+Wire Wire Line
+	2000 6700 2150 6700
+Wire Wire Line
+	1600 6700 1500 6700
+Wire Wire Line
+	1600 6800 1500 6800
+Wire Wire Line
+	1600 6900 1500 6900
+Text Notes 4100 2250 0    50   ~ 0
+100K
+Text Notes 1700 7100 0    50   ~ 0
+100K
+$Comp
+L Device:R_Pack02_SIP RN2
+U 1 1 639FE9B3
+P 4200 2650
+F 0 "RN2" H 4100 3000 50  0000 L CNN
+F 1 "R_Pack02_SIP" H 3950 2900 50  0000 L CNN
+F 2 "Resistor_THT:R_Array_SIP4" V 4575 2650 50  0001 C CNN
+F 3 "http://www.vishay.com/docs/31509/csc.pdf" H 4200 2650 50  0001 C CNN
+	1    4200 2650
+	1    0    0    -1
+$EndComp
+$Comp
+L power:GND #PWR0106
+U 1 1 63AC1D04
+P 4000 2950
+F 0 "#PWR0106" H 4000 2700 50  0001 C CNN
+F 1 "GND" V 4000 2750 50  0000 C CNN
+F 2 "" H 4000 2950 50  0001 C CNN
+F 3 "" H 4000 2950 50  0001 C CNN
+	1    4000 2950
+	1    0    0    -1
+$EndComp
+Wire Wire Line
+	4400 2850 4400 2950
+Wire Wire Line
+	4300 2850 4300 2950
+Wire Wire Line
+	4100 2850 4100 2950
+Wire Wire Line
+	4000 2850 4000 2950
 $EndSCHEMATC

Commit message: Add files via upload
Parts:
- K1, K2: footprint DP1600iAuxTop:VCF4-1000 -> Buggly SPD Aux:VCF4-1000
Changed lines of the file:
@@
 F 0 "K1" V 4300 1200 50  0000 C CNN
 F 1 "Main" V 4450 1200 50  0000 C CNN
-F 2 "DP1600iAuxTop:VCF4-1000" H 6040 1160 50  0001 C CNN
+F 2 "Buggly SPD Aux:VCF4-1000" H 6040 1160 50  0001 C CNN
 F 3 "http://gfinder.findernet.com/assets/Series/353/S40EN.pdf" H 4900 1200 50  0001 C CNN
 	1    4900 1200
@@
 F 0 "K2" V 5350 1200 50  0000 C CNN
 F 1 "Automatic Shut Down" V 5474 1200 50  0000 C CNN
-F 2 "DP1600iAuxTop:VCF4-1000" H 7090 1160 50  0001 C CNN
+F 2 "Buggly SPD Aux:VCF4-1000" H 7090 1160 50  0001 C CNN
 F 3 "http://gfinder.findernet.com/assets/Series/353/S40EN.pdf" H 5950 1200 50  0001 C CNN
 	1    5950 1200
