File: KiCad Files/DP1600iAuxBot/file64A3EE68.sch (KiCad schematic (older format))
At the start: 0 parts

Commit message: Add files via upload
Parts:
- added J36: Conn_01x01, Connector_PinHeader_2.54mm:PinHeader_1x01_P2.54mm_Vertical, symbol Connector_Generic:Conn_01x01
- added J37: Conn_01x02, Connector_PinHeader_2.54mm:PinHeader_1x02_P2.54mm_Vertical, symbol Connector_Generic:Conn_01x02
- added J38: Conn_01x03, Connector_PinHeader_2.54mm:PinHeader_1x03_P2.54mm_Vertical, symbol Connector_Generic:Conn_01x03
- added J39: Conn_01x04, Connector_PinHeader_2.54mm:PinHeader_1x04_P2.54mm_Vertical, symbol Connector_Generic:Conn_01x04
- added J40, J41, J43, J45, J46, J47, J48: Conn_01x05, Connector_PinHeader_2.54mm:PinHeader_1x05_P2.54mm_Vertical, symbol Connector_Generic:Conn_01x05
- added J49, J50: Conn_01x23, Connector_PinHeader_2.54mm:PinHeader_1x23_P2.54mm_Vertical, symbol Connector_Generic:Conn_01x23
- added J51, J52, J53: Conn_01x17, Connector_PinHeader_2.54mm:PinHeader_1x17_P2.54mm_Vertical, symbol Connector_Generic:Conn_01x17
- added J54, J55: Conn_01x10, Connector_PinHeader_2.54mm:PinHeader_1x10_P2.54mm_Vertical, symbol Connector_Generic:Conn_01x10
- added J56, J57: Conn_01x09, Connector_PinHeader_2.54mm:PinHeader_1x09_P2.54mm_Vertical, symbol Connector_Generic:Conn_01x09
Connections:
- no-connect marks 0 -> 180
Other:
- note added: "Proto header 10\n\n"
- note added: "Proto header 11\n\n"
- note added: "Proto header 12\n\n"
- note added: "Proto header 13\n\n\n"
- note added: "Proto header 14\n\n\n"
- note added: "Proto header 15\n\n\n"
- note added: "Proto header 16\n\n\n"
- note added: "Proto header 17\n\n\n"
- note added: "Proto header 2"
- note added: "Proto header 3"
- note added: "Proto header 4"
- note added: "Proto header 5"
- note added: "Proto header 6"
- note added: "Proto header 7"
- note added: "Proto header 8"
- note added: "Proto header 9\n"

Commit message: Add files via upload
Parts:
- removed J36: Conn_01x01, Connector_PinHeader_2.54mm:PinHeader_1x01_P2.54mm_Vertical, symbol Connector_Generic:Conn_01x01
- removed J37: Conn_01x02, Connector_PinHeader_2.54mm:PinHeader_1x02_P2.54mm_Vertical, symbol Connector_Generic:Conn_01x02
- removed J38: Conn_01x03, Connector_PinHeader_2.54mm:PinHeader_1x03_P2.54mm_Vertical, symbol Connector_Generic:Conn_01x03
- removed J39: Conn_01x04, Connector_PinHeader_2.54mm:PinHeader_1x04_P2.54mm_Vertical, symbol Connector_Generic:Conn_01x04
- removed J40, J41, J43, J45, J46, J47, J48: Conn_01x05, Connector_PinHeader_2.54mm:PinHeader_1x05_P2.54mm_Vertical, symbol Connector_Generic:Conn_01x05
- removed J49, J50: Conn_01x23, Connector_PinHeader_2.54mm:PinHeader_1x23_P2.54mm_Vertical, symbol Connector_Generic:Conn_01x23
- removed J51, J52, J53: Conn_01x17, Connector_PinHeader_2.54mm:PinHeader_1x17_P2.54mm_Vertical, symbol Connector_Generic:Conn_01x17
- removed J54, J55: Conn_01x10, Connector_PinHeader_2.54mm:PinHeader_1x10_P2.54mm_Vertical, symbol Connector_Generic:Conn_01x10
- removed J56, J57: Conn_01x09, Connector_PinHeader_2.54mm:PinHeader_1x09_P2.54mm_Vertical, symbol Connector_Generic:Conn_01x09
Connections:
- no-connect marks 180 -> 0
Other:
- note removed: "Proto header 10\n\n"
- note removed: "Proto header 11\n\n"
- note removed: "Proto header 12\n\n"
- note removed: "Proto header 13\n\n\n"
- note removed: "Proto header 14\n\n\n"
- note removed: "Proto header 15\n\n\n"
- note removed: "Proto header 16\n\n\n"
- note removed: "Proto header 17\n\n\n"
- note removed: "Proto header 2"
- note removed: "Proto header 3"
- note removed: "Proto header 4"
- note removed: "Proto header 5"
- note removed: "Proto header 6"
- note removed: "Proto header 7"
- note removed: "Proto header 8"
- note removed: "Proto header 9\n"
