File: KiCad Files/DP1600iAuxBot/DP1600iAuxBot.kicad_pcb (KiCad board)
At the start: 2 copper layers, 120.4 x 100.1 mm, 70 parts, among them IC1 Trig Cond Socket, J1 Conn_01x01, J10 Conn_01x01, J11 Conn_01x01, J12 Conn_01x01, J13 Conn_01x01, J14 Conn_01x01, J15 Conn_01x01, J16 Conn_01x01, J17 Conn_01x01, J18 Conn_01x01, J19 Conn_01x01, J2 Conn_01x01, J20 Conn_01x01, J21 Conn_01x01, J22 DB25_Female, J23 Conn_01x01, J24 Conn_01x01, J25 Conn_01x01, J26 Conn_01x01, J27 Conn_01x01, J28 Conn_01x01, J29 Conn_01x01, J3 Conn_01x01, J30 Conn_01x01, J31 Conn_01x01, J32 Conn_01x01, J33 Conn_01x01, J36 Conn_01x01, J37 Conn_01x02, J38 Conn_01x03, J39 Conn_01x04, J4 Conn_01x01, J40 Conn_01x05, J41 Conn_01x05, J43 Conn_01x05, J45 Conn_01x05, J46 Conn_01x05, J47 Conn_01x05, J48 Conn_01x05, J49 Conn_01x23, J5 Conn_01x01, J50 Conn_01x23, J51 Conn_01x17, J52 Conn_01x17, J53 Conn_01x17, J54 Conn_01x10, J55 Conn_01x10, J56 Conn_01x09, J57 Conn_01x09, J6 Conn_01x01, J7 Conn_01x01, J8 Conn_01x01, J9 Conn_01x01, Q1 2N3906

Commit message: Add files via upload
Parts:
- removed the J1 at (273.2, 131.1)
- removed J10, J11, J12, J13, J14, J15, J16, J17, J18, J19, J20, J21, J23, J24, J25, J26, J27, J28, J29, J30, J31, J32, J33, J36, J7, J8, J9: Conn_01x01, Connector_PinHeader_2.54mm:PinHeader_1x01_P2.54mm_Vertical
- removed J37: Conn_01x02, Connector_PinHeader_2.54mm:PinHeader_1x02_P2.54mm_Vertical
- removed J38: Conn_01x03, Connector_PinHeader_2.54mm:PinHeader_1x03_P2.54mm_Vertical
- removed J39: Conn_01x04, Connector_PinHeader_2.54mm:PinHeader_1x04_P2.54mm_Vertical
- removed J40, J41, J43, J45, J46, J47, J48: Conn_01x05, Connector_PinHeader_2.54mm:PinHeader_1x05_P2.54mm_Vertical
- removed J49, J50: Conn_01x23, Connector_PinHeader_2.54mm:PinHeader_1x23_P2.54mm_Vertical
- removed J51, J52, J53: Conn_01x17, Connector_PinHeader_2.54mm:PinHeader_1x17_P2.54mm_Vertical
- removed J54, J55: Conn_01x10, Connector_PinHeader_2.54mm:PinHeader_1x10_P2.54mm_Vertical
- removed J56, J57: Conn_01x09, Connector_PinHeader_2.54mm:PinHeader_1x09_P2.54mm_Vertical
- added R10: 10M, Resistor_THT:R_Axial_DIN0207_L6.3mm_D2.5mm_P7.62mm_Horizontal, F.Cu at (150.0, 110.2)
- added R11: 10M, Resistor_THT:R_Axial_DIN0207_L6.3mm_D2.5mm_P7.62mm_Horizontal, F.Cu at (153.3, 110.2)
- added R12: 10M, Resistor_THT:R_Axial_DIN0207_L6.3mm_D2.5mm_P7.62mm_Horizontal, F.Cu at (137.2, 56.7)
- added R13: 10M, Resistor_THT:R_Axial_DIN0207_L6.3mm_D2.5mm_P7.62mm_Horizontal, F.Cu at (137.2, 59.9)
- added R14: 1k, Resistor_THT:R_Axial_DIN0207_L6.3mm_D2.5mm_P7.62mm_Horizontal, F.Cu at (144.6, 67.8)
- added R15: 1k, Resistor_THT:R_Axial_DIN0207_L6.3mm_D2.5mm_P7.62mm_Horizontal, F.Cu at (144.9, 82.0)
- added R6: 10M, Resistor_THT:R_Axial_DIN0207_L6.3mm_D2.5mm_P7.62mm_Horizontal, F.Cu at (137.2, 50.3)
- added R7: 10M, Resistor_THT:R_Axial_DIN0207_L6.3mm_D2.5mm_P7.62mm_Horizontal, F.Cu at (137.2, 53.5)
- added R8: 10M, Resistor_THT:R_Axial_DIN0207_L6.3mm_D2.5mm_P7.62mm_Horizontal, F.Cu at (162.8, 110.3)
- added R9: 10M, Resistor_THT:R_Axial_DIN0207_L6.3mm_D2.5mm_P7.62mm_Horizontal, F.Cu at (137.2, 47.1)
- J2: value Conn_01x01 -> Conn_01x02; footprint Connector_PinHeader_2.54mm:PinHeader_1x01_P2.54mm_Vertical -> Connector_PinHeader_2.54mm:PinHeader_1x02_P2.54mm_Vertical
- J3: value Conn_01x01 -> Conn_01x03; footprint Connector_PinHeader_2.54mm:PinHeader_1x01_P2.54mm_Vertical -> Connector_PinHeader_2.54mm:PinHeader_1x03_P2.54mm_Vertical
- J4: value Conn_01x01 -> Conn_01x06; footprint Connector_PinHeader_2.54mm:PinHeader_1x01_P2.54mm_Vertical -> Connector_PinHeader_2.54mm:PinHeader_1x06_P2.54mm_Vertical
- J5: value Conn_01x01 -> Conn_01x09; footprint Connector_PinHeader_2.54mm:PinHeader_1x01_P2.54mm_Vertical -> Connector_PinHeader_2.54mm:PinHeader_1x09_P2.54mm_Vertical
- J6: value Conn_01x01 -> Conn_01x10; footprint Connector_PinHeader_2.54mm:PinHeader_1x01_P2.54mm_Vertical -> Connector_PinHeader_2.54mm:PinHeader_1x10_P2.54mm_Vertical
- JP2: value VR-HALL -> PULL-UP; footprint Connector_PinHeader_2.54mm:PinHeader_1x03_P2.54mm_Vertical -> Connector_PinHeader_2.54mm:PinHeader_1x02_P2.54mm_Vertical
- JP4: value PULL-UP -> VR-HALL; footprint Connector_PinHeader_2.54mm:PinHeader_1x02_P2.54mm_Vertical -> Connector_PinHeader_2.54mm:PinHeader_1x03_P2.54mm_Vertical
- Q1: footprint Package_TO_SOT_THT:TO-92_Wide -> Package_TO_SOT_THT:TO-92_Inline_Wide
- R1: value 1k -> 24K; footprint Resistor_THT:R_Axial_DIN0204_L3.6mm_D1.6mm_P5.08mm_Horizontal -> Resistor_THT:R_Axial_DIN0207_L6.3mm_D2.5mm_P7.62mm_Horizontal
- R2: value 24K -> 4.7K
- R3: value 1k -> 1K; footprint Resistor_THT:R_Axial_DIN0204_L3.6mm_D1.6mm_P5.08mm_Horizontal -> Resistor_THT:R_Axial_DIN0207_L6.3mm_D2.5mm_P7.62mm_Horizontal
- R4: value 4.7K -> 10M
- R5: value 1K -> 10M
- moved J4 174.7 mm to (120.7, 47.0)
- moved J2 165.9 mm to (120.7, 83.8)
- moved JP1 147.3 mm to (148.4, 70.4), turned to 180 degrees
- moved R3 125.3 mm to (128.5, 111.6)
- moved IC1 124.3 mm to (159.6, 70.9)
- moved J5 114.8 mm to (131.6, 121.3), turned to 270 degrees
- moved C1 107.3 mm to (172.5, 68.1), turned to 270 degrees
- moved D3 104.7 mm to (176.6, 77.0)
- moved R2 103.0 mm to (132.8, 116.4)
- moved R1 102.8 mm to (143.2, 116.4)
- moved JP3 101.4 mm to (154.5, 72.9), turned to 180 degrees
- moved C2 100.0 mm to (172.2, 77.0), turned to 270 degrees
- moved JP4 96.9 mm to (154.5, 76.7)
- moved JP2 96.0 mm to (148.7, 79.5)
- moved Q1 95.8 mm to (144.2, 111.6), turned to 180 degrees
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- renumbered J22 to J1
Connections:
- IC1 pad 1: CKP-VR- -> CKP-
- IC1 pad 4: CMP-VR- -> CMP-
- J2 pad 1: CKP-VR- -> CMP+
- J3 pad 1: CMP-VR- -> GND
- J4 pad 1: CMP-VR+ -> D48-control
- J6 pad 1: F7-out -> GND
- JP1 pad 1: CKP-VR+ -> CKP+
- JP2 pad 1: Net-(IC1-Pad2) -> CMP+
- JP2 pad 2: CKP-VR+ -> Net-(JP2-Pad2)
- JP3 pad 1: Net-(IC1-Pad3) -> Net-(IC1-Pad2)
- JP3 pad 2: CMP-VR+ -> CKP+
- JP3 pad 3: MCU-D18 -> MCU-D19
- JP4 pad 1: CMP-VR+ -> Net-(IC1-Pad3)
- JP4 pad 2: Net-(JP4-Pad2) -> CMP+
- Q1 pad 1: F7-out -> F9-out
- R1 pad 1: Net-(JP1-Pad2) -> Net-(Q1-Pad2)
- R1 pad 2: VDD -> F9-out
- R2 pad 1: Net-(Q1-Pad2) -> D49-control
- R2 pad 2: F7-out -> Net-(Q1-Pad2)
- R3 pad 1: Net-(JP4-Pad2) -> Tachometer
- R3 pad 2: VDD -> Net-(Q1-Pad3)
- R4 pad 1: D49-control -> GND
- R4 pad 2: Net-(Q1-Pad2) -> D8-control
- R5 pad 1: Tachometer -> GND
- R5 pad 2: Net-(Q1-Pad3) -> D9-control
Routing:
- net MCU-D18: track 0.00 -> 142.0 mm, vias 0 -> 6
- net VDD: track 0.00 -> 128.1 mm, vias 0 -> 1
- net MCU-D19: track 0.00 -> 99.7 mm, vias 0 -> 2
- net 12V-Raw: track 0.00 -> 89.8 mm
- net D12-control: track 0.00 -> 83.3 mm
- net D8-control: track 0.00 -> 82.7 mm, vias 0 -> 1
- net D9-control: track 0.00 -> 81.0 mm, vias 0 -> 1
- net D51-control: track 0.00 -> 76.5 mm
- net D50-control: track 0.00 -> 71.5 mm
- net D49-control: track 0.00 -> 66.9 mm
- net VDDA: track 0.00 -> 47.2 mm
- net SigRtn: track 0.00 -> 47.1 mm
- net CKP+: track 0.00 -> 46.3 mm, vias 0 -> 1
- net CMP-: track 0.00 -> 44.3 mm
- net F9-out: track 0.00 -> 43.8 mm
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- added copper zone on B.Cu, net GND
- added copper zone on F.Cu, net GND
Other:
- board text added: "12V-Raw"
- board text added: "CKP+"
- board text added: "CKP-"
- board text added: "CLT"
- board text added: "CMP+"
- board text added: "CMP-"
- board text added: "D10 cntrl"
- board text added: "D11 cntrl"
- board text added: "D12 cntrl"
- board text added: "D13 cntrl"
- board text added: "D48 cntrl"
- board text added: "D50 cntrl"
- board text added: "D51 cntrl"
- board text added: "D52 cntrl"
- board text added: "D53 cntrl"
- board text added: "D8 cntrl"
- board text added: "D9 cntrl"
- board text added: "F9 out"
- board text added: "Gnd"
- board text added: "IAT"
- board text added: "O2"
- board text added: "SigRtn"
- board text added: "Spare"
- board text added: "TPS"
- board text added: "Tachometer"
- board text added: "VDDA"

Commit message: Add files via upload
Other:
- board text added: "DP1600iAuxBot"
- board text added: "MADE FOR SPEEDUINO"
- board text added: "PCB design by Robert Hiebert December 2022"

Commit message: Add files via upload
Parts:
- removed R10, R11, R12, R13, R4, R5, R6, R7, R8, R9: 10M, Resistor_THT:R_Axial_DIN0207_L6.3mm_D2.5mm_P7.62mm_Horizontal
- added JP5: EN-DIS, Connector_PinHeader_2.54mm:PinHeader_1x03_P2.54mm_Vertical, F.Cu at (142.6, 77.6)
- added JP6: DIS-EN, Connector_PinHeader_2.54mm:PinHeader_1x03_P2.54mm_Vertical, F.Cu at (138.3, 87.0)
- added JP7: EN-DIS, Connector_PinHeader_2.54mm:PinHeader_1x03_P2.54mm_Vertical, F.Cu at (179.1, 84.6)
- D2, D4: value 1N5818 -> 1N5231B
- JP4: value VR-HALL -> HALL-VR
- moved D4 0.05 mm to (186.7, 80.2)
Connections:
- D2 pad 1: VDD -> GND
- D4 pad 1: VDD -> GND
- IC1 pad 4: CMP- -> Net-(IC1-Pad4)
- IC1 pad 7: MCU-D18 -> Net-(IC1-Pad7)
- JP4 pad 1: Net-(IC1-Pad3) -> Net-(JP4-Pad1)
Routing:
- net VDD: track 128.1 -> 90.5 mm
- net Net-(IC1-Pad7): track 0.00 -> 24.2 mm
- net Net-(IC1-Pad4): track 0.00 -> 23.7 mm
- net CMP-: track 44.3 -> 23.6 mm
- net Net-(JP4-Pad1): track 0.00 -> 12.3 mm
- net Net-(IC1-Pad3): track 5.40 -> 17.7 mm
- net D13-control: track 38.5 -> 28.5 mm
- net D10-control: track 36.6 -> 26.9 mm
- net D11-control: track 32.4 -> 23.0 mm
- net D52-control: track 41.8 -> 32.6 mm
- net D53-control: track 38.0 -> 29.1 mm
- net D12-control: track 83.3 -> 76.0 mm
- net D9-control: track 81.0 -> 74.0 mm
- net D8-control: track 82.7 -> 76.0 mm
- net D51-control: track 76.5 -> 70.0 mm
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Other:
- board text added: "CMP En/Dis"
- board text removed: "D10 cntrl"
- board text removed: "D11 cntrl"
- board text removed: "D13 cntrl"
- board text removed: "D52 cntrl"
- board text removed: "D53 cntrl"

Commit message: Add files via upload
Parts:
- moved D4 10.2 mm to (176.6, 80.3), turned to 0 degrees
- moved D2 10.2 mm to (176.8, 70.6), turned to 0 degrees
Connections:
- D2 pad 1: GND -> MCU-D19
- D2 pad 2: MCU-D19 -> GND
- D4 pad 1: GND -> MCU-D18
- D4 pad 2: MCU-D18 -> GND
