File: KiCad Files/DP1600iAuxBot/DP1600iAuxBot.sch (KiCad schematic (older format))
At the start: 49 parts

Commit message: Add files via upload
Parts:
- removed J?: DB25_Female, Connector_Dsub:DSUB-25_Female_Horizontal_P2.77x2.84mm_EdgePinOffset4.94mm_Housed_MountingHolesOffset7.48mm, symbol Connector:DB25_Female
- removed J?: Conn_01x01, symbol Connector_Generic:Conn_01x01
- added J22: DB25_Female, Connector_Dsub:DSUB-25_Female_Horizontal_P2.77x2.84mm_EdgePinOffset4.94mm_Housed_MountingHolesOffset7.48mm, symbol Connector:DB25_Female
- added J25: Conn_01x01, Connector_PinHeader_2.54mm:PinHeader_1x01_P2.54mm_Vertical, symbol Connector_Generic:Conn_01x01
- J1, J10, J11, J12, J13, J14, J15, J16, J17, J18, J19, J2, J20, J21, J23, J24, J26, J27, J29, J3, J30, J31, J32, J33, J4, J5, J6, J7, J8, J9: renamed from J?; footprint (none) -> Connector_PinHeader_2.54mm:PinHeader_1x01_P2.54mm_Vertical
- gave numbers to parts that had none: 17
Connections:
- net CLT_Sensor: now also J22.15 (P15)
- net D10-control: now also J22.24 (P24)
- net D11-control: now also J22.11
- net D12-control: now also J22.23 (P23)
- net D13-control: now also J22.10
- net D48-control: now also J22.22 (P22)
- net D49-control: now also J22.9
- net D50-control: now also J22.21 (P21)
- net D51-control: now also J22.8
- net D52-control: now also J22.20 (P20)
- net D53-control: now also J22.7
- net D8-control: now also J22.25 (P25)
- net D9-control: now also J22.12
- net GND: now also J22.18 (P18), J22.5
- net IAT_Sensor: now also J22.3
- net MCU-D18: now also J22.6
- net MCU-D19: now also J22.19 (P19)
- net O2_Sensor: now also J22.14 (P14)
- net SigRtn: now also J22.16 (P16)
- net Spare-ADC: now also J22.1
- net TPS_Sensor: now also J22.2
- net VDD: now also D2.1 (K), D4.1 (K), R1.2, R3.2, J22.17 (P17), J25.1 (Pin_1)
- net VDDA: now also J22.4; no longer D2.1 (K), D4.1 (K), R1.2, R3.2
- net 12V renamed 12V-Raw
- net 12V-Raw: now also J22.13
- no-connect marks 1 -> 0
Other:
- note added: "5 Volt ADC"
- note added: "5 volt"
- note removed: "5 volt ADC"
- moved on the sheet: J10, J11, J12, J13, J14, J15, J16, J17, J18, J19, J20, J21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

Commit message: Add files via upload
Parts:
- removed Q1: 2N3906, Package_TO_SOT_THT:TO-92_Wide, symbol Transistor_BJT:2N3906
- added Q1: 2N3906, Package_TO_SOT_THT:TO-92_Inline_Wide, symbol dk_Transistors-Bipolar-BJT-Single:2N3906
Connections:
- net F7-out: now also Q1.1 (E)
- net at R2.1, R4.2: now also Q1.2 (B)
- net at R5.2: now also Q1.3 (C)
Changed lines of the file:
@@
 Wire Wire Line
 	1000 2850 1000 2950
-$Comp
-L Transistor_BJT:2N3906 Q1
-U 1 1 64AAE622
-P 1100 2650
-F 0 "Q1" H 1291 2604 50  0000 L CNN
-F 1 "2N3906" H 1291 2695 50  0000 L CNN
-F 2 "Package_TO_SOT_THT:TO-92_Wide" H 1300 2575 50  0001 L CIN
-F 3 "https://www.fairchildsemi.com/datasheets/2N/2N3906.pdf" H 1100 2650 50  0001 L CNN
-	1    1100 2650
-	-1   0    0    1
-$EndComp
 Text Notes 2500 2700 0    50   ~ 0
 (Sinking Transistor PWM Output from ULN2003)
@@
 	0    -1   -1   0
 $EndComp
+$Comp
+L dk_Transistors-Bipolar-BJT-Single:2N3906 Q1
+U 1 1 63868997
+P 1100 2650
+F 0 "Q1" H 1287 2703 60  0000 L CNN
+F 1 "2N3906" H 1287 2597 60  0000 L CNN
+F 2 "Package_TO_SOT_THT:TO-92_Inline_Wide" H 1300 2850 60  0001 L CNN
+F 3 "https://my.centralsemi.com/get_document.php?cmp=1&mergetype=pd&mergepath=pd&pdf_id=LSSGP072.PDF" H 1300 2950 60  0001 L CNN
+F 4 "2N3906CS-ND" H 1300 3050 60  0001 L CNN "Digi-Key_PN"
+F 5 "2N3906" H 1300 3150 60  0001 L CNN "MPN"
+F 6 "Discrete Semiconductor Products" H 1300 3250 60  0001 L CNN "Category"
+F 7 "Transistors - Bipolar (BJT) - Single" H 1300 3350 60  0001 L CNN "Family"
+F 8 "https://my.centralsemi.com/get_document.php?cmp=1&mergetype=pd&mergepath=pd&pdf_id=LSSGP072.PDF" H 1300 3450 60  0001 L CNN "DK_Datasheet_Link"
+F 9 "/product-detail/en/central-semiconductor-corp/2N3906/2N3906CS-ND/4806878" H 1300 3550 60  0001 L CNN "DK_Detail_Page"
+F 10 "TRANS PNP 40V TO-92" H 1300 3650 60  0001 L CNN "Description"
+F 11 "Central Semiconductor Corp" H 1300 3750 60  0001 L CNN "Manufacturer"
+F 12 "Active" H 1300 3850 60  0001 L CNN "Status"
+	1    1100 2650
+	-1   0    0    -1
+$EndComp
 $EndSCHEMATC

Commit message: Add files via upload
Parts:
- removed J1, J10, J11, J12, J13, J14, J15, J16, J17, J18, J19, J2, J20, J21, J23, J24, J25, J26, J27, J29, J3, J30, J31, J32, J33, J4, J5, J6, J7, J8, J9: Conn_01x01, Connector_PinHeader_2.54mm:PinHeader_1x01_P2.54mm_Vertical, symbol Connector_Generic:Conn_01x01
- added J2: Conn_01x02, Connector_PinHeader_2.54mm:PinHeader_1x02_P2.54mm_Vertical, symbol Connector_Generic:Conn_01x02
- added J3: Conn_01x03, Connector_PinHeader_2.54mm:PinHeader_1x03_P2.54mm_Vertical, symbol Connector_Generic:Conn_01x03
- added J4: Conn_01x06, Connector_PinHeader_2.54mm:PinHeader_1x06_P2.54mm_Vertical, symbol Connector_Generic:Conn_01x06
- added J5: Conn_01x09, Connector_PinHeader_2.54mm:PinHeader_1x09_P2.54mm_Vertical, symbol Connector_Generic:Conn_01x09
- added J6: Conn_01x10, Connector_PinHeader_2.54mm:PinHeader_1x10_P2.54mm_Vertical, symbol Connector_Generic:Conn_01x10
- added R10, R11, R12, R13, R4, R5, R6, R7, R8, R9: 10M, Resistor_THT:R_Axial_DIN0207_L6.3mm_D2.5mm_P7.62mm_Horizontal, symbol Device:R
- R14: renamed from R1; footprint Resistor_THT:R_Axial_DIN0204_L3.6mm_D1.6mm_P5.08mm_Horizontal -> Resistor_THT:R_Axial_DIN0207_L6.3mm_D2.5mm_P7.62mm_Horizontal
- R15: renamed from R3; footprint Resistor_THT:R_Axial_DIN0204_L3.6mm_D1.6mm_P5.08mm_Horizontal -> Resistor_THT:R_Axial_DIN0207_L6.3mm_D2.5mm_P7.62mm_Horizontal
- renumbered J22 to J1, JP4 to JP2, JP2 to JP3, JP3 to JP4, R2 to R1, R4 to R2, R5 to R3
Connections:
- net 12V-Raw: now also J5.2 (Pin_2)
- net CLT_Sensor: now also J5.6 (Pin_6)
- net D10-control: now also J4.3 (Pin_3), R6.2
- net D11-control: now also J4.4 (Pin_4), R7.2
- net D12-control: now also J6.6 (Pin_6), R8.2
- net D13-control: now also J4.2 (Pin_2), R9.2
- net D48-control: now also J4.1 (Pin_1)
- net D50-control: now also J6.10 (Pin_10), R10.2
- net D51-control: now also J6.9 (Pin_9), R11.2
- net D52-control: now also J4.5 (Pin_5), R12.2
- net D53-control: now also J4.6 (Pin_6), R13.2
- net D8-control: now also J6.8 (Pin_8), R4.2
- net D9-control: now also J6.7 (Pin_7), R5.2
- net GND: now also J3.1 (Pin_1), J3.2 (Pin_2), J3.3 (Pin_3), J6.1 (Pin_1), J6.2 (Pin_2), R10.1, R11.1, R12.1, R13.1, R4.1, R5.1, R6.1, R7.1, R8.1, R9.1
- net IAT_Sensor: now also J5.5 (Pin_5)
- net O2_Sensor: now also J5.8 (Pin_8)
- net SigRtn: now also J5.4 (Pin_4)
- net Spare-ADC: now also J5.9 (Pin_9)
- net TPS_Sensor: now also J5.7 (Pin_7)
- net Tachometer: now also J5.1 (Pin_1)
- net VDDA: now also J5.3 (Pin_3)
- net CKP-VR+ renamed CKP+
- net CKP+: now also J6.3 (Pin_3)
- net CKP-VR- renamed CKP-
- net CKP-: now also J6.4 (Pin_4)
- net CMP-VR+ renamed CMP+
- net CMP+: now also J2.1 (Pin_1)
- net CMP-VR- renamed CMP-
- net CMP-: now also J2.2 (Pin_2)
- net F7-out renamed F9-out
- net F9-out: now also J6.5 (Pin_5)
Other:
- note added: "(ran out of real estate on top board)"
- note added: "Header sockets connection to DP1660iAuxTop board"
- note added: "Pull downs for high current drivers"
- note added: "Tachometer driver"
- note removed: "Cam VR sensor +\n"
- note removed: "Cam VR sensor -"

Commit message: Add files via upload
Other:
- note added: "Cam Angle Sensor conditioner"
- note added: "Crank Angle Sensor conditioner"
- note added: "DB25 connections to DP1600i board"
- note added: "Header sockets connections to DP1660iAuxTop board"
- note added: "Tachometer driver circuit"
- note removed: "Cam Angle Sensor"
- note removed: "Connections to DP1600i board"
- note removed: "Crank Angle Sensor"
- note removed: "Header sockets connection to DP1660iAuxTop board"
- note removed: "Tachometer driver"
Changed lines of the file:
@@
 	0    1    -1   0
 $EndComp
-Text Notes 8350 1000 0    74   ~ 0
-Crank Angle Sensor
+Text Notes 8100 700  0    74   ~ 0
+Crank Angle Sensor conditioner
 $Comp
 L Jumper:Jumper_2_Open JP2
@@
 Wire Wire Line
 	9900 900  9900 1000
-Text Notes 8400 2750 0    74   ~ 0
-Cam Angle Sensor
+Text Notes 8100 2950 0    74   ~ 0
+Cam Angle Sensor conditioner
 $Comp
 L Device:R R2
@@
 Tachometer
 Text Notes 800  4900 0    100  ~ 0
-Connections to DP1600i board
+DB25 connections to DP1600i board
 Text GLabel 1900 2650 2    50   Input ~ 0
 D49-control
@@
 Tachometer signal
 Text Notes 850  1500 0    100  ~ 0
-Tachometer driver
+Tachometer driver circuit
 Text Notes 6950 4000 0    100  ~ 0
-Header sockets connection to DP1660iAuxTop board
+Header sockets connections to DP1660iAuxTop board
 $EndSCHEMATC

Commit message: Add files via upload
Parts:
- removed D2, D4: 1N5818, Diode_THT:D_DO-41_SOD81_P10.16mm_Horizontal, symbol Diode:1N5818
- removed R10, R11, R12, R13, R4, R5, R6, R7, R8, R9: 10M, Resistor_THT:R_Axial_DIN0207_L6.3mm_D2.5mm_P7.62mm_Horizontal, symbol Device:R
- added D2, D4: 1N5231B, Diode_THT:D_DO-41_SOD81_P10.16mm_Horizontal, symbol V10-Ign-Inj-Drivers-V2-rescue:ZENERsmall
- added JP5, JP7: EN-DIS, Connector_PinHeader_2.54mm:PinHeader_1x03_P2.54mm_Vertical, symbol Jumper:Jumper_3_Open
- added JP6: DIS-EN, Connector_PinHeader_2.54mm:PinHeader_1x03_P2.54mm_Vertical, symbol Jumper:Jumper_3_Open
- JP4: value VR-HALL -> HALL-VR
Connections:
- net CMP-: now also JP6.2 (C); no longer IC1.4 (Pin_4)
- net GND: now also D2.1 (K), D4.1 (K), JP5.3 (B), JP6.1 (A), JP7.3 (B)
- net MCU-D18: now also D4.2 (A), JP7.1 (A); no longer IC1.7 (Pin_7)
- net MCU-D19: now also D2.2 (A)
- net at JP4.1 (A): now also JP5.1 (A); no longer IC1.3 (Pin_3)
- new net: IC1.7 (Pin_7), JP7.2 (C)
- new net: IC1.3 (Pin_3), JP5.2 (C)
- new net: IC1.4 (Pin_4), JP6.3 (B)
Other:
- note added: "(Pin defaults low. Goes high after boot sequence, goes low \nat start of coil dwell, goes Hi after end of coil dwell.)\n"
- note added: "CMP Enable/Disable"
- note added: "DIP8 sized socket pair will accept conditioner modules from WTMotronics, \nJB Perf V2.1, and possibly others that use the MAX9926 chip."
- note removed: "(ran out of real estate on top board)"
- note removed: "Pull downs for high current drivers"
- moved on the sheet: C2, D3, JP2, JP4, R15

Commit message: Add files via upload
Connections:
- net GND: now also D2.2 (A), D4.2 (A); no longer D2.1 (K), D4.1 (K)
- net MCU-D18: now also D4.1 (K); no longer D4.2 (A)
- net MCU-D19: now also D2.1 (K); no longer D2.2 (A)
Other:
- note added: "Optional"
Changed lines of the file:
@@
 U 1 1 639478FB
 P 10100 1000
-F 0 "D2" H 10100 1200 50  0000 C CNN
-F 1 "1N5231B" H 10100 1100 50  0000 C CNN
+F 0 "D2" H 10100 800 50  0000 C CNN
+F 1 "1N5231B" H 10100 900 50  0000 C CNN
 F 2 "Diode_THT:D_DO-41_SOD81_P10.16mm_Horizontal" H 10100 1000 50  0001 C CNN
 F 3 "" H 10100 1000 50  0000 C CNN
 	1    10100 1000
-	-1   0    0    1
+	1    0    0    -1
 $EndComp
 $Comp
@@
 U 1 1 639482ED
 P 10100 3300
-F 0 "D4" H 10100 3500 50  0000 C CNN
-F 1 "1N5231B" H 10100 3400 50  0000 C CNN
+F 0 "D4" H 10100 3050 50  0000 C CNN
+F 1 "1N5231B" H 10100 3150 50  0000 C CNN
 F 2 "Diode_THT:D_DO-41_SOD81_P10.16mm_Horizontal" H 10100 3300 50  0001 C CNN
 F 3 "" H 10100 3300 50  0000 C CNN
 	1    10100 3300
-	-1   0    0    1
+	1    0    0    -1
 $EndComp
 $Comp
@@
 Text Notes 8150 2000 0    50   ~ 0
 CMP Enable/Disable
+Text Notes 8200 3250 0    50   ~ 0
+Optional
 $EndSCHEMATC
